File: kicad/paddle before moving sd from back to front.kicad_pcb (KiCad board)
At the start: 4 copper layers, 198 x 224.8 mm, 175 parts, among them J1101 CONN_02X05, J301 Battery, M501 MICROSD, P1001 100k, P701 100k, P801 100k, P901 100k, Q201 MMBT4401, Q202 MMBT4401, Q301 DMG3414U, Q302 DMG3415U, Q303 DMG3415U, Q401 DMG3415U, Q501 DMG3415U, SW201 RESET*, SW202 BOOTLOAD*, SW301 SW_SPDT, U1001 INA333, U1002 ADS1115, U101 BME280, U102 ESP32-WROOM, U1101 SP3003-04, U1102 SP3003-04, U1201 DNP TLVH431, U1202 OPA333, U201 USB_B_Socket, U202 SP3003-04, U203 CP2104, U301 MCP73831/2, U302 NCP694-3.3, U401 FGPMMOPA6H GPS, U601 NCP694-3.3, U701 INA333, U702 ADS1115, U801 INA333, U802 ADS1115, U901 INA333, U902 ADS1115

Commit message: fix up buttons, move SD to top, add battery holder, add reverse diodes to regs,
change to spst switch and add header for switch
Parts:
- removed D302, D601: RB168LAM, paddle:D_SOD-128
- C501, C502, M501, Q501, R501: moved to B.Cu
- D301: value RB168LAM -> Schottky; footprint paddle:D_SOD-128 -> paddle:D_SMA
- R306: value 10k -> 100k
- SW301: value SW_SPDT -> SW_DPDT_x2; footprint paddle:Pin_Header_Straight_1x03_Pitch2.54mm -> paddle:dpdt_switch
- moved M501 14.4 mm to (85.0, 66.9), turned to 0 degrees
- moved J301 12.7 mm to (103.0, 73.8)
- moved R305 9.72 mm to (98.0, 58.8), turned to 0 degrees
- moved C303 0.50 mm to (107.2, 65.2)
- moved R306 0.50 mm to (107.2, 69.0)
- turned C501 to 270 degrees
- turned C502 to 90 degrees
Connections:
- R306 pad 1: GND -> /SHUTDOWN*
- R306 pad 2: /Power/SHUTDOWN -> +3V3
- SW301 pad 3: /Power/SHUTDOWN -> (no net)
- U102 pad 7: (no net) -> /SHUTDOWN*
Routing:
- net /SD_ENABLE*: track 7.96 -> 33.0 mm, vias 1 -> 3
- net /SD/CS: track 10.3 -> 35.2 mm
- net /SD/DATA_IN: track 18.4 -> 42.5 mm
- net /SD/DATA_OUT: track 11.5 -> 34.3 mm
- net /SD/SCLK: track 10.3 -> 33.2 mm
- net Net-(C501-Pad1): track 0.00 -> 12.4 mm
- net GND: track 13.4 -> 21.9 mm
- net +3V3: track 15.9 -> 17.0 mm, vias 4 -> 5
- net (no net): track 0.07 -> 0.00 mm, vias 1 -> 0
