File: kicad/paddle sd on front, switch on left study.kicad_pcb (KiCad board)
At the start: 4 copper layers, 198 x 224.8 mm, 175 parts, among them J1101 CONN_02X05, J301 Battery, M501 MICROSD, P1001 100k, P701 100k, P801 100k, P901 100k, Q201 MMBT4401, Q202 MMBT4401, Q301 DMG3414U, Q302 DMG3415U, Q303 DMG3415U, Q401 DMG3415U, Q501 DMG3415U, SW201 RESET*, SW202 BOOTLOAD*, SW301 SW_SPDT, U1001 INA333, U1002 ADS1115, U101 BME280, U102 ESP32-WROOM, U1101 SP3003-04, U1102 SP3003-04, U1201 DNP TLVH431, U1202 OPA333, U201 USB_B_Socket, U202 SP3003-04, U203 CP2104, U301 MCP73831/2, U302 NCP694-3.3, U401 FGPMMOPA6H GPS, U601 NCP694-3.3, U701 INA333, U702 ADS1115, U801 INA333, U802 ADS1115, U901 INA333, U902 ADS1115

Commit message: fix up buttons, move SD to top, add battery holder, add reverse diodes to regs,
change to spst switch and add header for switch
Parts:
- removed D302, D601: RB168LAM, paddle:D_SOD-128
- D301: value RB168LAM -> Schottky; footprint paddle:D_SOD-128 -> paddle:D_SMA
- R306: value 10k -> 100k
- SW301: value SW_SPDT -> SW_DPDT_x2; footprint paddle:Pin_Header_Straight_1x03_Pitch2.54mm -> paddle:dpdt_switch
Connections:
- R306 pad 1: GND -> /SHUTDOWN*
- R306 pad 2: /Power/SHUTDOWN -> +3V3
- SW301 pad 3: /Power/SHUTDOWN -> (no net)
- U102 pad 7: (no net) -> /SHUTDOWN*
