File: kicad/paddle.kicad_pcb (KiCad board)
At the start: 4 copper layers, 75 x 50 mm, 169 parts, among them J401 Battery, J501 CONN_02X05, M1101 MICROSD, P1001 100k, P201 100k, P801 100k, P901 100k, Q1101 DMG3415U, Q301 MMBT4401, Q302 MMBT4401, Q401 DMG3414U, Q402 DMG3415U, Q403 DMG3415U, Q701 DMG3415U, SW401 SW_DPDT_x2, U1001 INA333, U1002 ADS1115, U101 BME280, U102 ESP32-WROOM, U201 INA333, U202 ADS1115, U301 USB_B_Socket, U302 SP3003-04, U303 CP2104, U401 MCP73831/2, U402 NCP694-3.3, U403 NCP694-3.3, U501 SP3003-04, U502 SP3003-04, U601 DNP TLVH431, U602 OPA333, U701 FGPMMOPA6H GPS, U801 INA333, U802 ADS1115, U901 INA333, U902 ADS1115

Commit message: More placement studies, last commit before parts reduction
Parts:
- M1101: moved to B.Cu
- moved R502 72.8 mm to (236.2, 51.2)
- moved U502 72.8 mm to (238.9, 42.6)
- moved J501 72.8 mm to (248.6, 38.9)
- moved R501 72.8 mm to (259.8, 39.3)
- moved R504 72.8 mm to (240.1, 51.3)
- moved R506 72.8 mm to (259.5, 43.5)
- moved R508 72.8 mm to (259.5, 48.1)
- moved R503 72.8 mm to (255.6, 39.6)
- moved R505 72.8 mm to (255.6, 44.3)
- moved R507 72.8 mm to (254.8, 48.9)
- moved U501 72.8 mm to (248.2, 48.3)
- moved C1002 70.5 mm to (232.3, 36.8)
- moved C1005 70.5 mm to (226.8, 36.8)
- moved R1002 70.5 mm to (222.6, 30.9)
- moved U1001 70.5 mm to (209.3, 37.4)
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Routing:
- net GND: track 11.7 -> 30.3 mm, vias 6 -> 12
- net Net-(P201-Pad2): track 2.60 -> 4.80 mm
- net +3V3: track 0.00 -> 1.88 mm, vias 0 -> 1
- removed copper zone on In2.Cu, net +3.3VA
Other:
- net class Default: clearance 0.2 -> 0.127
- rule trace_clearance: 0.2 -> 0.127

Commit message: Added second board -
lost footprint changes
Parts:
- removed C402, C404, C407, C408, C411, C412: 0.1uF, paddle:SMD_0805
- added REF**: hole, paddle:KH_F20_mounting_hole, F.Cu at (62.5, 130.0)
- added REF**: hole, paddle:KH_F20_mounting_hole, F.Cu at (112.5, 130.0)
- added REF**: hole, paddle:KH_F20_mounting_hole, F.Cu at (112.5, 170.0)
- added REF**: hole, paddle:KH_F20_mounting_hole, F.Cu at (62.5, 170.0)
- C703: footprint paddle:SMD_1206 -> paddle:SMD_0805
- M1101: moved to F.Cu
- moved R305 202.7 mm to (55.5, 59.0), turned to 90 degrees
- moved Q301 198.3 mm to (52.0, 64.0)
- moved Q302 195.9 mm to (52.0, 59.0), turned to 180 degrees
- moved TP301 193.7 mm to (77.5, 52.5)
- moved R304 190.6 mm to (64.5, 59.5)
- moved R301 189.6 mm to (71.0, 66.5), turned to 180 degrees
- moved TP302 189.3 mm to (77.5, 51.0)
- moved C601 187.1 mm to (84.5, 173.3)
- moved C602 187.1 mm to (95.2, 174.1)
- moved R601 187.1 mm to (103.4, 166.3)
- moved R602 187.1 mm to (90.8, 174.1)
- moved R603 187.1 mm to (99.1, 166.3)
- moved TP601 187.1 mm to (99.9, 169.9)
- moved U601 187.1 mm to (85.6, 166.9)
- moved U602 187.1 mm to (93.9, 167.3)
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Connections:
- C101 pad 1: /RESET* -> /ESP32_RESET*
- L701 pad 1: (no net) -> Net-(C701-Pad1)
- L701 pad 2: (no net) -> Net-(L701-Pad2)
- Q301 pad 3: (no net) -> /ESP32_RESET*
- Q701 pad 3: Net-(C701-Pad1) -> Net-(L701-Pad2)
- R104 pad 2: /RESET* -> /ESP32_RESET*
- U102 pad 3: /RESET* -> /ESP32_RESET*
- U303 pad 25: Net-(U303-Pad25) -> GND
Other:
- board size 75 x 50 mm -> 75 x 125 mm

Commit message: Separate analog block in schematic, fix up board outline, allow for connector, delete bad zones
Parts:
- removed the C201 at (78.5, 135.8)
- removed the C202 at (78.5, 130.8)
- removed C203: DNP 0.01uF, paddle:SMD_0805
- removed C204: 0.1uF, paddle:SMD_0805
- removed C205: 0.01uF, paddle:SMD_0805
- removed C206: 0.22uF, paddle:SMD_0805
- removed C405, C410: 10uF, paddle:SMD_1206
- removed J501: CONN_02X05, paddle:header-0.050-10-pin-through-hole
- removed P201: 100k, paddle:TT_model_23_pot_smd_4mm
- removed the R204 at (74.8, 138.2)
- removed the R205 at (71.2, 136.2)
- removed R206, R603: 10k, paddle:SMD_0805
- removed R207: DNP 100k, paddle:SMD_0805
- removed the R301 at (71.0, 66.5)
- removed the R302 at (77.5, 67.0)
- removed the R303 at (80.5, 63.5)
- removed R406: 100k, paddle:SMD_0805
- removed the R501 at (172.3, 148.8)
- removed R502, R503, R504, R505, R506, R507, R508: 10k 0.1%, paddle:R_0805
- removed R602: 0, paddle:SMD_0805
- removed the TP201 at (80.8, 142.5)
- removed TP601: AN1, paddle:tp_th_1mm
- removed the U201 at (76.2, 141.2)
- removed the U302 at (83.5, 57.5)
- removed U403: NCP694-3.3, paddle:SOT89-5
- removed U501: SP3003-04, paddle:S-PDSO-G8
- removed U502: SP3003-04, paddle:VSSOP10-S-PDSO-G10
- removed U602: OPA333, paddle:sot23-5
- added C1201: DNP 0.1uF, paddle:SMD_0805, F.Cu at (129.3, 115.5)
- added C1202: 0.1uF, paddle:SMD_0805, F.Cu at (149.6, 108.5)
- added C701: 0.01uF, paddle:SMD_0805, F.Cu at (157.8, 82.2)
- added C702: 0.01uF, paddle:SMD_0805, F.Cu at (144.6, 95.4)
- added C703: DNP 0.01uF, paddle:SMD_0805, F.Cu at (129.8, 93.1)
- added C704: 0.1uF, paddle:SMD_0805, F.Cu at (154.2, 88.0)
- added C705: 0.01uF, paddle:SMD_0805, F.Cu at (163.3, 82.2)
- added C706: 0.22uF, paddle:SMD_0805, F.Cu at (150.1, 93.9)
- added J1101: CONN_02X05, paddle:header-0.050-10-pin-through-hole, F.Cu at (162.9, 107.2)
- added LED202: LED, paddle:SMD_D_0805, F.Cu at (80.0, 52.0)
- added P701: 100k, paddle:TT_model_23_pot_smd_4mm, F.Cu at (128.6, 82.1)
- added R1101: 10k 0.1%, paddle:R_0805, F.Cu at (181.3, 117.2)
- added R1102: 10k 0.1%, paddle:R_0805, F.Cu at (177.4, 117.2)
- added R1103: 10k 0.1%, paddle:R_0805, F.Cu at (181.3, 112.5)
- added R1104: 10k 0.1%, paddle:R_0805, F.Cu at (177.4, 112.5)
- added R1105: 10k 0.1%, paddle:R_0805, F.Cu at (181.3, 107.9)
- added R1106: 10k 0.1%, paddle:R_0805, F.Cu at (163.7, 116.8)
- added R1107: 10k 0.1%, paddle:R_0805, F.Cu at (177.4, 107.9)
- added R1108: 10k 0.1%, paddle:R_0805, F.Cu at (159.8, 116.8)
- added R1201: 10k, paddle:SMD_0805, F.Cu at (142.1, 116.3)
- added R1202: 0, paddle:SMD_0805, F.Cu at (147.3, 114.3)
- added R1203: 10k, paddle:SMD_0805, F.Cu at (144.4, 108.5)
- added R701: 10k 0.1%, paddle:SMD_0805, F.Cu at (128.8, 99.0)
- added R702: 20k 0.1%, paddle:SMD_0805, F.Cu at (151.4, 82.2)
- added R703: 1.0M, paddle:SMD_0805, F.Cu at (134.7, 99.0)
- added R704: 250, paddle:SMD_0805, F.Cu at (144.0, 89.5)
- added R705: 0, paddle:SMD_0805, F.Cu at (149.8, 88.0)
- added R706: 10k, paddle:SMD_0805, F.Cu at (138.9, 96.9)
- added R707: DNP 100k, paddle:SMD_0805, F.Cu at (136.1, 82.2)
- added TP101: IO26, paddle:tp_th_1mm, F.Cu at (245.6, 62.3)
- added TP102: IO33, paddle:tp_th_1mm, F.Cu at (247.3, 56.4)
- added TP1201: AN1, paddle:tp_th_1mm, F.Cu at (136.5, 114.2)
- added TP701: AN1, paddle:tp_th_1mm, F.Cu at (149.8, 97.5)
- added U1101: SP3003-04, paddle:SMD_SC70-6, F.Cu at (171.7, 107.4)
- added U1102: SP3003-04, paddle:SMD_SC70-6, F.Cu at (171.7, 114.1)
- added U1201: DNP TLVH431, paddle:SOT-23, F.Cu at (130.4, 109.1)
- added U1202: OPA333, paddle:sot23-5, F.Cu at (138.7, 109.5)
- added U701: INA333, paddle:S-PDSO-G8, F.Cu at (138.1, 88.7)
- added U702: ADS1115, paddle:VSSOP10-S-PDSO-G10, F.Cu at (143.9, 81.3)
- C601: value DNP 0.1uF -> 10uF; footprint paddle:SMD_0805 -> paddle:SMD_1206
- C602: value 0.1uF -> 10uF; footprint paddle:SMD_0805 -> paddle:SMD_1206
- M501: renamed from M1101; moved to B.Cu
- R201: value 10k 0.1% -> 1k; footprint paddle:SMD_0805 -> paddle:R_0805
- R202: value 20k 0.1% -> 330; footprint paddle:SMD_0805 -> paddle:R_0805
- R203: value 1.0M -> 330; footprint paddle:SMD_0805 -> paddle:R_0805
- R601: value 10k -> 100k
- U202: value ADS1115 -> SP3003-04; footprint paddle:VSSOP10-S-PDSO-G10 -> paddle:SMD_SC70-6
- U601: value DNP TLVH431 -> NCP694-3.3; footprint paddle:SOT-23 -> paddle:SOT89-5
- moved R401 180.3 mm to (194.9, 117.7)
- moved R403 171.8 mm to (190.6, 117.7)
- moved C601 162.8 mm to (232.7, 106.0)
- moved C602 148.3 mm to (226.8, 106.0)
- moved U601 146.5 mm to (219.2, 107.0)
- moved R601 134.0 mm to (226.0, 112.4)
- moved R802 106.1 mm to (201.3, 52.7)
- moved R102 100.7 mm to (243.7, 52.7)
- moved C805 92.4 mm to (212.0, 52.7)
- moved C804 92.4 mm to (204.1, 58.6)
- moved C103 89.5 mm to (238.3, 58.6)
- moved U202 89.4 mm to (71.0, 58.0), turned to 0 degrees
- moved R105 87.6 mm to (247.9, 52.7)
- moved R804 87.3 mm to (207.1, 52.7)
- moved R806 81.9 mm to (193.9, 60.1)
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- renumbered C301 to C201, C302 to C202, C401 to C301, C403 to C302, C406 to C303, C409 to C304, C701 to C401, C702 to C402, C703 to C403, C1101 to C501, C1102 to C502, D401 to D301, F401 to F301, J401 to J301, L701 to L401, LED301 to LED201, LED401 to LED301, LED701 to LED401, Q302 to Q201, Q301 to Q202, Q401 to Q301, Q402 to Q302, Q403 to Q303, Q701 to Q401, Q1101 to Q501, R304 to R204, R305 to R205, R401 to R301, R402 to R302, R403 to R303, R404 to R304, R405 to R305, R407 to R306, R701 to R401, R702 to R402, R703 to R403, R704 to R404, R1101 to R501, SW401 to SW301, TP301 to TP201, TP302 to TP202, U301 to U201, U303 to U203, U401 to U301, U402 to U302, U701 to U401
Connections:
- net /Power/V_UNREG_SW renamed /Power/+V_UNREG_SW
- C601 pad 1: Net-(C601-Pad1) -> /+V_UNREG_SW
- LED201 pad A: Net-(LED301-PadA) (its old number) -> Net-(LED201-PadA)
- R1001 pad 2: /IN_3 -> /analog/IN_3
- R1002 pad 2: /VREF -> /analog/VREF
- R1006 pad 2: /AUX_IN_3 -> /analog/AUX_IN_3
- R103 pad 2: /SDA -> /ALERT0
- R201 pad 1: Net-(C201-Pad1) -> Net-(R201-Pad1)
- R201 pad 2: /IN_0 -> +3V3
- R202 pad 1: Net-(C202-Pad1) -> Net-(R202-Pad1)
- R202 pad 2: /VREF -> Net-(LED201-PadA)
- R203 pad 1: Net-(C202-Pad1) -> Net-(R203-Pad1)
- R601 pad 1: Net-(C601-Pad1) -> GND
- R601 pad 2: Net-(R601-Pad2) -> /+3.3VA_ENABLE
- R801 pad 2: /IN_1 -> /analog/IN_1
- R802 pad 2: /VREF -> /analog/VREF
- R806 pad 2: /AUX_IN_1 -> /analog/AUX_IN_1
- R901 pad 2: /IN_2 -> /analog/IN_2
- R902 pad 2: /VREF -> /analog/VREF
- R906 pad 2: /AUX_IN_2 -> /analog/AUX_IN_2
- U1001 pad 5: /VREF -> /analog/VREF
- U1002 pad 7: /VREF -> /analog/VREF
- U1002 pad 9: /SDA -> /ALERT0
- U101 pad 3: /SDA -> /ALERT0
- U102 pad 10: (no net) -> Net-(TP101-Pad1)
- U102 pad 33: /SDA -> /ALERT0
- U102 pad 9: (no net) -> Net-(TP102-Pad1)
- U201 pad 2: Net-(U301-Pad2) -> Net-(U201-Pad2)
- U201 pad 3: Net-(U301-Pad3) -> Net-(U201-Pad3)
- U202 pad 1: GND -> (no net)
- U202 pad 2: /ALERT0 -> GND
- U202 pad 3: GND -> Net-(U201-Pad3)
- U202 pad 4: Net-(C205-Pad1) -> Net-(U201-Pad2)
- U202 pad 5: Net-(TP201-Pad1) -> +3V3
- U202 pad 6: Net-(U201-Pad6) -> /Power/+VBUS
- U203 pad 13: Net-(R303-Pad1) -> Net-(R203-Pad1)
- U203 pad 14: Net-(R302-Pad1) -> Net-(R202-Pad1)
- U203 pad 3: Net-(U301-Pad2) -> Net-(U201-Pad2)
- U203 pad 4: Net-(U301-Pad3) -> Net-(U201-Pad3)
- U203 pad 9: Net-(R301-Pad1) -> Net-(R201-Pad1)
- U601 pad 1: Net-(R601-Pad2) -> (no net)
- U601 pad 2: Net-(C601-Pad1) -> GND
- U601 pad 3: GND -> /+3.3VA_ENABLE
- U801 pad 5: /VREF -> /analog/VREF
- U802 pad 1: +3V3 -> +3.3VA
- U802 pad 7: /VREF -> /analog/VREF
- U802 pad 9: /SDA -> /ALERT0
- U901 pad 5: /VREF -> /analog/VREF
- U902 pad 1: /SDA -> /ALERT0
- U902 pad 7: /VREF -> /analog/VREF
- U902 pad 9: /SDA -> /ALERT0
Routing:
- net /VREF: track 30.5 -> 0.00 mm
- net GND: track 30.3 -> 0.00 mm, vias 12 -> 0
- net Net-(C202-Pad1): track 22.3 -> 0.00 mm, vias 2 -> 0
- net Net-(C205-Pad1): track 11.0 -> 0.00 mm
- net Net-(C201-Pad1): track 10.5 -> 0.00 mm
- net Net-(U201-Pad6): track 8.16 -> 0.00 mm, vias 2 -> 0
- net Net-(R205-Pad2): track 7.11 -> 0.00 mm
- net Net-(R204-Pad2): track 4.91 -> 0.00 mm, vias 2 -> 0
- net Net-(LED202-PadA): track 4.80 -> 0.00 mm
- net +3.3VA: track 4.79 -> 0.00 mm, vias 2 -> 0
- net Net-(R204-Pad1): track 2.13 -> 0.00 mm
- added copper zone on In1.Cu, net +3V3
- added copper zone on In2.Cu, net GND
- removed copper zone on In1.Cu, net GND
Other:
- board size 75 x 125 mm -> 198 x 224.8 mm

Commit message: fix up buttons, move SD to top, add battery holder, add reverse diodes to regs,
change to spst switch and add header for switch
Parts:
- added BT401: CR1025, paddle:CR1025_holder, B.Cu at (55.8, 84.8)
- added D302: RB168LAM, paddle:D_SOD-128, F.Cu at (102.5, 73.0)
- added D601: RB168LAM, paddle:D_SOD-128, F.Cu at (219.0, 101.5)
- added SW201: SWITCH_PUSHBUTTON, paddle:SW_TACTILE_PB_SMD_6MM, F.Cu at (110.2, 80.5)
- added SW202: SWITCH_PUSHBUTTON, paddle:SW_TACTILE_PB_SMD_6MM, F.Cu at (110.2, 74.2)
- D301: value Schottky -> RB168LAM; footprint paddle:D_SMA -> paddle:D_SOD-123
- J301: moved to B.Cu
- M501: moved to F.Cu
- R306: value 100k -> 10k
- SW301: value SW_DPDT_x2 -> SW_SPDT; footprint paddle:dpdt_switch -> paddle:Pin_Header_Straight_1x03_Pitch2.54mm
- moved R105 183.6 mm to (69.2, 95.0), turned to 270 degrees
- moved R108 171.9 mm to (67.2, 95.0), turned to 270 degrees
- moved R102 170.5 mm to (77.2, 90.0)
- moved LED104 167.4 mm to (67.2, 98.2), turned to 90 degrees
- moved LED102 167.3 mm to (73.2, 98.2), turned to 90 degrees
- moved R107 166.7 mm to (71.2, 95.0), turned to 270 degrees
- moved LED101 164.4 mm to (69.2, 98.2), turned to 90 degrees
- moved R106 157.7 mm to (73.2, 95.0), turned to 270 degrees
- moved R103 156.4 mm to (77.2, 85.8)
- moved LED103 154.5 mm to (71.2, 98.2), turned to 90 degrees
- moved TP102 148.6 mm to (101.0, 82.2)
- moved TP101 145.8 mm to (101.0, 81.0)
- moved C103 141.5 mm to (100.8, 92.0), turned to 270 degrees
- moved R101 141.1 mm to (104.0, 84.5)
- moved R401 139.6 mm to (62.2, 74.0)
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Connections:
- net /GPS_RESET* renamed /gps/GPS_RESET*
- C303 pad 1: /Power/+V_UNREG_SW -> /+V_UNREG_SW
- Q302 pad 3: /Power/+V_UNREG_SW -> /+V_UNREG_SW
- R103 pad 2: /ALERT0 -> /SDA
- R306 pad 1: /SHUTDOWN* -> GND
- R306 pad 2: +3V3 -> /Power/SHUTDOWN
- SW301 pad 2: /Power/+V_UNREG_SW -> /+V_UNREG_SW
- SW301 pad 3: (no net) -> /Power/SHUTDOWN
- U1002 pad 9: /ALERT0 -> /SDA
- U101 pad 3: /ALERT0 -> /SDA
- U102 pad 33: /ALERT0 -> /SDA
- U102 pad 7: /SHUTDOWN* -> (no net)
- U202 pad 3: Net-(U201-Pad3) -> Net-(U201-Pad2)
- U202 pad 4: Net-(U201-Pad2) -> Net-(U201-Pad3)
- U203 pad 3: Net-(U201-Pad2) -> Net-(U201-Pad3)
- U203 pad 4: Net-(U201-Pad3) -> Net-(U201-Pad2)
- U302 pad 3: /Power/+V_UNREG_SW -> /+V_UNREG_SW
- U302 pad 4: /Power/+V_UNREG_SW -> /+V_UNREG_SW
- U702 pad 9: /ALERT0 -> /SDA
- U802 pad 9: /ALERT0 -> /SDA
- U902 pad 1: /ALERT0 -> /SDA
- U902 pad 9: /ALERT0 -> /SDA
Routing:
- net /LEDB: track 0.00 -> 46.9 mm, vias 0 -> 2
- net /RXD: track 0.00 -> 38.6 mm, vias 0 -> 2
- net /TXD: track 0.00 -> 38.6 mm, vias 0 -> 2
- net Net-(R402-Pad2): track 0.00 -> 31.5 mm
- net Net-(R403-Pad2): track 0.00 -> 29.5 mm
- net /1PPS: track 0.00 -> 27.6 mm
- net Net-(R203-Pad1): track 0.00 -> 27.4 mm
- net /LEDR: track 0.00 -> 26.1 mm
- net /Power/+VBUS: track 0.00 -> 25.2 mm
- net /LEDY: track 0.00 -> 19.2 mm, vias 0 -> 1
- net Net-(R202-Pad1): track 0.00 -> 18.8 mm, vias 0 -> 2
- net /SD/DATA_IN: track 0.00 -> 18.4 mm, vias 0 -> 1
- net /Power/V_BAT: track 0.00 -> 15.1 mm, vias 0 -> 2
- net +3V3: track 2.27 -> 15.9 mm, vias 1 -> 4
- net GND: track 0.00 -> 13.4 mm, vias 0 -> 6
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