File: kicad/paddle.kicad_pcb (KiCad board)
At the start: 4 copper layers, 198 x 224.8 mm, 175 parts, among them J1101 CONN_02X05, J301 Battery, M501 MICROSD, P1001 100k, P701 100k, P801 100k, P901 100k, Q201 MMBT4401, Q202 MMBT4401, Q301 DMG3414U, Q302 DMG3415U, Q303 DMG3415U, Q401 DMG3415U, Q501 DMG3415U, SW201 SWITCH_PUSHBUTTON, SW202 SWITCH_PUSHBUTTON, SW301 SW_SPDT, U1001 INA333, U1002 ADS1115, U101 BME280, U102 ESP32-WROOM, U1101 SP3003-04, U1102 SP3003-04, U1201 DNP TLVH431, U1202 OPA333, U201 USB_B_Socket, U202 SP3003-04, U203 CP2104, U301 MCP73831/2, U302 NCP694-3.3, U401 FGPMMOPA6H GPS, U601 NCP694-3.3, U701 INA333, U702 ADS1115, U801 INA333, U802 ADS1115, U901 INA333, U902 ADS1115

Commit message: fix diodes - last before 24-bit
add switches?
Parts:
- D301: footprint paddle:D_SOD-123 -> paddle:D_SOD-128
- moved D302 0.35 mm to (102.2, 73.2), turned to 0 degrees
- turned D301 to 0 degrees
Routing:
- net /Power/V_UNREG: track 9.52 -> 13.7 mm
- net /Power/+VBUS: track 25.2 -> 21.0 mm

Commit message: Start switch to 24-bit a/d, smaller buttons, add io expansion, prelim route digital
Parts:
- removed C1001, C1002, C1005, C701, C702, C705, C801, C802, C805, C901, C902, C905: 0.01uF, paddle:SMD_0805
- removed C1003, C703, C803, C903: DNP 0.01uF, paddle:SMD_0805
- removed C1004, C704, C804, C904: 0.1uF, paddle:SMD_0805
- removed C1006, C706, C806, C906: 0.22uF, paddle:SMD_0805
- removed C1201: DNP 0.1uF, paddle:SMD_0805
- removed P1001, P701, P801, P901: 100k, paddle:TT_model_23_pot_smd_4mm
- removed R1001, R701, R801, R901: 10k 0.1%, paddle:SMD_0805
- removed R1002, R702, R802, R902: 20k 0.1%, paddle:SMD_0805
- removed R1003, R703, R803, R903: 1.0M, paddle:SMD_0805
- removed R1004, R704, R804, R904: 250, paddle:SMD_0805
- removed R1005, R1202, R705, R805, R905: 0, paddle:SMD_0805
- removed R1006, R1201, R1203, R706, R806, R906: 10k, paddle:SMD_0805
- removed R1007, R707, R807, R907: DNP 100k, paddle:SMD_0805
- removed TP1001, TP701, TP801, TP901: AN1, paddle:tp_th_1mm
- removed TP101: IO26, paddle:tp_th_1mm
- removed TP102: IO33, paddle:tp_th_1mm
- removed U1201: DNP TLVH431, paddle:SOT-23
- added U103: TCA9534A, paddle:TSSOP-16-1EP_4.4x5mm_Pitch0.65mm, F.Cu at (108.6, 88.8)
- D301: footprint paddle:D_SOD-128 -> paddle:D_SOD-123
- SW201, SW202: footprint paddle:SW_TACTILE_PB_SMD_6MM -> paddle:SW_KMR7
- U1001, U701, U801, U901: value INA333 -> OPA388D
- U1002, U702, U802, U902: value ADS1115 -> LTC2440
- moved SW301 65.4 mm to (53.5, 57.2)
- moved LED104 40.0 mm to (107.2, 98.2)
- moved R108 40.0 mm to (107.2, 95.0)
- moved LED101 36.0 mm to (105.2, 98.2)
- moved R105 36.0 mm to (105.2, 95.0)
- moved LED103 32.0 mm to (103.2, 98.2)
- moved R107 32.0 mm to (103.2, 95.0)
- moved LED102 28.0 mm to (101.2, 98.2)
- moved R106 28.0 mm to (101.2, 95.0)
- moved LED401 11.3 mm to (51.2, 74.0), turned to 90 degrees
- moved C401 9.45 mm to (63.0, 74.0), turned to 0 degrees
- moved R404 9.12 mm to (53.8, 74.0), turned to 270 degrees
- moved L401 8.75 mm to (67.0, 74.0), turned to 270 degrees
- moved C403 7.50 mm to (56.2, 74.0), turned to 270 degrees
- moved R401 7.25 mm to (69.5, 74.0), turned to 90 degrees
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Connections:
- net /gps/GPS_RESET* renamed Net-(U401-Pad2)
- Q401 pad 1: /GPS_EN* -> /GPS_ENABLE*
- R401 pad 2: /GPS_EN* -> /GPS_ENABLE*
- U1001 pad 1: Net-(R1004-Pad1) -> (no net)
- U1001 pad 2: Net-(C1002-Pad1) -> (no net)
- U1001 pad 3: Net-(C1001-Pad1) -> (no net)
- U1001 pad 4: Net-(R1005-Pad2) -> (no net)
- U1001 pad 5: /analog/VREF -> (no net)
- U1001 pad 6: Net-(U1001-Pad6) -> (no net)
- U1001 pad 7: +3.3VA -> (no net)
- U1001 pad 8: Net-(R1004-Pad2) -> (no net)
- U1002 pad 1: /SCK -> (no net)
- U1002 pad 10: /SCK -> (no net)
- U1002 pad 2: /ALERT0 -> (no net)
- U1002 pad 3: GND -> (no net)
- U1002 pad 4: Net-(C1005-Pad1) -> (no net)
- U1002 pad 5: Net-(TP1001-Pad1) -> (no net)
- U1002 pad 6: Net-(U1001-Pad6) -> (no net)
- U1002 pad 7: /analog/VREF -> (no net)
- U1002 pad 8: +3.3VA -> (no net)
- U1002 pad 9: /SDA -> (no net)
- U102 pad 10: Net-(TP101-Pad1) -> (no net)
- U102 pad 11: /KEEPALIVE -> (no net)
- U102 pad 12: /SD_ENABLE* -> (no net)
- U102 pad 13: /LEDG -> (no net)
- U102 pad 14: /LEDY -> (no net)
- U102 pad 16: /LEDR -> (no net)
- U102 pad 23: /LEDB -> (no net)
- U102 pad 24: /1PPS -> (no net)
- U102 pad 26: /GPS_EN* -> (no net)
- U102 pad 4: (no net) -> /1PPS
- U102 pad 8: /+3.3VA_ENABLE -> (no net)
- U102 pad 9: Net-(TP102-Pad1) -> (no net)
- U1202 pad 3: Net-(C1201-Pad1) -> (no net)
- U701 pad 1: Net-(R704-Pad1) -> (no net)
- U701 pad 2: Net-(C702-Pad1) -> (no net)
- U701 pad 3: Net-(C701-Pad1) -> (no net)
- U701 pad 4: Net-(R705-Pad2) -> (no net)
- U701 pad 5: /analog/VREF -> (no net)
- U701 pad 6: Net-(U701-Pad6) -> (no net)
- U701 pad 7: +3.3VA -> (no net)
- U701 pad 8: Net-(R704-Pad2) -> (no net)
- U702 pad 1: GND -> (no net)
- U702 pad 10: /SCK -> (no net)
- U702 pad 2: /ALERT0 -> (no net)
- U702 pad 3: GND -> (no net)
- U702 pad 4: Net-(C705-Pad1) -> (no net)
- U702 pad 5: Net-(TP701-Pad1) -> (no net)
- U702 pad 6: Net-(U701-Pad6) -> (no net)
- U702 pad 7: /analog/VREF -> (no net)
- U702 pad 8: +3.3VA -> (no net)
- U702 pad 9: /SDA -> (no net)
- U801 pad 1: Net-(R804-Pad1) -> (no net)
- U801 pad 2: Net-(C802-Pad1) -> (no net)
- U801 pad 3: Net-(C801-Pad1) -> (no net)
- U801 pad 4: Net-(R805-Pad2) -> (no net)
- U801 pad 5: /analog/VREF -> (no net)
- U801 pad 6: Net-(U801-Pad6) -> (no net)
- U801 pad 7: +3.3VA -> (no net)
- U801 pad 8: Net-(R804-Pad2) -> (no net)
- U802 pad 1: +3.3VA -> (no net)
- U802 pad 10: /SCK -> (no net)
- U802 pad 2: /ALERT0 -> (no net)
- U802 pad 3: GND -> (no net)
- U802 pad 4: Net-(C805-Pad1) -> (no net)
- U802 pad 5: Net-(TP801-Pad1) -> (no net)
- U802 pad 6: Net-(U801-Pad6) -> (no net)
- U802 pad 7: /analog/VREF -> (no net)
- U802 pad 8: +3.3VA -> (no net)
- U802 pad 9: /SDA -> (no net)
- U901 pad 1: Net-(R904-Pad1) -> (no net)
- U901 pad 2: Net-(C902-Pad1) -> (no net)
- U901 pad 3: Net-(C901-Pad1) -> (no net)
- U901 pad 4: Net-(R905-Pad2) -> (no net)
- U901 pad 5: /analog/VREF -> (no net)
- U901 pad 6: Net-(U901-Pad6) -> (no net)
- U901 pad 7: +3.3VA -> (no net)
- U901 pad 8: Net-(R904-Pad2) -> (no net)
- U902 pad 1: /SDA -> (no net)
- U902 pad 10: /SCK -> (no net)
- U902 pad 2: /ALERT0 -> (no net)
- U902 pad 3: GND -> (no net)
- U902 pad 4: Net-(C905-Pad1) -> (no net)
- U902 pad 5: Net-(TP901-Pad1) -> (no net)
- U902 pad 6: Net-(U901-Pad6) -> (no net)
- U902 pad 7: /analog/VREF -> (no net)
- U902 pad 8: +3.3VA -> (no net)
- U902 pad 9: /SDA -> (no net)
Routing:
- net GND: track 13.4 -> 90.6 mm, vias 6 -> 24
- net /BOOTLOAD*: track 0.00 -> 56.8 mm, vias 0 -> 2
- net /ESP32_RESET*: track 0.00 -> 49.0 mm
- net /SDA: track 0.00 -> 48.9 mm, vias 0 -> 2
- net /SCK: track 2.29 -> 49.2 mm, vias 0 -> 2
- net /LEDB: track 46.9 -> 4.42 mm, vias 2 -> 0
- net /RXD: track 38.6 -> 8.73 mm
- net Net-(BT401-Pad+): track 0.00 -> 29.0 mm, vias 0 -> 2
- net /SD/SCLK: track 10.3 -> 39.2 mm, vias 1 -> 4
- net /SD/DATA_IN: track 18.4 -> 46.3 mm, vias 1 -> 2
- net /1PPS: track 27.6 -> 0.00 mm
- net Net-(R203-Pad1): track 27.4 -> 0.00 mm
- net /SD/CS: track 10.3 -> 35.5 mm, vias 1 -> 2
- net Net-(C401-Pad1): track 0.00 -> 24.0 mm
- net Net-(C501-Pad1): track 0.00 -> 21.2 mm
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Other:
- net class power1: clearance 0.2 -> 0.127

Commit message: more layout of digital, LTC2440 test code started
Parts:
- moved SW202 5.10 mm to (111.8, 74.0)
- moved SW201 5.06 mm to (108.5, 74.0)
- turned C402 to 90 degrees
Routing:
- net /SD/DATA_OUT: track 5.19 -> 41.8 mm, vias 1 -> 4
- net Net-(R203-Pad1): track 0.00 -> 22.1 mm, vias 0 -> 2
- net /BOOTLOAD*: track 56.8 -> 35.9 mm
- net Net-(R202-Pad1): track 0.00 -> 18.7 mm, vias 0 -> 2
- net Net-(C401-Pad1): track 24.0 -> 7.24 mm
- net Net-(U201-Pad2): track 0.00 -> 15.1 mm, vias 0 -> 3
- net /Power/+VBUS: track 6.35 -> 16.6 mm, vias 0 -> 2
- net Net-(U201-Pad3): track 0.00 -> 10.0 mm, vias 0 -> 2
- net /GPS_ENABLE*: track 0.00 -> 9.73 mm, vias 0 -> 2
- net Net-(L401-Pad2): track 0.00 -> 6.52 mm
- net /ESP32_RESET*: track 49.0 -> 43.6 mm
- net +3V3: track 15.6 -> 20.4 mm, vias 6 -> 10
- net Net-(Q201-Pad1): track 0.00 -> 4.41 mm, vias 0 -> 2
- net GND: track 90.6 -> 86.4 mm, vias 24 -> 22
- net Net-(Q201-Pad2): track 4.75 -> 7.75 mm
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
Commit message: Fix up digital connections - not done
Parts:
- removed J1101: CONN_02X05, paddle:header-0.050-10-pin-through-hole
- removed R1105, R1106, R1107, R1108: 10k 0.1%, paddle:R_0805
- removed TP1201: AN1, paddle:tp_th_1mm
- removed U802: LTC2440, paddle:VSSOP10-S-PDSO-G10
- added C1001: 0.01uF, paddle:SMD_0805, F.Cu at (234.7, 101.2)
- added C1002: 0.1uF, paddle:SMD_0805, F.Cu at (240.7, 100.9)
- added C1003: 0.01uF, paddle:SMD_0805, F.Cu at (234.7, 106.9)
- added C1004: 1uF, paddle:SMD_0805, F.Cu at (246.4, 94.0)
- added C1005: 0.1uF, paddle:SMD_0805, F.Cu at (246.4, 99.7)
- added C1006: 10uF, paddle:SMD_1206, F.Cu at (241.1, 94.6)
- added C1101: 0.01uF, paddle:SMD_0805, F.Cu at (288.5, 71.1)
- added C1102: 0.1uF, paddle:SMD_0805, F.Cu at (278.0, 83.3)
- added C1103: 0.01uF, paddle:SMD_0805, F.Cu at (283.2, 82.5)
- added C1104: 1uF, paddle:SMD_0805, F.Cu at (288.4, 76.8)
- added C1105: 0.1uF, paddle:SMD_0805, F.Cu at (278.0, 77.6)
- added C1106: 10uF, paddle:SMD_1206, F.Cu at (272.3, 71.7)
- added C1201: 0.01uF, paddle:SMD_0805, F.Cu at (325.4, 76.8)
- added C1203: 0.01uF, paddle:SMD_0805, F.Cu at (320.1, 76.8)
- added C1204: 1uF, paddle:SMD_0805, F.Cu at (314.9, 82.5)
- added C1205: 0.1uF, paddle:SMD_0805, F.Cu at (324.6, 71.1)
- added C1206: 10uF, paddle:SMD_1206, F.Cu at (309.1, 71.7)
- added C701: 0.01uF, paddle:SMD_0805, F.Cu at (246.6, 76.8)
- added C702: 0.1uF, paddle:SMD_0805, F.Cu at (255.5, 71.1)
- added C703: 0.01uF, paddle:SMD_0805, F.Cu at (250.7, 71.1)
- added C704: 1uF, paddle:SMD_0805, F.Cu at (242.6, 83.7)
- added C705: 0.1uF, paddle:SMD_0805, F.Cu at (238.3, 83.7)
- added C706: 10uF, paddle:SMD_1206, F.Cu at (241.1, 71.7)
- added C901: 10uF, paddle:SMD_1206, F.Cu at (277.9, 93.7)
- added C902: 1uF, paddle:SMD_0805, F.Cu at (286.9, 93.1)
- added C903: 10uF, paddle:SMD_1206, F.Cu at (272.6, 100.7)
- added C904: 1uF, paddle:SMD_0805, F.Cu at (277.5, 105.7)
- added C905: 0.1uF, paddle:SMD_0805, F.Cu at (281.8, 104.5)
- added J801: CONN_02X05, paddle:header-0.050-10-pin-through-hole, F.Cu at (267.2, 113.6)
- added Q1001: DMG3414U, paddle:SOT-23, F.Cu at (227.9, 103.5)
- added Q1101: DMG3414U, paddle:SOT-23, F.Cu at (266.3, 80.6)
- added Q1201: DMG3414U, paddle:SOT-23, F.Cu at (303.2, 80.6)
- added Q701: DMG3414U, paddle:SOT-23, F.Cu at (227.9, 80.6)
- added R1001: 10k, paddle:SMD_0805, F.Cu at (239.9, 106.6)
- added R1002: DNP, paddle:SMD_0805, F.Cu at (251.5, 94.0)
- added R1003: 10, paddle:SMD_0805, F.Cu at (251.5, 99.7)
- added R1004: 5k, paddle:SMD_0805, F.Cu at (245.8, 105.4)
- added R1201: 10k, paddle:SMD_0805, F.Cu at (314.9, 76.8)
- added R1202: DNP, paddle:SMD_0805, F.Cu at (319.5, 71.1)
- added R1203: 10, paddle:SMD_0805, F.Cu at (309.8, 78.0)
- added R1204: 5k, paddle:SMD_0805, F.Cu at (314.5, 71.1)
- added R701: 10k, paddle:SMD_0805, F.Cu at (234.1, 78.3)
- added R702: DNP, paddle:SMD_0805, F.Cu at (240.3, 78.0)
- added R703: 10, paddle:SMD_0805, F.Cu at (234.1, 84.0)
- added R704: 5k, paddle:SMD_0805, F.Cu at (246.0, 71.1)
- added R801: 10k 0.1%, paddle:R_0805, F.Cu at (281.5, 118.8)
- added R802: 10k 0.1%, paddle:R_0805, F.Cu at (277.7, 120.9)
- added R803: 10k 0.1%, paddle:R_0805, F.Cu at (281.4, 114.3)
- added R804: 10k 0.1%, paddle:R_0805, F.Cu at (274.0, 120.9)
- added R901: 10k, paddle:SMD_0805, F.Cu at (282.8, 93.1)
- added R902: 10k, paddle:SMD_0805, F.Cu at (277.5, 100.0)
- added R903: 1R0, paddle:SMD_0805, F.Cu at (282.8, 98.8)
- added TP901: VREF, paddle:tp_th_1mm, F.Cu at (291.4, 91.0)
- added U903: OPA333, paddle:sot23-5, F.Cu at (265.2, 94.1)
- R102: value 4.7k -> 10k
- R104: value 10k -> 4.7k
- R1101: value 10k 0.1% -> 10k; footprint paddle:R_0805 -> paddle:SMD_0805
- R1102: value 10k 0.1% -> DNP; footprint paddle:R_0805 -> paddle:SMD_0805
- R1103: value 10k 0.1% -> 10; footprint paddle:R_0805 -> paddle:SMD_0805
- R1104: value 10k 0.1% -> 5k; footprint paddle:R_0805 -> paddle:SMD_0805
- U1002, U702: footprint paddle:VSSOP10-S-PDSO-G10 -> paddle:SSOP-16_3.9x4.9mm_Pitch0.635mm
- U101: value BME280 -> ESP32-WROOM; footprint paddle:BME280 -> paddle:ESP32-WROOM
- U102: value ESP32-WROOM -> BME280; footprint paddle:ESP32-WROOM -> paddle:BME280
- U1101: value SP3003-04 -> OPA388D
- U1102: value SP3003-04 -> LTC2440; footprint paddle:SMD_SC70-6 -> paddle:SSOP-16_3.9x4.9mm_Pitch0.635mm
- U1202: value OPA333 -> LTC2440; footprint paddle:sot23-5 -> paddle:SSOP-16_3.9x4.9mm_Pitch0.635mm
- U801: value OPA388D -> SP3003-04; footprint paddle:S-PDSO-G8 -> paddle:SMD_SC70-6
- U901: value OPA388D -> REF5030; footprint paddle:S-PDSO-G8 -> paddle:TSSOP-8_3x3mm_Pitch0.65mm
- U902: value LTC2440 -> TS5A3160
- moved C1202 167.0 mm to (319.9, 82.5)
- moved U1202 162.4 mm to (302.6, 72.7)
- moved U701 115.8 mm to (234.6, 70.2)
- moved U702 99.5 mm to (227.4, 72.7)
- moved U901 95.4 mm to (271.6, 93.8)
- moved R1102 92.0 mm to (283.3, 71.1)
- moved U1101 87.4 mm to (277.9, 70.0)
- moved R1104 86.2 mm to (283.3, 76.8)
- moved U1102 79.8 mm to (265.8, 72.7)
- moved U902 78.5 mm to (266.0, 100.0)
- moved R1103 73.7 mm to (273.0, 78.0)
- moved R1101 73.1 mm to (273.0, 83.7)
- moved U1001 51.0 mm to (234.6, 93.1)
- moved U1002 43.9 mm to (227.4, 95.6)
- moved U801 37.4 mm to (275.8, 113.8)
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Connections:
- C1202 pad 1: +3.3VA -> GND
- C1202 pad 2: GND -> +3.3VA
- R102 pad 2: /SCK -> /ESP32_RESET*
- R103 pad 2: /SDA -> /SCK
- R104 pad 2: /ESP32_RESET* -> /SDA
- R1101 pad 1: /analog/AUX_IN_0 -> Net-(C1101-Pad2)
- R1101 pad 2: Net-(J1101-Pad3) -> /analog/IN_2
- R1102 pad 1: /analog/AUX_IN_1 -> Net-(C1103-Pad2)
- R1102 pad 2: Net-(J1101-Pad5) -> /analog/VREF
- R1103 pad 1: /analog/AUX_IN_2 -> Net-(C1103-Pad1)
- R1103 pad 2: Net-(J1101-Pad7) -> Net-(C1104-Pad1)
- R1104 pad 1: /analog/AUX_IN_3 -> Net-(C1103-Pad2)
- R1104 pad 2: Net-(J1101-Pad9) -> Net-(C1104-Pad1)
- U1001 pad 2: (no net) -> Net-(C1003-Pad2)
- U1001 pad 3: (no net) -> Net-(C1001-Pad2)
- U1001 pad 4: (no net) -> GND
- U1001 pad 6: (no net) -> Net-(C1003-Pad1)
- U1001 pad 7: (no net) -> +3.3VA
- U1002 pad 1: (no net) -> GND
- U1002 pad 10: (no net) -> GND
- U1002 pad 2: (no net) -> +3.3VA
- U1002 pad 3: (no net) -> /analog/VREF
- U1002 pad 4: (no net) -> GND
- U1002 pad 5: (no net) -> Net-(C1004-Pad1)
- U1002 pad 6: (no net) -> /analog/VREF
- U1002 pad 7: (no net) -> /analog/SDI
- U1002 pad 8: (no net) -> GND
- U1002 pad 9: (no net) -> GND
- U101 pad 3: /SDA -> /ESP32_RESET*
- U101 pad 4: /SCK -> /1PPS
- U101 pad 5: GND -> (no net)
- U101 pad 6: +3V3 -> /ALERT0
- U101 pad 7: GND -> (no net)
- U101 pad 8: +3V3 -> (no net)
- U102 pad 3: /ESP32_RESET* -> /SDA
- U102 pad 4: /1PPS -> /SCK
- U102 pad 5: (no net) -> GND
- U102 pad 6: /ALERT0 -> +3V3
- U102 pad 7: (no net) -> GND
- U102 pad 8: (no net) -> +3V3
- U1101 pad 1: /analog/AUX_IN_3 -> (no net)
- U1101 pad 2: GND -> Net-(C1103-Pad2)
- U1101 pad 3: /analog/AUX_IN_2 -> Net-(C1101-Pad2)
- U1101 pad 4: /analog/AUX_IN_1 -> GND
- U1101 pad 5: +3V3 -> (no net)
- U1101 pad 6: /analog/AUX_IN_0 -> Net-(C1103-Pad1)
- U1102 pad 1: /analog/IN_3 -> GND
- U1102 pad 2: GND -> +3.3VA
- U1102 pad 3: /analog/IN_2 -> /analog/VREF
- U1102 pad 4: /analog/IN_1 -> GND
- U1102 pad 5: +3V3 -> Net-(C1104-Pad1)
- U1102 pad 6: /analog/IN_0 -> /analog/VREF
- U1202 pad 1: /analog/VREF -> GND
- U1202 pad 2: GND -> +3.3VA
- U1202 pad 3: (no net) -> /analog/VREF
- U1202 pad 4: /analog/VREF -> GND
- U1202 pad 5: +3.3VA -> Net-(C1204-Pad1)
- U701 pad 2: (no net) -> Net-(C703-Pad2)
- U701 pad 3: (no net) -> Net-(C701-Pad2)
- U701 pad 4: (no net) -> GND
- U701 pad 6: (no net) -> Net-(C703-Pad1)
- U701 pad 7: (no net) -> +3.3VA
- U702 pad 1: (no net) -> GND
- U702 pad 10: (no net) -> GND
- U702 pad 2: (no net) -> +3.3VA
- U702 pad 3: (no net) -> /analog/VREF
- U702 pad 4: (no net) -> GND
- U702 pad 5: (no net) -> Net-(C704-Pad1)
- U702 pad 6: (no net) -> /analog/VREF
- U702 pad 7: (no net) -> /analog/SDI
- U702 pad 8: (no net) -> GND
- U702 pad 9: (no net) -> GND
- U801 pad 1: (no net) -> /analog/IN_3
- U801 pad 2: (no net) -> GND
- U801 pad 3: (no net) -> /analog/IN_2
- U801 pad 4: (no net) -> /analog/IN_1
- U801 pad 5: (no net) -> +3V3
- U801 pad 6: (no net) -> /analog/IN_0
- U901 pad 2: (no net) -> +3.3VA
- U901 pad 4: (no net) -> GND
- U901 pad 5: (no net) -> Net-(C902-Pad1)
- U901 pad 6: (no net) -> Net-(C904-Pad1)
- U902 pad 1: (no net) -> Net-(C904-Pad1)
- U902 pad 2: (no net) -> GND
- U902 pad 3: (no net) -> Net-(R901-Pad1)
- U902 pad 4: (no net) -> Net-(U902-Pad4)
- U902 pad 5: (no net) -> +3.3VA
Routing:
- net /SCK: track 49.2 -> 0.00 mm, vias 2 -> 0
- net /SDA: track 48.9 -> 1.35 mm, vias 2 -> 0
- net /ESP32_RESET*: track 43.6 -> 0.00 mm
- net (no net): track 0.00 -> 9.73 mm, vias 1 -> 5
- net /ALERT0: track 5.84 -> 0.67 mm
- net GND: track 86.4 -> 81.9 mm, vias 22 -> 20
- net +3V3: track 20.4 -> 16.0 mm, vias 10 -> 8

Commit message: Verify sensor, USB, part of power, add QI charger rectifier
Parts:
- added C801: 0.01uF, paddle:SMD_0805, F.Cu at (196.7, 52.7)
- added LED105: LED, paddle:SMD_D_0805, F.Cu at (207.6, 80.6)
- added LED106: LED, paddle:SMD_D_0805, F.Cu at (207.6, 74.9)
- added R109: 330, paddle:SMD_0805, F.Cu at (216.7, 74.9)
- added R110: 330, paddle:SMD_0805, F.Cu at (212.5, 74.9)
- added U1201: OPA388D, paddle:S-PDSO-G8, F.Cu at (30.2, 284.9)
- C101: value 1.0uF -> 1uF
- R901, R902: value 10k -> 20k 0.1%
- U1101: footprint paddle:SMD_SC70-6 -> paddle:S-PDSO-G8
- moved C902 112.9 mm to (177.5, 65.4)
- moved R901 112.8 mm to (177.5, 52.7)
- moved R1003 111.9 mm to (140.2, 88.6)
- moved C905 107.5 mm to (181.7, 65.4)
- moved R1002 105.8 mm to (146.4, 82.5)
- moved R1104 105.2 mm to (178.6, 87.5)
- moved C702 104.6 mm to (151.7, 58.4)
- moved R1202 104.4 mm to (215.8, 59.6)
- moved R902 104.2 mm to (184.7, 52.7)
- moved R801 103.1 mm to (179.6, 102.9)
- moved U902 102.7 mm to (171.6, 59.5)
- moved U903 102.7 mm to (170.8, 53.7)
- moved R1001 102.5 mm to (140.2, 82.9)
- moved R903 102.5 mm to (186.0, 65.3)
- moved R702 102.2 mm to (139.7, 59.9)
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Connections:
- net /+3.3VA_ENABLE renamed /ENABLE_+3.3VA
- net /ESP32_RESET* renamed /RESET_ESP*
- net /GPS_ENABLE* renamed /ENABLE_GPS*
- net /GPS_RXD renamed /TXD_GPS
- net /GPS_TXD renamed /RXD_GPS
- net /SCK renamed /SCK_I2C
- net /SD/CS renamed /CS_SD*
- net /SD/DATA_OUT renamed /SDI_SPI
- net /SDA renamed /SDA_I2C
- M501 pad 3: /SD/DATA_IN -> /SDO_SPI
- M501 pad 5: /SD/SCLK -> /SCLK_SPI
- Q1001 pad 3: /analog/BUSY* -> /BUSY*
- Q1101 pad 3: /analog/BUSY* -> /BUSY*
- Q1201 pad 3: /analog/BUSY* -> /BUSY*
- Q701 pad 3: /analog/BUSY* -> /BUSY*
- R101 pad 2: /ALERT0 -> /BUSY*
- R306 pad 2: /Power/SHUTDOWN -> /SHUTDOWN*
- SW301 pad 3: /Power/SHUTDOWN -> /SHUTDOWN*
- TP201 pad 1: /TXD -> /TXD_CON
- TP202 pad 1: /RXD -> /RXD_CON
- U1002 pad 12: /analog/SDO -> /SDO_SPI
- U1002 pad 13: /analog/SCLK -> /SCLK_SPI
- U1002 pad 7: /analog/SDI -> /SDO_SPI
- U101 pad 11: (no net) -> /BLINK
- U101 pad 26: (no net) -> /KEEPALIVE
- U101 pad 30: /SD/SCLK -> /SCLK_SPI
- U101 pad 34: /TXD -> /RXD_CON
- U101 pad 35: /RXD -> /TXD_CON
- U101 pad 37: /SD/DATA_IN -> /SDO_SPI
- U101 pad 5: (no net) -> /BUSY*
- U101 pad 6: /ALERT0 -> (no net)
- U101 pad 7: (no net) -> /SHUTDOWN*
- U103 pad 11: /SD_ENABLE* -> (no net)
- U103 pad 12: /KEEPALIVE -> (no net)
- U1102 pad 12: /analog/SDO -> /SDO_SPI
- U1102 pad 13: /analog/SCLK -> /SCLK_SPI
- U1102 pad 7: /analog/SDI -> /SDO_SPI
- U1202 pad 12: /analog/SDO -> /SDO_SPI
- U1202 pad 13: /analog/SCLK -> /SCLK_SPI
- U1202 pad 7: /analog/SDI -> /SDO_SPI
- U203 pad 20: /TXD -> /TXD_CON
- U203 pad 21: /RXD -> /RXD_CON
- U702 pad 12: /analog/SDO -> /SDO_SPI
- U702 pad 13: /analog/SCLK -> /SCLK_SPI
- U702 pad 7: /analog/SDI -> /SDO_SPI
Routing:
- net /SDO_SPI: track 0.00 -> 46.3 mm, vias 0 -> 2
- net /SD/DATA_IN: track 46.3 -> 0.00 mm, vias 2 -> 0
- net /SD/SCLK: track 39.0 -> 0.00 mm, vias 4 -> 0
- net /SCLK_SPI: track 0.00 -> 39.0 mm, vias 0 -> 4
- net /TXD: track 37.4 -> 0.00 mm, vias 2 -> 0
- net (no net): track 9.73 -> 0.00 mm, vias 5 -> 1
- net /RXD_CON: track 0.00 -> 8.73 mm, vias 0 -> 2
- net /RXD: track 8.73 -> 0.00 mm, vias 2 -> 0
- net GND: track 81.9 -> 86.4 mm, vias 20 -> 22
- net +3V3: track 16.0 -> 20.4 mm, vias 8 -> 10
- net /SDA_I2C: track 1.35 -> 2.10 mm
- net /BUSY*: track 0.00 -> 0.67 mm
- net /ALERT0: track 0.67 -> 0.00 mm

Commit message: Start fix up of analog inputs and input+/-/ref tracking, amp model
Parts:
- added C104: 0.1uF, paddle:SMD_0805, F.Cu at (380.6, 97.8)
- added J201: V_QI, paddle:TH_1.0, F.Cu at (311.0, 121.9)
- added J202: GND, paddle:TH_1.0, F.Cu at (307.1, 121.9)
- added Q203: DMG3415U, paddle:SOT-23, F.Cu at (301.0, 128.2)
- added Q204: DMG3415U, paddle:SOT-23, F.Cu at (301.0, 121.3)
- added R206: 1.0Meg, paddle:SMD_0805, F.Cu at (315.7, 120.7)
- added R207: 1.0Meg, paddle:SMD_0805, F.Cu at (307.9, 127.7)
- C301, C302: value 10uF -> 4.7uF
- D301, D302: value RB168LAM -> RB168LAM-30
- F301: footprint paddle:radial-0.2-in-0.7mm-hole -> paddle:SMD_1812
- R304: value 4.7K -> 10K
- U203: value CP2104 -> CP2102N
- U301: value MCP73831/2 -> MCP73832
- moved U1201 379.9 mm to (346.2, 73.9)
- moved C704 260.9 mm to (403.9, 86.2)
- moved R703 260.9 mm to (400.1, 80.5)
- moved R702 257.3 mm to (395.6, 86.2)
- moved R701 255.3 mm to (399.8, 86.2)
- moved Q701 245.4 mm to (377.9, 84.3)
- moved U701 245.4 mm to (384.6, 73.9)
- moved C703 245.4 mm to (401.0, 74.8)
- moved C706 245.4 mm to (391.1, 75.4)
- moved U702 245.4 mm to (377.4, 76.4)
- moved C702 245.0 mm to (396.1, 74.8)
- moved R704 236.3 mm to (396.0, 80.5)
- moved C701 235.5 mm to (390.9, 81.7)
- moved C705 234.4 mm to (384.2, 82.0)
- moved C601 207.1 mm to (353.7, 120.6)
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Connections:
- C301 pad 1: /Power/+VBUS -> /Power/+V_CHARGE
- D301 pad 1: /Power/+VBUS -> /Power/+V_CHARGE
- Q303 pad 1: /Power/+VBUS -> /Power/+V_CHARGE
- R301 pad 1: /Power/+VBUS -> /Power/+V_CHARGE
- R305 pad 2: /Power/+VBUS -> /Power/+V_CHARGE
- U301 pad 4: /Power/+VBUS -> /Power/+V_CHARGE
Routing:
- net /Power/+V_CHARGE: track 0.00 -> 6.35 mm
- net /Power/+VBUS: track 16.6 -> 10.2 mm
