File: kicad/analog/analog.sch (KiCad schematic (older format))
At the start: 6 parts, among them U601 NCP694-3.3

Commit message: checkpoint
Parts:
- gave numbers to parts that had none: 1
- renumbered C601 to C101, C602 to C102, D601 to D101, R601 to R101, U601 to U101
Changed lines of the file:
@@
 LIBS:paddle
 LIBS:analog-cache
-LIBS:processor-cache
 EELAYER 25 0
 EELAYER END
@@
 S 1050 1300 850  1350
 U 59CF67CB
-F0 "sheet59CF67C1" 60
+F0 "input" 60
 F1 "input.sch" 60
 F2 "IN_0" I R 1900 1450 60
@@
 VREF
 $Comp
-L C_Small C601
+L C_Small C101
 U 1 1 59CFCD12
 P 7750 3650
-F 0 "C601" H 7760 3720 50  0000 L CNN
+F 0 "C101" H 7760 3720 50  0000 L CNN
 F 1 "10uF" H 7760 3570 50  0000 L CNN
 F 2 "paddle:SMD_1206" H 7750 3650 50  0001 C CNN
@@
 $EndComp
 $Comp
-L GND #PWR501
+L GND #PWR101
 U 1 1 59CFCD19
 P 7750 3800
-F 0 "#PWR501" H 7750 3550 50  0001 C CNN
+F 0 "#PWR101" H 7750 3550 50  0001 C CNN
 F 1 "GND" H 7750 3650 50  0000 C CNN
 F 2 "" H 7750 3800 50  0001 C CNN
@@
 $EndComp
 $Comp
-L GND #PWR503
+L GND #PWR103
 U 1 1 59CFCD24
 P 8150 4100
-F 0 "#PWR503" H 8150 3850 50  0001 C CNN
+F 0 "#PWR103" H 8150 3850 50  0001 C CNN
 F 1 "GND" H 8150 3950 50  0000 C CNN
 F 2 "" H 8150 4100 50  0001 C CNN
@@
 $EndComp
 $Comp
-L C_Small C602
+L C_Small C102
 U 1 1 59CFCD2C
 P 9450 3650
-F 0 "C602" H 9460 3720 50  0000 L CNN
+F 0 "C102" H 9460 3720 50  0000 L CNN
 F 1 "10uF" H 9460 3570 50  0000 L CNN
 F 2 "paddle:SMD_1206" H 9450 3650 50  0001 C CNN
@@
 $EndComp
 $Comp
-L GND #PWR504
+L GND #PWR105
 U 1 1 59CFCD33
 P 9450 3800
-F 0 "#PWR504" H 9450 3550 50  0001 C CNN
+F 0 "#PWR105" H 9450 3550 50  0001 C CNN
 F 1 "GND" H 9450 3650 50  0000 C CNN
 F 2 "" H 9450 3800 50  0001 C CNN
@@
 $EndComp
 $Comp
-L NCP694-3.3 U601
+L NCP694-3.3 U101
 U 1 1 59CFCD3E
 P 8800 3650
-F 0 "U601" H 8750 3150 60  0000 L CNN
+F 0 "U101" H 8750 3150 60  0000 L CNN
 F 1 "NCP694-3.3" H 8500 3050 60  0000 L CNN
 F 2 "paddle:SOT89-5" H 8900 3550 30  0001 L CNN
@@
 +3.3VA_ENABLE
 $Comp
-L R_US R601
+L R_US R101
 U 1 1 59CFCD48
 P 8000 4750
-F 0 "R601" H 8025 4850 60  0000 C CNN
+F 0 "R101" H 8025 4850 60  0000 C CNN
 F 1 "100k" H 7950 4650 60  0000 C CNN
 F 2 "paddle:SMD_0805" H 8000 4400 60  0001 C CNN
@@
 $EndComp
 $Comp
-L GND #PWR502
+L GND #PWR102
 U 1 1 59CFCD50
 P 8000 5050
-F 0 "#PWR502" H 8000 4800 50  0001 C CNN
+F 0 "#PWR102" H 8000 4800 50  0001 C CNN
 F 1 "GND" H 8000 4900 50  0000 C CNN
 F 2 "" H 8000 5050 50  0001 C CNN
@@
 +V_UNREG_SW
 $Comp
-L +3.3VA #PWR505
+L +3.3VA #PWR106
 U 1 1 59D18927
 P 9950 3450
-F 0 "#PWR505" H 9950 3250 50  0001 C CNN
+F 0 "#PWR106" H 9950 3250 50  0001 C CNN
 F 1 "+3.3VA" H 9950 3650 50  0000 C CNN
 F 2 "" H 9950 3450 50  0001 C CNN
@@
 $EndComp
 $Comp
-L Schottky D601
+L Schottky D101
 U 1 1 59D18A85
 P 8800 3150
-F 0 "D601" H 8800 3250 50  0000 C CNN
+F 0 "D101" H 8800 3250 50  0000 C CNN
 F 1 "RB168LAM" H 8800 3050 50  0000 C CNN
 F 2 "paddle:D_SOD-128" H 8800 2975 50  0001 C CNN
@@
 SDI
 $Comp
-L GND #PWR?
+L GND #PWR104
 U 1 1 59FF8EC4
 P 8250 1450
-F 0 "#PWR?" H 8250 1200 50  0001 C CNN
+F 0 "#PWR104" H 8250 1200 50  0001 C CNN
 F 1 "GND" H 8250 1300 50  0000 C CNN
 F 2 "" H 8250 1450 50  0001 C CNN
@@
 	9550 1900 9650 1900
 $Comp
-L CONN_02X07 J?
+L CONN_02X07 J101
 U 1 1 59FF8EC5
 P 9300 1700
-F 0 "J?" H 9300 2100 50  0000 C CNN
+F 0 "J101" H 9300 2100 50  0000 C CNN
 F 1 "CONN_02X07" V 9300 1700 50  0000 C CNN
 F 2 "" H 9300 500 50  0001 C CNN

Commit message: Update analog board to kicad v4
Parts:
- C101, C102: symbol C_Small -> device:C_Small
- D101: symbol Schottky -> paddle:Schottky
- J101: symbol CONN_02X07 -> paddle:CONN_02X07
- R101: symbol R_US -> paddle:R_US
- U101: symbol NCP694-3.3 -> paddle:NCP694-3.3
Changed lines of the file:
@@
-EESchema Schematic File Version 2
-LIBS:power
-LIBS:device
-LIBS:transistors
-LIBS:conn
-LIBS:linear
-LIBS:regul
-LIBS:paddle
+EESchema Schematic File Version 4
 LIBS:analog-cache
-EELAYER 25 0
+EELAYER 26 0
 EELAYER END
 $Descr A 11000 8500
@@
 VREF
 $Comp
-L C_Small C101
+L device:C_Small C101
 U 1 1 59CFCD12
 P 7750 3650
@@
 $EndComp
 $Comp
-L GND #PWR101
+L power:GND #PWR101
 U 1 1 59CFCD19
 P 7750 3800
@@
 $EndComp
 $Comp
-L GND #PWR103
+L power:GND #PWR103
 U 1 1 59CFCD24
 P 8150 4100
@@
 $EndComp
 $Comp
-L C_Small C102
+L device:C_Small C102
 U 1 1 59CFCD2C
 P 9450 3650
@@
 $EndComp
 $Comp
-L GND #PWR105
+L power:GND #PWR105
 U 1 1 59CFCD33
 P 9450 3800
@@
 $EndComp
 $Comp
-L NCP694-3.3 U101
+L paddle:NCP694-3.3 U101
 U 1 1 59CFCD3E
 P 8800 3650
@@
 +3.3VA_ENABLE
 $Comp
-L R_US R101
+L paddle:R_US R101
 U 1 1 59CFCD48
 P 8000 4750
@@
 $EndComp
 $Comp
-L GND #PWR102
+L power:GND #PWR102
 U 1 1 59CFCD50
 P 8000 5050
@@
 +V_UNREG_SW
 $Comp
-L +3.3VA #PWR106
+L power:+3.3VA #PWR106
 U 1 1 59D18927
 P 9950 3450
@@
 $EndComp
 $Comp
-L Schottky D101
+L paddle:Schottky D101
 U 1 1 59D18A85
 P 8800 3150
@@
 Text Label 5700 3700 0    60   ~ 0
 SDI
-Text HLabel 9950 1500 2    60   Input ~ 0
-SCLK
-Text HLabel 9950 1600 2    60   Output ~ 0
-SDO
-Text HLabel 9950 1700 2    60   Input ~ 0
-SDI
-Text HLabel 9950 1400 2    60   Output ~ 0
-BUSY*
-Text Label 9600 1400 0    60   ~ 0
+Text Label 9700 1200 0    60   ~ 0
 BUSY*
 Text Label 9600 1500 0    60   ~ 0
@@
 SDI
 $Comp
-L GND #PWR104
+L power:GND #PWR104
 U 1 1 59FF8EC4
 P 8250 1450
@@
 Text HLabel 9000 1600 0    60   Input ~ 0
 CS3*
-Text HLabel 9000 1500 0    60   Input ~ 0
-AN_REFSEL
 Wire Wire Line
 	9550 1400 9950 1400
@@
 	9550 1900 9650 1900
 $Comp
-L CONN_02X07 J101
+L paddle:CONN_02X07 J101
 U 1 1 59FF8EC5
 P 9300 1700
@@
 Wire Wire Line
 	9600 2000 9550 2000
+Text Label 8900 1100 2    60   ~ 0
+AN_REFSEL
 $EndSCHEMATC
