File: kicad/analog/analog.sch (KiCad schematic (older format))
At the start: 6 parts, among them J101 CONN_02X07, U101 NCP694-3.3

Commit message: Add ADS1220 A/D
Parts:
- added R101, R102: 10k, paddle:SMD_0805, symbol paddle:R_US
- renumbered R101 to R103
Connections:
- net labels added: BRIDGE_COMP, SPARE
- net labels removed: AN_REFSEL, CS1*, CS2*, CS3*
- wire segments 66 -> 77

Commit message: Switch analog to ADS1220 a/d converter
Parts:
- removed R101, R102: 10k, paddle:SMD_0805, symbol paddle:R_US
- renumbered R103 to R101
Connections:
- net labels added: CS1*, CS2*, CS3*
- wire segments 77 -> 74
Changed lines of the file:
@@
 F1 "reference.sch" 60
 F2 "VREF" O R 1950 4700 60
+F3 "BRIDGE_COMP" O R 1950 4450 50
 $EndSheet
-Text Label 2300 4700 2    60   ~ 0
+Text Label 2100 4700 0    60   ~ 0
 VREF
 $Comp
@@
 $EndComp
 $Comp
-L power:GND #PWR0103
+L power:GND #PWR0101
 U 1 1 59CFCD19
 P 7750 3800
-F 0 "#PWR0103" H 7750 3550 50  0001 C CNN
+F 0 "#PWR0101" H 7750 3550 50  0001 C CNN
 F 1 "GND" H 7750 3650 50  0000 C CNN
 F 2 "" H 7750 3800 50  0001 C CNN
@@
 $EndComp
 $Comp
-L power:GND #PWR0105
+L power:GND #PWR0103
 U 1 1 59CFCD24
 P 8150 4100
-F 0 "#PWR0105" H 8150 3850 50  0001 C CNN
+F 0 "#PWR0103" H 8150 3850 50  0001 C CNN
 F 1 "GND" H 8150 3950 50  0000 C CNN
 F 2 "" H 8150 4100 50  0001 C CNN
@@
 $EndComp
 $Comp
-L power:GND #PWR0107
+L power:GND #PWR0105
 U 1 1 59CFCD33
 P 9450 3800
-F 0 "#PWR0107" H 9450 3550 50  0001 C CNN
+F 0 "#PWR0105" H 9450 3550 50  0001 C CNN
 F 1 "GND" H 9450 3650 50  0000 C CNN
 F 2 "" H 9450 3800 50  0001 C CNN
@@
 +3.3V_AN_ENABLE
 $Comp
-L paddle:R_US R103
+L paddle:R_US R101
 U 1 1 59CFCD48
 P 8000 4750
-F 0 "R103" H 8025 4850 60  0000 C CNN
+F 0 "R101" H 8025 4850 60  0000 C CNN
 F 1 "100k" H 7950 4650 60  0000 C CNN
 F 2 "paddle:SMD_0805" H 8000 4400 60  0001 C CNN
@@
 $EndComp
 $Comp
-L power:GND #PWR0104
+L power:GND #PWR0102
 U 1 1 59CFCD50
 P 8000 5050
-F 0 "#PWR0104" H 8000 4800 50  0001 C CNN
+F 0 "#PWR0102" H 8000 4800 50  0001 C CNN
 F 1 "GND" H 8000 4900 50  0000 C CNN
 F 2 "" H 8000 5050 50  0001 C CNN
@@
 +V_UNREG_SW
 $Comp
-L power:+3.3VA #PWR0108
+L power:+3.3VA #PWR0106
 U 1 1 59D18927
 P 9950 3450
-F 0 "#PWR0108" H 9950 3250 50  0001 C CNN
+F 0 "#PWR0106" H 9950 3250 50  0001 C CNN
 F 1 "+3.3VA" H 9950 3650 50  0000 C CNN
 F 2 "" H 9950 3450 50  0001 C CNN
@@
 SPI_SDI
 $Comp
-L power:GND #PWR0106
+L power:GND #PWR0104
 U 1 1 59FF8EC4
 P 8650 1950
-F 0 "#PWR0106" H 8650 1700 50  0001 C CNN
+F 0 "#PWR0104" H 8650 1700 50  0001 C CNN
 F 1 "GND" H 8650 1800 50  0000 C CNN
 F 2 "" H 8650 1950 50  0001 C CNN
@@
 Connection ~ 8200 3500
 Wire Wire Line
-	1950 4700 2300 4700
+	1950 4700 2100 4700
 Wire Wire Line
 	5550 1900 5700 1900
@@
 Text Label 7950 1450 2    60   ~ 0
 I2C_SCK
-$Comp
-L paddle:R_US R101
-U 1 1 5A9F5198
-P 3250 1100
-F 0 "R101" H 3275 1200 60  0000 C CNN
-F 1 "10k" H 3200 1000 60  0000 C CNN
-F 2 "paddle:SMD_0805" H 3250 750 60  0001 C CNN
-F 3 "" H 3275 1200 60  0000 C CNN
-	1    3250 1100
-	0    -1   -1   0
-$EndComp
-$Comp
-L paddle:R_US R102
-U 1 1 5A9F519F
-P 3250 1750
-F 0 "R102" H 3275 1850 60  0000 C CNN
-F 1 "10k" H 3200 1650 60  0000 C CNN
-F 2 "paddle:SMD_0805" H 3250 1400 60  0001 C CNN
-F 3 "" H 3275 1850 60  0000 C CNN
-	1    3250 1750
-	0    -1   -1   0
-$EndComp
-Wire Wire Line
-	3250 1300 3250 1450
-Wire Wire Line
-	3250 1450 3450 1450
-Wire Wire Line
-	3250 1550 3250 1450
-Connection ~ 3250 1450
-$Comp
-L power:GND #PWR0102
-U 1 1 5A9F51AA
-P 3250 2050
-F 0 "#PWR0102" H 3250 1800 50  0001 C CNN
-F 1 "GND" H 3250 1900 50  0000 C CNN
-F 2 "" H 3250 2050 50  0001 C CNN
-F 3 "" H 3250 2050 50  0001 C CNN
-	1    3250 2050
-	1    0    0    -1
-$EndComp
-Wire Wire Line
-	3250 1950 3250 2050
-$Comp
-L power:+3.3VA #PWR0101
-U 1 1 5A9F51B1
-P 3250 900
-F 0 "#PWR0101" H 3250 700 50  0001 C CNN
-F 1 "+3.3VA" H 3250 1100 50  0000 C CNN
-F 2 "" H 3250 900 50  0001 C CNN
-F 3 "" H 3250 900 50  0001 C CNN
-	1    3250 900
-	1    0    0    -1
-$EndComp
-Text Label 3450 1450 0    50   ~ 0
-BRIDGE_COMP
 Text Label 4550 2050 2    50   ~ 0
 BRIDGE_COMP
@@
 	5550 4050 5700 4050
 Text Label 5700 4050 0    60   ~ 0
-CS0*
+CS1*
 $Sheet
 S 4600 4650 950  1450
@@
 	5550 5900 5700 5900
 Text Label 5700 5900 0    60   ~ 0
-CS0*
+CS2*
 $Sheet
 S 4600 6450 950  1450
@@
 	5550 7700 5700 7700
 Text Label 5700 7700 0    60   ~ 0
-CS0*
+CS3*
 Text Label 8650 1650 0    50   ~ 0
 SPARE
+Text Label 2100 4450 0    50   ~ 0
+BRIDGE_COMP
+Wire Wire Line
+	1950 4450 2100 4450
 $EndSCHEMATC

Commit message: Analog board outline, holes, most footprints, schematic complete
Parts:
- removed J101: CONN_02X07, symbol paddle:CONN_02X07
- added J101: CONN_02X07_1, symbol paddle:CONN_02X07_1
- D101: value RB168LAM -> SS24FL; footprint paddle:D_SOD-128 -> D_SOD-123
Connections:
- net labels added: IN_, PIO_A, PIO_B_BUSY*, SPI_MISO, SPI_MOSI
- net labels removed: BUSY*, CS0*, CS1*, CS2*, CS3*, SCK, SDI, SDO, SPARE, SPI_SDI, SPI_SDO
- wire segments 74 -> 75
- no-connect marks 0 -> 1

Commit message: Fix FCI connector refs, footprints, all packages for analog, starting parts placement
Parts:
- removed J101: CONN_02X07_1, symbol paddle:CONN_02X07_1
- added J101: FCI 20021221-00014T4LF, paddle:conn_FCI_14_NH, symbol paddle:CONN_02X07_0
Other:
- note added: "Note: connector pinout is mirror-image to processor board"
Changed lines of the file:
@@
 Wire Wire Line
 	1950 4450 2100 4450
-$Comp
-L paddle:CONN_02X07_1 J101
-U 1 1 5AA6807C
-P 8300 1650
-F 0 "J101" H 8300 2165 50  0000 C CNN
-F 1 "CONN_02X07_1" H 8300 2074 50  0000 C CNN
-F 2 "" H 8300 450 50  0001 C CNN
-F 3 "" H 8300 450 50  0001 C CNN
-	1    8300 1650
-	1    0    0    -1
-$EndComp
 $Sheet
 S 4600 2800 950  1450
@@
 	1    0    0    -1
 $EndComp
+$Comp
+L paddle:CONN_02X07_0 J101
+U 1 1 5AA83A8D
+P 8300 1650
+F 0 "J101" H 8300 2165 50  0000 C CNN
+F 1 "FCI 20021221-00014T4LF" H 8300 2074 50  0000 C CNN
+F 2 "paddle:conn_FCI_14_NH" H 8300 450 50  0001 C CNN
+F 3 "" H 8300 450 50  0001 C CNN
+	1    8300 1650
+	1    0    0    -1
+$EndComp
+Text Notes 7250 2250 0    50   ~ 0
+Note: connector pinout is mirror-image to processor board
 $EndSCHEMATC

Commit message: Sch: Added bypass caps opamps
Layout: placement and traces for 1 a/d channel ok, connector in right location and pinout (mirror image of processor)
Connections:
- net labels removed: IN_
Other:
- note added: "Note: connector pinout is mirror-image \nto processor board"
- note removed: "Note: connector pinout is mirror-image to processor board"
Changed lines of the file:
@@
 $EndSheet
 Text Label 4550 1250 2    60   ~ 0
-IN_
+IN_0
 Text Label 4550 1650 2    60   ~ 0
 VREF
@@
 $EndSheet
 Text Label 4550 3150 2    60   ~ 0
-IN_
+IN_1
 Text Label 4550 3550 2    60   ~ 0
 VREF
@@
 $EndSheet
 Text Label 4550 5000 2    60   ~ 0
-IN_
+IN_2
 Text Label 4550 5400 2    60   ~ 0
 VREF
@@
 $EndSheet
 Text Label 4550 6800 2    60   ~ 0
-IN_
+IN_3
 Text Label 4550 7200 2    60   ~ 0
 VREF
@@
 	1    0    0    -1
 $EndComp
-Text Notes 7250 2250 0    50   ~ 0
-Note: connector pinout is mirror-image to processor board
+Text Notes 7250 2350 0    50   ~ 0
+Note: connector pinout is mirror-image \nto processor board
 $EndSCHEMATC

Commit message: add bulk caps to analog
Parts:
- added 100uF101, 100uF102: CP, paddle:CP_Radial_D6.3mm_P2.50mm, symbol paddle:CP
Connections:
- wire segments 75 -> 77
Changed lines of the file:
@@
 Connection ~ 7750 3500
 Wire Wire Line
-	7550 3500 7750 3500
+	7250 3500 7400 3500
 Wire Wire Line
 	7750 3500 7950 3500
@@
 Wire Wire Line
 	7950 3500 8200 3500
-Text Label 7550 3500 2    60   ~ 0
+Text Label 7250 3500 2    60   ~ 0
 +V_UNREG_SW
 Text Label 8450 4450 0    60   ~ 0
@@
 Connection ~ 9350 3500
 Wire Wire Line
-	9450 3500 9950 3500
+	9450 3500 9850 3500
 Connection ~ 9450 3500
 $Comp
@@
 Text Notes 7250 2350 0    50   ~ 0
 Note: connector pinout is mirror-image \nto processor board
+$Comp
+L paddle:CP 100uF101
+U 1 1 5AAF46F9
+P 9850 3650
+F 0 "100uF101" H 9968 3696 50  0000 L CNN
+F 1 "CP" H 9968 3605 50  0000 L CNN
+F 2 "paddle:CP_Radial_D6.3mm_P2.50mm" H 9888 3500 50  0001 C CNN
+F 3 "" H 9850 3650 50  0001 C CNN
+	1    9850 3650
+	1    0    0    -1
+$EndComp
+Connection ~ 9850 3500
+Wire Wire Line
+	9850 3500 9950 3500
+$Comp
+L power:GND #PWR0108
+U 1 1 5AAF477B
+P 9850 3800
+F 0 "#PWR0108" H 9850 3550 50  0001 C CNN
+F 1 "GND" H 9855 3627 50  0000 C CNN
+F 2 "" H 9850 3800 50  0001 C CNN
+F 3 "" H 9850 3800 50  0001 C CNN
+	1    9850 3800
+	1    0    0    -1
+$EndComp
+$Comp
+L paddle:CP 100uF102
+U 1 1 5AAF4990
+P 7400 3650
+F 0 "100uF102" H 7518 3696 50  0000 L CNN
+F 1 "CP" H 7518 3605 50  0000 L CNN
+F 2 "paddle:CP_Radial_D6.3mm_P2.50mm" H 7438 3500 50  0001 C CNN
+F 3 "" H 7400 3650 50  0001 C CNN
+	1    7400 3650
+	1    0    0    -1
+$EndComp
+$Comp
+L power:GND #PWR0109
+U 1 1 5AAF4997
+P 7400 3800
+F 0 "#PWR0109" H 7400 3550 50  0001 C CNN
+F 1 "GND" H 7405 3627 50  0000 C CNN
+F 2 "" H 7400 3800 50  0001 C CNN
+F 3 "" H 7400 3800 50  0001 C CNN
+	1    7400 3800
+	1    0    0    -1
+$EndComp
+Connection ~ 7400 3500
+Wire Wire Line
+	7400 3500 7750 3500
 $EndSCHEMATC

Commit message: Analog board and second rev processor board as sent to Goldphoenix
Parts:
- C103: renamed from 100uF102; value CP -> 100uF
- C104: renamed from 100uF101; value CP -> 100uF
Changed lines of the file:
@@
 	9350 3500 9450 3500
 Connection ~ 9350 3500
-Wire Wire Line
-	9450 3500 9850 3500
 Connection ~ 9450 3500
 $Comp
@@
 Note: connector pinout is mirror-image \nto processor board
 $Comp
-L paddle:CP 100uF101
+L paddle:CP C104
 U 1 1 5AAF46F9
 P 9850 3650
-F 0 "100uF101" H 9968 3696 50  0000 L CNN
-F 1 "CP" H 9968 3605 50  0000 L CNN
+F 0 "C104" H 9968 3696 50  0000 L CNN
+F 1 "100uF" H 9968 3605 50  0000 L CNN
 F 2 "paddle:CP_Radial_D6.3mm_P2.50mm" H 9888 3500 50  0001 C CNN
 F 3 "" H 9850 3650 50  0001 C CNN
@@
 	1    0    0    -1
 $EndComp
-Connection ~ 9850 3500
-Wire Wire Line
-	9850 3500 9950 3500
 $Comp
 L power:GND #PWR0108
@@
 $EndComp
 $Comp
-L paddle:CP 100uF102
+L paddle:CP C103
 U 1 1 5AAF4990
 P 7400 3650
-F 0 "100uF102" H 7518 3696 50  0000 L CNN
-F 1 "CP" H 7518 3605 50  0000 L CNN
+F 0 "C103" H 7518 3696 50  0000 L CNN
+F 1 "100uF" H 7518 3605 50  0000 L CNN
 F 2 "paddle:CP_Radial_D6.3mm_P2.50mm" H 7438 3500 50  0001 C CNN
 F 3 "" H 7400 3650 50  0001 C CNN
@@
 Wire Wire Line
 	7400 3500 7750 3500
+Connection ~ 9850 3500
+Wire Wire Line
+	9850 3500 9950 3500
+Wire Wire Line
+	9450 3500 9850 3500
 $EndSCHEMATC
