File: kicad/analog/amp_ad.sch (KiCad schematic (older format))
At the start: 12 parts, among them Q701 DMG3414U, U702 LTC2440

Commit message: checkpoint
Parts:
- gave numbers to parts that had none: 8
- renumbered C705 to C205, C706 to C206, Q701 to Q201, U702 to U202

Commit message: Update analog board to kicad v4
Parts:
- C201, C202, C203, C204, C205, C206: symbol C_Small -> device:C_Small
- Q201: symbol Q_NMOS_GSD -> device:Q_NMOS_GSD
- R201, R202, R203: symbol R_US -> paddle:R_US
- U201: symbol LTC2052 -> paddle:LTC2052
- U202: symbol LTC2440 -> paddle:LTC2440
Changed lines of the file:
@@
-EESchema Schematic File Version 2
-LIBS:power
-LIBS:device
-LIBS:transistors
-LIBS:conn
-LIBS:linear
-LIBS:regul
-LIBS:paddle
+EESchema Schematic File Version 4
 LIBS:analog-cache
-EELAYER 25 0
+EELAYER 26 0
 EELAYER END
 $Descr A 11000 8500
@@
 $EndDescr
 $Comp
-L GND #PWR212
+L power:GND #PWR212
 U 1 1 59DEB50B
 P 6700 4650
@@
 $EndComp
 $Comp
-L GND #PWR211
+L power:GND #PWR211
 U 1 1 59DEB5C9
 P 6050 3450
@@
 $EndComp
 $Comp
-L GND #PWR214
+L power:GND #PWR214
 U 1 1 59DEB702
 P 7050 4050
@@
 $EndComp
 $Comp
-L GND #PWR213
+L power:GND #PWR213
 U 1 1 59DEC1A6
 P 7050 3200
@@
 CS*
 $Comp
-L Q_NMOS_GSD Q201
+L device:Q_NMOS_GSD Q201
 U 1 1 59DECDAE
 P 8000 3100
@@
 $EndComp
 $Comp
-L GND #PWR215
+L power:GND #PWR215
 U 1 1 59DECF72
 P 8100 3300
@@
 ANALOG_IN
 $Comp
-L +3.3VA #PWR207
+L power:+3.3VA #PWR207
 U 1 1 59DED17B
 P 5700 2550
@@
 $EndComp
 $Comp
-L C_Small C206
+L device:C_Small C206
 U 1 1 59DED524
 P 5900 2700
@@
 $EndComp
 $Comp
-L GND #PWR210
+L power:GND #PWR210
 U 1 1 59DED543
 P 5900 2850
@@
 $EndComp
 $Comp
-L C_Small C205
+L device:C_Small C205
 U 1 1 59DED56F
 P 5700 2700
@@
 $EndComp
 $Comp
-L GND #PWR208
+L power:GND #PWR208
 U 1 1 59DED6A0
 P 5700 2850
@@
 $EndComp
 $Comp
-L LTC2440 U202
+L paddle:LTC2440 U202
 U 1 1 59DEE409
 P 6550 3650
@@
 	4900 3300 6050 3300
 $Comp
-L R_US R203
+L paddle:R_US R203
 U 1 1 59F5CA97
 P 4700 3300
@@
 $EndComp
 $Comp
-L C_Small C204
+L device:C_Small C204
 U 1 1 59F5CA9E
 P 5050 3550
@@
 $EndComp
 $Comp
-L GND #PWR206
+L power:GND #PWR206
 U 1 1 59F5CAA5
 P 5050 3700
@@
 $EndComp
 $Comp
-L GND #PWR201
+L power:GND #PWR201
 U 1 1 59F5CAB9
 P 3050 4200
@@
 $EndComp
 $Comp
-L C_Small C201
+L device:C_Small C201
 U 1 1 59F5CABF
 P 3050 4050
@@
 $EndComp
 $Comp
-L GND #PWR204
+L power:GND #PWR204
 U 1 1 59F5CAC6
 P 3800 4200
@@
 $EndComp
 $Comp
-L R_US R201
+L paddle:R_US R201
 U 1 1 59F5CACC
 P 2550 3800
@@
 $EndComp
 $Comp
-L +3.3VA #PWR203
+L power:+3.3VA #PWR203
 U 1 1 59F5CAD5
 P 3800 3100
@@
 $EndComp
 $Comp
-L C_Small C202
+L device:C_Small C202
 U 1 1 59F5CADB
 P 3600 3350
@@
 $EndComp
 $Comp
-L GND #PWR202
+L power:GND #PWR202
 U 1 1 59F5CAE2
 P 3600 3500
@@
 $EndComp
 $Comp
-L LTC2052 U201
+L paddle:LTC2052 U201
 U 1 1 59F5CAE8
 P 3800 3900
@@
 	4750 3900 5450 3900
 $Comp
-L R_US R202
+L paddle:R_US R202
 U 1 1 59F675EB
 P 4550 3900
@@
 $EndComp
 $Comp
-L C_Small C203
+L device:C_Small C203
 U 1 1 59F675F1
 P 4900 4150
@@
 $EndComp
 $Comp
-L GND #PWR205
+L power:GND #PWR205
 U 1 1 59F675F7
 P 4900 4300
@@
 	6050 3900 5700 3900
 $Comp
-L GND #PWR209
+L power:GND #PWR209
 U 1 1 59F93A49
 P 5700 4050

Commit message: Add ADS1220 A/D
Parts:
- removed C202: 0.1uF, paddle:SMD_0805, symbol device:C_Small
- removed R202: 40.2, paddle:SMD_0805, symbol paddle:R_US
- removed U202: LTC2440, paddle:SSOP-16_3.9x4.9mm_Pitch0.635mm, symbol paddle:LTC2440
- added C201: 100pF, paddle:SMD_0805, symbol device:C_Small
- added C?: 0.1uF, paddle:SMD_0805, symbol device:C_Small
- added R201: 1.0k, paddle:SMD_0805, symbol paddle:R_US
- added R203, R204: DNP, paddle:SMD_0805, symbol paddle:R_US
- added unit 1 of U201
- added U?: ADS1220, symbol paddle:ADS1220
- C202: renamed from C201; value 0.001uF -> 100pF
- C203: value 1uF -> 0.1uF
- C207: renamed from C204; value 1uF -> 100pF
- R202: renamed from R201; value 10k -> 1.0k
- R207: renamed from R203; value 40.2 -> 1k
- renumbered C205 to C208, C206 to C209
Connections:
- net labels added: BRIDGE_COMP
- wire segments 40 -> 69

Commit message: Switch analog to ADS1220 a/d converter
Parts:
- removed C201: 100pF, paddle:SMD_0805, symbol device:C_Small
- removed C203: 0.1uF, paddle:SMD_0805, symbol device:C_Small
- removed R201: 1.0k, paddle:SMD_0805, symbol paddle:R_US
- removed R203: DNP, paddle:SMD_0805, symbol paddle:R_US
- removed unit 1 of U201
- R201: renamed from R202; value 1.0k -> 10.0k
- R203: renamed from R207; value 1k -> 10.0k
- gave numbers to parts that had none: 2
- renumbered C202 to C201, C207 to C202, C208 to C203, C209 to C204, R204 to R202
Connections:
- wire segments 69 -> 53

Commit message: Analog board outline, holes, most footprints, schematic complete
Parts:
- removed U202: ADS1220, symbol paddle:ADS1220
- added U201: ADS1220, symbol paddle:ADS1220
- U202: renamed from U201; footprint (none) -> paddle:SO-8_5.3x6.2mm_Pitch1.27mm
- renumbered C203 to C201, C204 to C202, C205 to C203, C202 to C204, C201 to C205, R203 to R201, R201 to R202, R202 to R203

Commit message: Fix FCI connector refs, footprints, all packages for analog, starting parts placement
Parts:
- U201: footprint (none) -> paddle:TSSOP-16-1EP_4.4x5mm_Pitch0.65mm
Changed lines of the file:
@@
 AR Path="/5AA70A0F/59DECDAE" Ref="Q601"  Part="1"
 AR Path="/5AA725C2/59DECDAE" Ref="Q701"  Part="1"
-F 0 "Q201" H 9000 3750 50  0000 L CNN
+F 0 "Q701" H 9000 3750 50  0000 L CNN
 F 1 "DMG3414U" H 9000 3650 50  0000 L CNN
 F 2 "paddle:SOT-23" H 9000 3800 50  0001 C CNN
@@
 AR Path="/5AA70A0F/59DED524" Ref="C602"  Part="1"
 AR Path="/5AA725C2/59DED524" Ref="C702"  Part="1"
-F 0 "C202" H 6410 2670 50  0000 L CNN
+F 0 "C702" H 6410 2670 50  0000 L CNN
 F 1 "10uF" H 6410 2520 50  0000 L CNN
 F 2 "paddle:SMD_1206" H 6400 2600 50  0001 C CNN
@@
 AR Path="/5AA70A0F/59DED56F" Ref="C601"  Part="1"
 AR Path="/5AA725C2/59DED56F" Ref="C701"  Part="1"
-F 0 "C201" H 6210 2670 50  0000 L CNN
+F 0 "C701" H 6210 2670 50  0000 L CNN
 F 1 "0.1uF" H 6210 2520 50  0000 L CNN
 F 2 "paddle:SMD_0805" H 6200 2600 50  0001 C CNN
@@
 AR Path="/5AA70A0F/59F5CA97" Ref="R601"  Part="1"
 AR Path="/5AA725C2/59F5CA97" Ref="R701"  Part="1"
-F 0 "R201" H 5575 3200 60  0000 C CNN
+F 0 "R701" H 5575 3200 60  0000 C CNN
 F 1 "10.0k" H 5500 3000 60  0000 C CNN
 F 2 "paddle:SMD_0805" H 5550 2750 60  0001 C CNN
@@
 AR Path="/5AA70A0F/59F5CA9E" Ref="C604"  Part="1"
 AR Path="/5AA725C2/59F5CA9E" Ref="C704"  Part="1"
-F 0 "C204" H 5910 3320 50  0000 L CNN
+F 0 "C704" H 5910 3320 50  0000 L CNN
 F 1 "100pF" H 5910 3170 50  0000 L CNN
 F 2 "paddle:SMD_0805" H 5900 3250 50  0001 C CNN
@@
 AR Path="/5AA70A0F/59F5CABF" Ref="C605"  Part="1"
 AR Path="/5AA725C2/59F5CABF" Ref="C705"  Part="1"
-F 0 "C205" H 3060 3970 50  0000 L CNN
+F 0 "C705" H 3060 3970 50  0000 L CNN
 F 1 "100pF" H 3060 3820 50  0000 L CNN
 F 2 "paddle:SMD_0805" H 3050 3900 50  0001 C CNN
@@
 AR Path="/5AA70A0F/59F5CACC" Ref="R602"  Part="1"
 AR Path="/5AA725C2/59F5CACC" Ref="R702"  Part="1"
-F 0 "R202" H 2575 3750 60  0000 C CNN
+F 0 "R702" H 2575 3750 60  0000 C CNN
 F 1 "10.0k" H 2500 3550 60  0000 C CNN
 F 2 "paddle:SMD_0805" H 2550 3300 60  0001 C CNN
@@
 $Comp
 L paddle:LTC2052 U202
-U 1 1 59F5CAE8
+U 2 1 59F5CAE8
 P 3800 3750
 AR Path="/59CF60C9/59F5CAE8" Ref="U202"  Part="1"
@@
 AR Path="/5AA70A0F/59F5CAE8" Ref="U602"  Part="1"
 AR Path="/5AA725C2/59F5CAE8" Ref="U602"  Part="2"
-F 0 "U202" H 3800 3950 50  0000 L CNN
+F 0 "U602" H 3800 3950 50  0000 L CNN
 F 1 "LTC2052" H 3800 3550 50  0000 L CNN
 F 2 "paddle:SO-8_5.3x6.2mm_Pitch1.27mm" H 3800 3750 50  0001 C CNN
 F 3 "" H 3800 3750 50  0001 C CNN
-	1    3800 3750
+	2    3800 3750
 	1    0    0    -1
 $EndComp
@@
 AR Path="/5AA70A0F/5A9CCC42" Ref="R603"  Part="1"
 AR Path="/5AA725C2/5A9CCC42" Ref="R703"  Part="1"
-F 0 "R203" H 3625 4750 60  0000 C CNN
+F 0 "R703" H 3625 4750 60  0000 C CNN
 F 1 "DNP" H 3550 4550 60  0000 C CNN
 F 2 "paddle:SMD_0805" H 3600 4300 60  0001 C CNN
@@
 AR Path="/5AA70A0F/5AA1D367" Ref="C603"  Part="1"
 AR Path="/5AA725C2/5AA1D367" Ref="C703"  Part="1"
-F 0 "C203" H 7560 2670 50  0000 L CNN
+F 0 "C703" H 7560 2670 50  0000 L CNN
 F 1 "0.1uF" H 7560 2520 50  0000 L CNN
 F 2 "paddle:SMD_0805" H 7550 2600 50  0001 C CNN
@@
 AR Path="/5AA70A0F/5AA64A6D" Ref="U601"  Part="1"
 AR Path="/5AA725C2/5AA64A6D" Ref="U701"  Part="1"
-F 0 "U201" H 7200 4678 50  0000 C CNN
+F 0 "U701" H 7200 4678 50  0000 C CNN
 F 1 "ADS1220" H 7200 4587 50  0000 C CNN
-F 2 "" H 7850 2700 50  0001 C CNN
+F 2 "paddle:TSSOP-16-1EP_4.4x5mm_Pitch0.65mm" H 7850 2700 50  0001 C CNN
 F 3 "" H 7850 2700 50  0001 C CNN
 	1    7200 3600

Commit message: separate opamps for - input
Parts:
- added C202: 100pF, paddle:SMD_0805, symbol device:C_Small
- added R202: 20.0k, paddle:SMD_0805, symbol paddle:R_US
- added R204: DNP, paddle:SMD_0805, symbol paddle:R_US
- added unit 2 of U201
- U201: renamed from U202; footprint paddle:SO-8_5.3x6.2mm_Pitch1.27mm -> paddle:TSSOP-8_3x3mm_Pitch0.65mm
- renumbered C205 to C201, C204 to C203, C201 to C204, C202 to C205, C203 to C206, R202 to R201, R201 to R205, U201 to U202
Connections:
- wire segments 53 -> 69

Commit message: Sch: Added bypass caps opamps
Layout: placement and traces for 1 a/d channel ok, connector in right location and pinout (mirror image of processor)
Parts:
- added C207: 0.1uF, paddle:SMD_0805, symbol device:C_Small
Connections:
- wire segments 69 -> 72
Changed lines of the file:
@@
 $Descr A 11000 8500
 encoding utf-8
-Sheet 2 7
+Sheet 6 7
 Title ""
 Date ""
@@
 L power:+3.3VA #PWR0203
 U 1 1 5AA635D2
-P 3800 3550
+P 3800 3250
 AR Path="/59CF60C9/5AA635D2" Ref="#PWR0203"  Part="1"
 AR Path="/5AA6CD5B/5AA635D2" Ref="#PWR0503"  Part="1"
 AR Path="/5AA70A0F/5AA635D2" Ref="#PWR0603"  Part="1"
 AR Path="/5AA725C2/5AA635D2" Ref="#PWR0703"  Part="1"
-F 0 "#PWR0203" H 3800 3350 50  0001 C CNN
-F 1 "+3.3VA" H 3800 3750 50  0000 C CNN
-F 2 "" H 3800 3550 50  0001 C CNN
-F 3 "" H 3800 3550 50  0001 C CNN
-	1    3800 3550
+F 0 "#PWR0203" H 3800 3050 50  0001 C CNN
+F 1 "+3.3VA" H 3800 3450 50  0000 C CNN
+F 2 "" H 3800 3250 50  0001 C CNN
+F 3 "" H 3800 3250 50  0001 C CNN
+	1    3800 3250
 	1    0    0    -1
 $EndComp
@@
 	5650 3900 5650 5150
 Connection ~ 4300 5150
+$Comp
+L device:C_Small C207
+U 1 1 5AAC9B85
+P 4200 3400
+AR Path="/59CF60C9/5AAC9B85" Ref="C207"  Part="1"
+AR Path="/5AA6CD5B/5AAC9B85" Ref="C507"  Part="1"
+AR Path="/5AA70A0F/5AAC9B85" Ref="C607"  Part="1"
+AR Path="/5AA725C2/5AAC9B85" Ref="C707"  Part="1"
+F 0 "C207" H 4210 3470 50  0000 L CNN
+F 1 "0.1uF" H 4210 3320 50  0000 L CNN
+F 2 "paddle:SMD_0805" H 4200 3400 50  0001 C CNN
+F 3 "" H 4200 3400 50  0001 C CNN
+	1    4200 3400
+	-1   0    0    1
+$EndComp
+Wire Wire Line
+	3800 3250 3800 3300
+Wire Wire Line
+	4200 3300 3800 3300
+Connection ~ 3800 3300
+Wire Wire Line
+	3800 3300 3800 3550
+$Comp
+L power:GND #PWR0217
+U 1 1 5AACE164
+P 4200 3500
+AR Path="/59CF60C9/5AACE164" Ref="#PWR0217"  Part="1"
+AR Path="/5AA6CD5B/5AACE164" Ref="#PWR0517"  Part="1"
+AR Path="/5AA70A0F/5AACE164" Ref="#PWR0617"  Part="1"
+AR Path="/5AA725C2/5AACE164" Ref="#PWR0717"  Part="1"
+F 0 "#PWR0217" H 4200 3250 50  0001 C CNN
+F 1 "GND" H 4205 3327 50  0000 C CNN
+F 2 "" H 4200 3500 50  0001 C CNN
+F 3 "" H 4200 3500 50  0001 C CNN
+	1    4200 3500
+	1    0    0    -1
+$EndComp
 $EndSCHEMATC
