File: kicad/analog/amp_ad.sch (KiCad schematic (older format))
At the start: 15 parts, among them Q201 DMG3414U, U201 LTC2052, U202 ADS1220

Commit message: analog routed DRC passes
Changed lines of the file:
@@
 AR Path="/5AA70A0F/59DECDAE" Ref="Q601"  Part="1"
 AR Path="/5AA725C2/59DECDAE" Ref="Q701"  Part="1"
-F 0 "Q201" H 9000 3750 50  0000 L CNN
+F 0 "Q501" H 9000 3750 50  0000 L CNN
 F 1 "DMG3414U" H 9000 3650 50  0000 L CNN
 F 2 "paddle:SOT-23" H 9000 3800 50  0001 C CNN
@@
 AR Path="/5AA70A0F/59DED17B" Ref="#PWR0607"  Part="1"
 AR Path="/5AA725C2/59DED17B" Ref="#PWR0707"  Part="1"
-F 0 "#PWR0207" H 6200 2250 50  0001 C CNN
+F 0 "#PWR0707" H 6200 2250 50  0001 C CNN
 F 1 "+3.3VA" H 6200 2650 50  0000 C CNN
 F 2 "" H 6200 2450 50  0001 C CNN
@@
 AR Path="/5AA70A0F/59DED524" Ref="C605"  Part="1"
 AR Path="/5AA725C2/59DED524" Ref="C705"  Part="1"
-F 0 "C205" H 6410 2670 50  0000 L CNN
+F 0 "C505" H 6410 2670 50  0000 L CNN
 F 1 "10uF" H 6410 2520 50  0000 L CNN
 F 2 "paddle:SMD_1206" H 6400 2600 50  0001 C CNN
@@
 AR Path="/5AA70A0F/59DED56F" Ref="C604"  Part="1"
 AR Path="/5AA725C2/59DED56F" Ref="C704"  Part="1"
-F 0 "C204" H 6210 2670 50  0000 L CNN
+F 0 "C504" H 6210 2670 50  0000 L CNN
 F 1 "0.1uF" H 6210 2520 50  0000 L CNN
 F 2 "paddle:SMD_0805" H 6200 2600 50  0001 C CNN
@@
 AR Path="/5AA70A0F/59F5CA97" Ref="R605"  Part="1"
 AR Path="/5AA725C2/59F5CA97" Ref="R705"  Part="1"
-F 0 "R205" H 5575 3200 60  0000 C CNN
+F 0 "R505" H 5575 3200 60  0000 C CNN
 F 1 "10.0k" H 5500 3000 60  0000 C CNN
 F 2 "paddle:SMD_0805" H 5550 2750 60  0001 C CNN
@@
 AR Path="/5AA70A0F/59F5CA9E" Ref="C603"  Part="1"
 AR Path="/5AA725C2/59F5CA9E" Ref="C703"  Part="1"
-F 0 "C203" H 5910 3320 50  0000 L CNN
+F 0 "C503" H 5910 3320 50  0000 L CNN
 F 1 "100pF" H 5910 3170 50  0000 L CNN
 F 2 "paddle:SMD_0805" H 5900 3250 50  0001 C CNN
@@
 AR Path="/5AA70A0F/59F5CABF" Ref="C601"  Part="1"
 AR Path="/5AA725C2/59F5CABF" Ref="C701"  Part="1"
-F 0 "C201" H 3060 3970 50  0000 L CNN
+F 0 "C501" H 3060 3970 50  0000 L CNN
 F 1 "100pF" H 3060 3820 50  0000 L CNN
 F 2 "paddle:SMD_0805" H 3050 3900 50  0001 C CNN
@@
 AR Path="/5AA70A0F/59F5CACC" Ref="R601"  Part="1"
 AR Path="/5AA725C2/59F5CACC" Ref="R701"  Part="1"
-F 0 "R201" H 2575 3750 60  0000 C CNN
+F 0 "R501" H 2575 3750 60  0000 C CNN
 F 1 "10.0k" H 2500 3550 60  0000 C CNN
 F 2 "paddle:SMD_0805" H 2550 3300 60  0001 C CNN
@@
 AR Path="/5AA70A0F/59F5CAE8" Ref="U601"  Part="1"
 AR Path="/5AA725C2/59F5CAE8" Ref="U701"  Part="1"
-F 0 "U201" H 3800 3950 50  0000 L CNN
+F 0 "U501" H 3800 3950 50  0000 L CNN
 F 1 "LTC2052" H 3800 3550 50  0000 L CNN
 F 2 "paddle:TSSOP-8_3x3mm_Pitch0.65mm" H 3800 3750 50  0001 C CNN
@@
 AR Path="/5AA70A0F/5A9CCC42" Ref="R603"  Part="1"
 AR Path="/5AA725C2/5A9CCC42" Ref="R703"  Part="1"
-F 0 "R203" H 3625 4750 60  0000 C CNN
+F 0 "R503" H 3625 4750 60  0000 C CNN
 F 1 "DNP" H 3550 4550 60  0000 C CNN
 F 2 "paddle:SMD_0805" H 3600 4300 60  0001 C CNN
@@
 AR Path="/5AA70A0F/5AA1D367" Ref="C606"  Part="1"
 AR Path="/5AA725C2/5AA1D367" Ref="C706"  Part="1"
-F 0 "C206" H 7560 2670 50  0000 L CNN
+F 0 "C506" H 7560 2670 50  0000 L CNN
 F 1 "0.1uF" H 7560 2520 50  0000 L CNN
 F 2 "paddle:SMD_0805" H 7550 2600 50  0001 C CNN
@@
 AR Path="/5AA70A0F/5AA23513" Ref="#PWR0605"  Part="1"
 AR Path="/5AA725C2/5AA23513" Ref="#PWR0705"  Part="1"
-F 0 "#PWR0205" H 5250 2250 50  0001 C CNN
+F 0 "#PWR0705" H 5250 2250 50  0001 C CNN
 F 1 "+3.3VA" H 5250 2650 50  0000 C CNN
 F 2 "" H 5250 2450 50  0001 C CNN
@@
 AR Path="/5AA70A0F/5AA635D2" Ref="#PWR0603"  Part="1"
 AR Path="/5AA725C2/5AA635D2" Ref="#PWR0703"  Part="1"
-F 0 "#PWR0203" H 3800 3050 50  0001 C CNN
+F 0 "#PWR0703" H 3800 3050 50  0001 C CNN
 F 1 "+3.3VA" H 3800 3450 50  0000 C CNN
 F 2 "" H 3800 3250 50  0001 C CNN
@@
 AR Path="/5AA70A0F/5AA64A6D" Ref="U602"  Part="1"
 AR Path="/5AA725C2/5AA64A6D" Ref="U702"  Part="1"
-F 0 "U202" H 7200 4678 50  0000 C CNN
+F 0 "U502" H 7200 4678 50  0000 C CNN
 F 1 "ADS1220" H 7200 4587 50  0000 C CNN
 F 2 "paddle:TSSOP-16-1EP_4.4x5mm_Pitch0.65mm" H 7850 2700 50  0001 C CNN
@@
 AR Path="/5AA70A0F/5AA868FF" Ref="#PWR0601"  Part="1"
 AR Path="/5AA725C2/5AA868FF" Ref="#PWR0701"  Part="1"
-F 0 "#PWR0201" H 3050 3800 50  0001 C CNN
+F 0 "#PWR0701" H 3050 3800 50  0001 C CNN
 F 1 "GND" H 3055 3877 50  0000 C CNN
 F 2 "" H 3050 4050 50  0001 C CNN
@@
 AR Path="/5AA70A0F/5AA86963" Ref="#PWR0604"  Part="1"
 AR Path="/5AA725C2/5AA86963" Ref="#PWR0704"  Part="1"
-F 0 "#PWR0204" H 3800 3700 50  0001 C CNN
+F 0 "#PWR0704" H 3800 3700 50  0001 C CNN
 F 1 "GND" H 3805 3777 50  0000 C CNN
 F 2 "" H 3800 3950 50  0001 C CNN
@@
 AR Path="/5AA70A0F/5AA869C7" Ref="#PWR0612"  Part="1"
 AR Path="/5AA725C2/5AA869C7" Ref="#PWR0712"  Part="1"
-F 0 "#PWR0212" H 7000 4400 50  0001 C CNN
+F 0 "#PWR0712" H 7000 4400 50  0001 C CNN
 F 1 "GND" H 7005 4477 50  0000 C CNN
 F 2 "" H 7000 4650 50  0001 C CNN
@@
 AR Path="/5AA70A0F/5AA86A0A" Ref="#PWR0613"  Part="1"
 AR Path="/5AA725C2/5AA86A0A" Ref="#PWR0713"  Part="1"
-F 0 "#PWR0213" H 7400 4400 50  0001 C CNN
+F 0 "#PWR0713" H 7400 4400 50  0001 C CNN
 F 1 "GND" H 7405 4477 50  0000 C CNN
 F 2 "" H 7400 4650 50  0001 C CNN
@@
 AR Path="/5AA70A0F/5AA86A8F" Ref="#PWR0615"  Part="1"
 AR Path="/5AA725C2/5AA86A8F" Ref="#PWR0715"  Part="1"
-F 0 "#PWR0215" H 8100 3750 50  0001 C CNN
+F 0 "#PWR0715" H 8100 3750 50  0001 C CNN
 F 1 "GND" H 8105 3827 50  0000 C CNN
 F 2 "" H 8100 4000 50  0001 C CNN
@@
 AR Path="/5AA70A0F/5AA86AC7" Ref="#PWR0616"  Part="1"
 AR Path="/5AA725C2/5AA86AC7" Ref="#PWR0716"  Part="1"
-F 0 "#PWR0216" H 8900 3750 50  0001 C CNN
+F 0 "#PWR0716" H 8900 3750 50  0001 C CNN
 F 1 "GND" H 8905 3827 50  0000 C CNN
 F 2 "" H 8900 4000 50  0001 C CNN
@@
 AR Path="/5AA70A0F/5AA86B4C" Ref="#PWR0608"  Part="1"
 AR Path="/5AA725C2/5AA86B4C" Ref="#PWR0708"  Part="1"
-F 0 "#PWR0208" H 6200 2500 50  0001 C CNN
+F 0 "#PWR0708" H 6200 2500 50  0001 C CNN
 F 1 "GND" H 6205 2577 50  0000 C CNN
 F 2 "" H 6200 2750 50  0001 C CNN
@@
 AR Path="/5AA70A0F/5AA86B84" Ref="#PWR0611"  Part="1"
 AR Path="/5AA725C2/5AA86B84" Ref="#PWR0711"  Part="1"
-F 0 "#PWR0211" H 6400 2500 50  0001 C CNN
+F 0 "#PWR0711" H 6400 2500 50  0001 C CNN
 F 1 "GND" H 6405 2577 50  0000 C CNN
 F 2 "" H 6400 2750 50  0001 C CNN
@@
 AR Path="/5AA70A0F/5AA86BC7" Ref="#PWR0610"  Part="1"
 AR Path="/5AA725C2/5AA86BC7" Ref="#PWR0710"  Part="1"
-F 0 "#PWR0210" H 6300 3000 50  0001 C CNN
+F 0 "#PWR0710" H 6300 3000 50  0001 C CNN
 F 1 "GND" H 6305 3077 50  0000 C CNN
 F 2 "" H 6300 3250 50  0001 C CNN
@@
 AR Path="/5AA70A0F/5AA86C15" Ref="#PWR0606"  Part="1"
 AR Path="/5AA725C2/5AA86C15" Ref="#PWR0706"  Part="1"
-F 0 "#PWR0206" H 5900 3150 50  0001 C CNN
+F 0 "#PWR0706" H 5900 3150 50  0001 C CNN
 F 1 "GND" H 5905 3227 50  0000 C CNN
 F 2 "" H 5900 3400 50  0001 C CNN
@@
 AR Path="/5AA70A0F/5AA86C4D" Ref="#PWR0609"  Part="1"
 AR Path="/5AA725C2/5AA86C4D" Ref="#PWR0709"  Part="1"
-F 0 "#PWR0209" H 6250 3950 50  0001 C CNN
+F 0 "#PWR0709" H 6250 3950 50  0001 C CNN
 F 1 "GND" H 6255 4027 50  0000 C CNN
 F 2 "" H 6250 4200 50  0001 C CNN
@@
 AR Path="/5AA70A0F/5AA86DAD" Ref="#PWR0614"  Part="1"
 AR Path="/5AA725C2/5AA86DAD" Ref="#PWR0714"  Part="1"
-F 0 "#PWR0214" H 7550 2450 50  0001 C CNN
+F 0 "#PWR0714" H 7550 2450 50  0001 C CNN
 F 1 "GND" H 7555 2527 50  0000 C CNN
 F 2 "" H 7550 2700 50  0001 C CNN
@@
 AR Path="/5AA70A0F/5AA8D6EA" Ref="C602"  Part="1"
 AR Path="/5AA725C2/5AA8D6EA" Ref="C702"  Part="1"
-F 0 "C202" H 3060 5370 50  0000 L CNN
+F 0 "C502" H 3060 5370 50  0000 L CNN
 F 1 "100pF" H 3060 5220 50  0000 L CNN
 F 2 "paddle:SMD_0805" H 3050 5300 50  0001 C CNN
@@
 AR Path="/5AA70A0F/5AA8D6F1" Ref="R602"  Part="1"
 AR Path="/5AA725C2/5AA8D6F1" Ref="R702"  Part="1"
-F 0 "R202" H 2575 5150 60  0000 C CNN
+F 0 "R502" H 2575 5150 60  0000 C CNN
 F 1 "20.0k" H 2500 4950 60  0000 C CNN
 F 2 "paddle:SMD_0805" H 2550 4700 60  0001 C CNN
@@
 AR Path="/5AA70A0F/5AA8D6F8" Ref="U601"  Part="2"
 AR Path="/5AA725C2/5AA8D6F8" Ref="U701"  Part="2"
-F 0 "U201" H 3800 5350 50  0000 L CNN
+F 0 "U501" H 3800 5350 50  0000 L CNN
 F 1 "LTC2052" H 3800 4950 50  0000 L CNN
 F 2 "paddle:TSSOP-8_3x3mm_Pitch0.65mm" H 3800 5150 50  0001 C CNN
@@
 AR Path="/5AA70A0F/5AA8D70C" Ref="R604"  Part="1"
 AR Path="/5AA725C2/5AA8D70C" Ref="R704"  Part="1"
-F 0 "R204" H 3625 6150 60  0000 C CNN
+F 0 "R504" H 3625 6150 60  0000 C CNN
 F 1 "DNP" H 3550 5950 60  0000 C CNN
 F 2 "paddle:SMD_0805" H 3600 5700 60  0001 C CNN
@@
 AR Path="/5AA70A0F/5AA8D721" Ref="#PWR0602"  Part="1"
 AR Path="/5AA725C2/5AA8D721" Ref="#PWR0702"  Part="1"
-F 0 "#PWR0202" H 3050 5200 50  0001 C CNN
+F 0 "#PWR0702" H 3050 5200 50  0001 C CNN
 F 1 "GND" H 3055 5277 50  0000 C CNN
 F 2 "" H 3050 5450 50  0001 C CNN
@@
 AR Path="/5AA70A0F/5AAC9B85" Ref="C607"  Part="1"
 AR Path="/5AA725C2/5AAC9B85" Ref="C707"  Part="1"
-F 0 "C207" H 4210 3470 50  0000 L CNN
+F 0 "C507" H 4210 3470 50  0000 L CNN
 F 1 "0.1uF" H 4210 3320 50  0000 L CNN
 F 2 "paddle:SMD_0805" H 4200 3400 50  0001 C CNN
@@
 AR Path="/5AA70A0F/5AACE164" Ref="#PWR0617"  Part="1"
 AR Path="/5AA725C2/5AACE164" Ref="#PWR0717"  Part="1"
-F 0 "#PWR0217" H 4200 3250 50  0001 C CNN
+F 0 "#PWR0717" H 4200 3250 50  0001 C CNN
 F 1 "GND" H 4205 3327 50  0000 C CNN
 F 2 "" H 4200 3500 50  0001 C CNN

Commit message: add bulk caps to analog
Changed lines of the file:
@@
 AR Path="/5AA70A0F/59DECDAE" Ref="Q601"  Part="1"
 AR Path="/5AA725C2/59DECDAE" Ref="Q701"  Part="1"
-F 0 "Q501" H 9000 3750 50  0000 L CNN
+F 0 "Q701" H 9000 3750 50  0000 L CNN
 F 1 "DMG3414U" H 9000 3650 50  0000 L CNN
 F 2 "paddle:SOT-23" H 9000 3800 50  0001 C CNN
@@
 AR Path="/5AA70A0F/59DED524" Ref="C605"  Part="1"
 AR Path="/5AA725C2/59DED524" Ref="C705"  Part="1"
-F 0 "C505" H 6410 2670 50  0000 L CNN
+F 0 "C705" H 6410 2670 50  0000 L CNN
 F 1 "10uF" H 6410 2520 50  0000 L CNN
 F 2 "paddle:SMD_1206" H 6400 2600 50  0001 C CNN
@@
 AR Path="/5AA70A0F/59DED56F" Ref="C604"  Part="1"
 AR Path="/5AA725C2/59DED56F" Ref="C704"  Part="1"
-F 0 "C504" H 6210 2670 50  0000 L CNN
+F 0 "C704" H 6210 2670 50  0000 L CNN
 F 1 "0.1uF" H 6210 2520 50  0000 L CNN
 F 2 "paddle:SMD_0805" H 6200 2600 50  0001 C CNN
@@
 AR Path="/5AA70A0F/59F5CA97" Ref="R605"  Part="1"
 AR Path="/5AA725C2/59F5CA97" Ref="R705"  Part="1"
-F 0 "R505" H 5575 3200 60  0000 C CNN
+F 0 "R705" H 5575 3200 60  0000 C CNN
 F 1 "10.0k" H 5500 3000 60  0000 C CNN
 F 2 "paddle:SMD_0805" H 5550 2750 60  0001 C CNN
@@
 AR Path="/5AA70A0F/59F5CA9E" Ref="C603"  Part="1"
 AR Path="/5AA725C2/59F5CA9E" Ref="C703"  Part="1"
-F 0 "C503" H 5910 3320 50  0000 L CNN
+F 0 "C703" H 5910 3320 50  0000 L CNN
 F 1 "100pF" H 5910 3170 50  0000 L CNN
 F 2 "paddle:SMD_0805" H 5900 3250 50  0001 C CNN
@@
 AR Path="/5AA70A0F/59F5CABF" Ref="C601"  Part="1"
 AR Path="/5AA725C2/59F5CABF" Ref="C701"  Part="1"
-F 0 "C501" H 3060 3970 50  0000 L CNN
+F 0 "C701" H 3060 3970 50  0000 L CNN
 F 1 "100pF" H 3060 3820 50  0000 L CNN
 F 2 "paddle:SMD_0805" H 3050 3900 50  0001 C CNN
@@
 AR Path="/5AA70A0F/59F5CACC" Ref="R601"  Part="1"
 AR Path="/5AA725C2/59F5CACC" Ref="R701"  Part="1"
-F 0 "R501" H 2575 3750 60  0000 C CNN
+F 0 "R701" H 2575 3750 60  0000 C CNN
 F 1 "10.0k" H 2500 3550 60  0000 C CNN
 F 2 "paddle:SMD_0805" H 2550 3300 60  0001 C CNN
@@
 AR Path="/5AA70A0F/59F5CAE8" Ref="U601"  Part="1"
 AR Path="/5AA725C2/59F5CAE8" Ref="U701"  Part="1"
-F 0 "U501" H 3800 3950 50  0000 L CNN
+F 0 "U701" H 3800 3950 50  0000 L CNN
 F 1 "LTC2052" H 3800 3550 50  0000 L CNN
 F 2 "paddle:TSSOP-8_3x3mm_Pitch0.65mm" H 3800 3750 50  0001 C CNN
@@
 AR Path="/5AA70A0F/5A9CCC42" Ref="R603"  Part="1"
 AR Path="/5AA725C2/5A9CCC42" Ref="R703"  Part="1"
-F 0 "R503" H 3625 4750 60  0000 C CNN
+F 0 "R703" H 3625 4750 60  0000 C CNN
 F 1 "DNP" H 3550 4550 60  0000 C CNN
 F 2 "paddle:SMD_0805" H 3600 4300 60  0001 C CNN
@@
 AR Path="/5AA70A0F/5AA1D367" Ref="C606"  Part="1"
 AR Path="/5AA725C2/5AA1D367" Ref="C706"  Part="1"
-F 0 "C506" H 7560 2670 50  0000 L CNN
+F 0 "C706" H 7560 2670 50  0000 L CNN
 F 1 "0.1uF" H 7560 2520 50  0000 L CNN
 F 2 "paddle:SMD_0805" H 7550 2600 50  0001 C CNN
@@
 AR Path="/5AA70A0F/5AA64A6D" Ref="U602"  Part="1"
 AR Path="/5AA725C2/5AA64A6D" Ref="U702"  Part="1"
-F 0 "U502" H 7200 4678 50  0000 C CNN
+F 0 "U702" H 7200 4678 50  0000 C CNN
 F 1 "ADS1220" H 7200 4587 50  0000 C CNN
 F 2 "paddle:TSSOP-16-1EP_4.4x5mm_Pitch0.65mm" H 7850 2700 50  0001 C CNN
@@
 AR Path="/5AA70A0F/5AA8D6EA" Ref="C602"  Part="1"
 AR Path="/5AA725C2/5AA8D6EA" Ref="C702"  Part="1"
-F 0 "C502" H 3060 5370 50  0000 L CNN
+F 0 "C702" H 3060 5370 50  0000 L CNN
 F 1 "100pF" H 3060 5220 50  0000 L CNN
 F 2 "paddle:SMD_0805" H 3050 5300 50  0001 C CNN
@@
 AR Path="/5AA70A0F/5AA8D6F1" Ref="R602"  Part="1"
 AR Path="/5AA725C2/5AA8D6F1" Ref="R702"  Part="1"
-F 0 "R502" H 2575 5150 60  0000 C CNN
+F 0 "R702" H 2575 5150 60  0000 C CNN
 F 1 "20.0k" H 2500 4950 60  0000 C CNN
 F 2 "paddle:SMD_0805" H 2550 4700 60  0001 C CNN
@@
 AR Path="/5AA70A0F/5AA8D6F8" Ref="U601"  Part="2"
 AR Path="/5AA725C2/5AA8D6F8" Ref="U701"  Part="2"
-F 0 "U501" H 3800 5350 50  0000 L CNN
+F 0 "U701" H 3800 5350 50  0000 L CNN
 F 1 "LTC2052" H 3800 4950 50  0000 L CNN
 F 2 "paddle:TSSOP-8_3x3mm_Pitch0.65mm" H 3800 5150 50  0001 C CNN
@@
 AR Path="/5AA70A0F/5AA8D70C" Ref="R604"  Part="1"
 AR Path="/5AA725C2/5AA8D70C" Ref="R704"  Part="1"
-F 0 "R504" H 3625 6150 60  0000 C CNN
+F 0 "R704" H 3625 6150 60  0000 C CNN
 F 1 "DNP" H 3550 5950 60  0000 C CNN
 F 2 "paddle:SMD_0805" H 3600 5700 60  0001 C CNN
@@
 AR Path="/5AA70A0F/5AAC9B85" Ref="C607"  Part="1"
 AR Path="/5AA725C2/5AAC9B85" Ref="C707"  Part="1"
-F 0 "C507" H 4210 3470 50  0000 L CNN
+F 0 "C707" H 4210 3470 50  0000 L CNN
 F 1 "0.1uF" H 4210 3320 50  0000 L CNN
 F 2 "paddle:SMD_0805" H 4200 3400 50  0001 C CNN

Commit message: Analog board and second rev processor board as sent to Goldphoenix
Changed lines of the file:
@@
 AR Path="/5AA70A0F/59DECDAE" Ref="Q601"  Part="1"
 AR Path="/5AA725C2/59DECDAE" Ref="Q701"  Part="1"
-F 0 "Q701" H 9000 3750 50  0000 L CNN
+F 0 "Q201" H 9000 3750 50  0000 L CNN
 F 1 "DMG3414U" H 9000 3650 50  0000 L CNN
 F 2 "paddle:SOT-23" H 9000 3800 50  0001 C CNN
@@
 AR Path="/5AA70A0F/59DED17B" Ref="#PWR0607"  Part="1"
 AR Path="/5AA725C2/59DED17B" Ref="#PWR0707"  Part="1"
-F 0 "#PWR0707" H 6200 2250 50  0001 C CNN
+F 0 "#PWR0207" H 6200 2250 50  0001 C CNN
 F 1 "+3.3VA" H 6200 2650 50  0000 C CNN
 F 2 "" H 6200 2450 50  0001 C CNN
@@
 AR Path="/5AA70A0F/59DED524" Ref="C605"  Part="1"
 AR Path="/5AA725C2/59DED524" Ref="C705"  Part="1"
-F 0 "C705" H 6410 2670 50  0000 L CNN
+F 0 "C205" H 6410 2670 50  0000 L CNN
 F 1 "10uF" H 6410 2520 50  0000 L CNN
 F 2 "paddle:SMD_1206" H 6400 2600 50  0001 C CNN
@@
 AR Path="/5AA70A0F/59DED56F" Ref="C604"  Part="1"
 AR Path="/5AA725C2/59DED56F" Ref="C704"  Part="1"
-F 0 "C704" H 6210 2670 50  0000 L CNN
+F 0 "C204" H 6210 2670 50  0000 L CNN
 F 1 "0.1uF" H 6210 2520 50  0000 L CNN
 F 2 "paddle:SMD_0805" H 6200 2600 50  0001 C CNN
@@
 AR Path="/5AA70A0F/59F5CA97" Ref="R605"  Part="1"
 AR Path="/5AA725C2/59F5CA97" Ref="R705"  Part="1"
-F 0 "R705" H 5575 3200 60  0000 C CNN
+F 0 "R205" H 5575 3200 60  0000 C CNN
 F 1 "10.0k" H 5500 3000 60  0000 C CNN
 F 2 "paddle:SMD_0805" H 5550 2750 60  0001 C CNN
@@
 AR Path="/5AA70A0F/59F5CA9E" Ref="C603"  Part="1"
 AR Path="/5AA725C2/59F5CA9E" Ref="C703"  Part="1"
-F 0 "C703" H 5910 3320 50  0000 L CNN
+F 0 "C203" H 5910 3320 50  0000 L CNN
 F 1 "100pF" H 5910 3170 50  0000 L CNN
 F 2 "paddle:SMD_0805" H 5900 3250 50  0001 C CNN
@@
 AR Path="/5AA70A0F/59F5CABF" Ref="C601"  Part="1"
 AR Path="/5AA725C2/59F5CABF" Ref="C701"  Part="1"
-F 0 "C701" H 3060 3970 50  0000 L CNN
+F 0 "C201" H 3060 3970 50  0000 L CNN
 F 1 "100pF" H 3060 3820 50  0000 L CNN
 F 2 "paddle:SMD_0805" H 3050 3900 50  0001 C CNN
@@
 AR Path="/5AA70A0F/59F5CACC" Ref="R601"  Part="1"
 AR Path="/5AA725C2/59F5CACC" Ref="R701"  Part="1"
-F 0 "R701" H 2575 3750 60  0000 C CNN
+F 0 "R201" H 2575 3750 60  0000 C CNN
 F 1 "10.0k" H 2500 3550 60  0000 C CNN
 F 2 "paddle:SMD_0805" H 2550 3300 60  0001 C CNN
@@
 AR Path="/5AA70A0F/59F5CAE8" Ref="U601"  Part="1"
 AR Path="/5AA725C2/59F5CAE8" Ref="U701"  Part="1"
-F 0 "U701" H 3800 3950 50  0000 L CNN
+F 0 "U201" H 3800 3950 50  0000 L CNN
 F 1 "LTC2052" H 3800 3550 50  0000 L CNN
 F 2 "paddle:TSSOP-8_3x3mm_Pitch0.65mm" H 3800 3750 50  0001 C CNN
@@
 AR Path="/5AA70A0F/5A9CCC42" Ref="R603"  Part="1"
 AR Path="/5AA725C2/5A9CCC42" Ref="R703"  Part="1"
-F 0 "R703" H 3625 4750 60  0000 C CNN
+F 0 "R203" H 3625 4750 60  0000 C CNN
 F 1 "DNP" H 3550 4550 60  0000 C CNN
 F 2 "paddle:SMD_0805" H 3600 4300 60  0001 C CNN
@@
 AR Path="/5AA70A0F/5AA1D367" Ref="C606"  Part="1"
 AR Path="/5AA725C2/5AA1D367" Ref="C706"  Part="1"
-F 0 "C706" H 7560 2670 50  0000 L CNN
+F 0 "C206" H 7560 2670 50  0000 L CNN
 F 1 "0.1uF" H 7560 2520 50  0000 L CNN
 F 2 "paddle:SMD_0805" H 7550 2600 50  0001 C CNN
@@
 AR Path="/5AA70A0F/5AA23513" Ref="#PWR0605"  Part="1"
 AR Path="/5AA725C2/5AA23513" Ref="#PWR0705"  Part="1"
-F 0 "#PWR0705" H 5250 2250 50  0001 C CNN
+F 0 "#PWR0205" H 5250 2250 50  0001 C CNN
 F 1 "+3.3VA" H 5250 2650 50  0000 C CNN
 F 2 "" H 5250 2450 50  0001 C CNN
@@
 AR Path="/5AA70A0F/5AA635D2" Ref="#PWR0603"  Part="1"
 AR Path="/5AA725C2/5AA635D2" Ref="#PWR0703"  Part="1"
-F 0 "#PWR0703" H 3800 3050 50  0001 C CNN
+F 0 "#PWR0203" H 3800 3050 50  0001 C CNN
 F 1 "+3.3VA" H 3800 3450 50  0000 C CNN
 F 2 "" H 3800 3250 50  0001 C CNN
@@
 AR Path="/5AA70A0F/5AA64A6D" Ref="U602"  Part="1"
 AR Path="/5AA725C2/5AA64A6D" Ref="U702"  Part="1"
-F 0 "U702" H 7200 4678 50  0000 C CNN
+F 0 "U202" H 7200 4678 50  0000 C CNN
 F 1 "ADS1220" H 7200 4587 50  0000 C CNN
 F 2 "paddle:TSSOP-16-1EP_4.4x5mm_Pitch0.65mm" H 7850 2700 50  0001 C CNN
@@
 AR Path="/5AA70A0F/5AA868FF" Ref="#PWR0601"  Part="1"
 AR Path="/5AA725C2/5AA868FF" Ref="#PWR0701"  Part="1"
-F 0 "#PWR0701" H 3050 3800 50  0001 C CNN
+F 0 "#PWR0201" H 3050 3800 50  0001 C CNN
 F 1 "GND" H 3055 3877 50  0000 C CNN
 F 2 "" H 3050 4050 50  0001 C CNN
@@
 AR Path="/5AA70A0F/5AA86963" Ref="#PWR0604"  Part="1"
 AR Path="/5AA725C2/5AA86963" Ref="#PWR0704"  Part="1"
-F 0 "#PWR0704" H 3800 3700 50  0001 C CNN
+F 0 "#PWR0204" H 3800 3700 50  0001 C CNN
 F 1 "GND" H 3805 3777 50  0000 C CNN
 F 2 "" H 3800 3950 50  0001 C CNN
@@
 AR Path="/5AA70A0F/5AA869C7" Ref="#PWR0612"  Part="1"
 AR Path="/5AA725C2/5AA869C7" Ref="#PWR0712"  Part="1"
-F 0 "#PWR0712" H 7000 4400 50  0001 C CNN
+F 0 "#PWR0212" H 7000 4400 50  0001 C CNN
 F 1 "GND" H 7005 4477 50  0000 C CNN
 F 2 "" H 7000 4650 50  0001 C CNN
@@
 AR Path="/5AA70A0F/5AA86A0A" Ref="#PWR0613"  Part="1"
 AR Path="/5AA725C2/5AA86A0A" Ref="#PWR0713"  Part="1"
-F 0 "#PWR0713" H 7400 4400 50  0001 C CNN
+F 0 "#PWR0213" H 7400 4400 50  0001 C CNN
 F 1 "GND" H 7405 4477 50  0000 C CNN
 F 2 "" H 7400 4650 50  0001 C CNN
@@
 AR Path="/5AA70A0F/5AA86A8F" Ref="#PWR0615"  Part="1"
 AR Path="/5AA725C2/5AA86A8F" Ref="#PWR0715"  Part="1"
-F 0 "#PWR0715" H 8100 3750 50  0001 C CNN
+F 0 "#PWR0215" H 8100 3750 50  0001 C CNN
 F 1 "GND" H 8105 3827 50  0000 C CNN
 F 2 "" H 8100 4000 50  0001 C CNN
@@
 AR Path="/5AA70A0F/5AA86AC7" Ref="#PWR0616"  Part="1"
 AR Path="/5AA725C2/5AA86AC7" Ref="#PWR0716"  Part="1"
-F 0 "#PWR0716" H 8900 3750 50  0001 C CNN
+F 0 "#PWR0216" H 8900 3750 50  0001 C CNN
 F 1 "GND" H 8905 3827 50  0000 C CNN
 F 2 "" H 8900 4000 50  0001 C CNN
@@
 AR Path="/5AA70A0F/5AA86B4C" Ref="#PWR0608"  Part="1"
 AR Path="/5AA725C2/5AA86B4C" Ref="#PWR0708"  Part="1"
-F 0 "#PWR0708" H 6200 2500 50  0001 C CNN
+F 0 "#PWR0208" H 6200 2500 50  0001 C CNN
 F 1 "GND" H 6205 2577 50  0000 C CNN
 F 2 "" H 6200 2750 50  0001 C CNN
@@
 AR Path="/5AA70A0F/5AA86B84" Ref="#PWR0611"  Part="1"
 AR Path="/5AA725C2/5AA86B84" Ref="#PWR0711"  Part="1"
-F 0 "#PWR0711" H 6400 2500 50  0001 C CNN
+F 0 "#PWR0211" H 6400 2500 50  0001 C CNN
 F 1 "GND" H 6405 2577 50  0000 C CNN
 F 2 "" H 6400 2750 50  0001 C CNN
@@
 AR Path="/5AA70A0F/5AA86BC7" Ref="#PWR0610"  Part="1"
 AR Path="/5AA725C2/5AA86BC7" Ref="#PWR0710"  Part="1"
-F 0 "#PWR0710" H 6300 3000 50  0001 C CNN
+F 0 "#PWR0210" H 6300 3000 50  0001 C CNN
 F 1 "GND" H 6305 3077 50  0000 C CNN
 F 2 "" H 6300 3250 50  0001 C CNN
@@
 AR Path="/5AA70A0F/5AA86C15" Ref="#PWR0606"  Part="1"
 AR Path="/5AA725C2/5AA86C15" Ref="#PWR0706"  Part="1"
-F 0 "#PWR0706" H 5900 3150 50  0001 C CNN
+F 0 "#PWR0206" H 5900 3150 50  0001 C CNN
 F 1 "GND" H 5905 3227 50  0000 C CNN
 F 2 "" H 5900 3400 50  0001 C CNN
@@
 AR Path="/5AA70A0F/5AA86C4D" Ref="#PWR0609"  Part="1"
 AR Path="/5AA725C2/5AA86C4D" Ref="#PWR0709"  Part="1"
-F 0 "#PWR0709" H 6250 3950 50  0001 C CNN
+F 0 "#PWR0209" H 6250 3950 50  0001 C CNN
 F 1 "GND" H 6255 4027 50  0000 C CNN
 F 2 "" H 6250 4200 50  0001 C CNN
@@
 AR Path="/5AA70A0F/5AA86DAD" Ref="#PWR0614"  Part="1"
 AR Path="/5AA725C2/5AA86DAD" Ref="#PWR0714"  Part="1"
-F 0 "#PWR0714" H 7550 2450 50  0001 C CNN
+F 0 "#PWR0214" H 7550 2450 50  0001 C CNN
 F 1 "GND" H 7555 2527 50  0000 C CNN
 F 2 "" H 7550 2700 50  0001 C CNN
@@
 AR Path="/5AA70A0F/5AA8D6EA" Ref="C602"  Part="1"
 AR Path="/5AA725C2/5AA8D6EA" Ref="C702"  Part="1"
-F 0 "C702" H 3060 5370 50  0000 L CNN
+F 0 "C202" H 3060 5370 50  0000 L CNN
 F 1 "100pF" H 3060 5220 50  0000 L CNN
 F 2 "paddle:SMD_0805" H 3050 5300 50  0001 C CNN
@@
 AR Path="/5AA70A0F/5AA8D6F1" Ref="R602"  Part="1"
 AR Path="/5AA725C2/5AA8D6F1" Ref="R702"  Part="1"
-F 0 "R702" H 2575 5150 60  0000 C CNN
+F 0 "R202" H 2575 5150 60  0000 C CNN
 F 1 "20.0k" H 2500 4950 60  0000 C CNN
 F 2 "paddle:SMD_0805" H 2550 4700 60  0001 C CNN
@@
 AR Path="/5AA70A0F/5AA8D6F8" Ref="U601"  Part="2"
 AR Path="/5AA725C2/5AA8D6F8" Ref="U701"  Part="2"
-F 0 "U701" H 3800 5350 50  0000 L CNN
+F 0 "U201" H 3800 5350 50  0000 L CNN
 F 1 "LTC2052" H 3800 4950 50  0000 L CNN
 F 2 "paddle:TSSOP-8_3x3mm_Pitch0.65mm" H 3800 5150 50  0001 C CNN
@@
 AR Path="/5AA70A0F/5AA8D70C" Ref="R604"  Part="1"
 AR Path="/5AA725C2/5AA8D70C" Ref="R704"  Part="1"
-F 0 "R704" H 3625 6150 60  0000 C CNN
+F 0 "R204" H 3625 6150 60  0000 C CNN
 F 1 "DNP" H 3550 5950 60  0000 C CNN
 F 2 "paddle:SMD_0805" H 3600 5700 60  0001 C CNN
@@
 AR Path="/5AA70A0F/5AA8D721" Ref="#PWR0602"  Part="1"
 AR Path="/5AA725C2/5AA8D721" Ref="#PWR0702"  Part="1"
-F 0 "#PWR0702" H 3050 5200 50  0001 C CNN
+F 0 "#PWR0202" H 3050 5200 50  0001 C CNN
 F 1 "GND" H 3055 5277 50  0000 C CNN
 F 2 "" H 3050 5450 50  0001 C CNN
@@
 AR Path="/5AA70A0F/5AAC9B85" Ref="C607"  Part="1"
 AR Path="/5AA725C2/5AAC9B85" Ref="C707"  Part="1"
-F 0 "C707" H 4210 3470 50  0000 L CNN
+F 0 "C207" H 4210 3470 50  0000 L CNN
 F 1 "0.1uF" H 4210 3320 50  0000 L CNN
 F 2 "paddle:SMD_0805" H 4200 3400 50  0001 C CNN
@@
 AR Path="/5AA70A0F/5AACE164" Ref="#PWR0617"  Part="1"
 AR Path="/5AA725C2/5AACE164" Ref="#PWR0717"  Part="1"
-F 0 "#PWR0717" H 4200 3250 50  0001 C CNN
+F 0 "#PWR0217" H 4200 3250 50  0001 C CNN
 F 1 "GND" H 4205 3327 50  0000 C CNN
 F 2 "" H 4200 3500 50  0001 C CNN
