File: kicad/analog/input.sch (KiCad schematic (older format))
At the start: 6 parts, among them J801 CONN_02X05, U801 SP3003-04

Commit message: checkpoint
Parts:
- renumbered J801 to J301, R801 to R301, R802 to R302, R803 to R303, R804 to R304, U801 to U301
Changed lines of the file:
@@
 LIBS:paddle
 LIBS:analog-cache
-LIBS:processor-cache
 EELAYER 25 0
 EELAYER END
@@
 $EndDescr
 $Comp
-L CONN_02X05 J801
+L CONN_02X05 J301
 U 1 1 59CECF11
 P 5300 3050
-F 0 "J801" H 5300 3350 50  0000 C CNN
+F 0 "J301" H 5300 3350 50  0000 C CNN
 F 1 "CONN_02X05" H 5300 2750 50  0000 C CNN
 F 2 "paddle:header-0.050-10-pin-through-hole" H 5300 1850 50  0001 C CNN
@@
 $EndComp
 $Comp
-L +3.3VA #PWR701
+L +3.3VA #PWR301
 U 1 1 59CECF30
 P 4900 2800
-F 0 "#PWR701" H 4900 2600 50  0001 C CNN
+F 0 "#PWR301" H 4900 2600 50  0001 C CNN
 F 1 "+3.3VA" H 4900 3000 50  0000 C CNN
 F 2 "" H 4900 2800 50  0001 C CNN
@@
 $EndComp
 $Comp
-L GND #PWR704
+L GND #PWR304
 U 1 1 59CECF36
 P 5700 3350
-F 0 "#PWR704" H 5700 3100 50  0001 C CNN
+F 0 "#PWR304" H 5700 3100 50  0001 C CNN
 F 1 "GND" H 5700 3200 50  0000 C CNN
 F 2 "" H 5700 3350 50  0001 C CNN
@@
 $EndComp
 $Comp
-L SP3003-04 U801
+L SP3003-04 U301
 U 1 1 59CECF3F
 P 6050 4350
-F 0 "U801" H 5800 4900 60  0000 C CNN
+F 0 "U301" H 5800 4900 60  0000 C CNN
 F 1 "SP3003-04" H 6200 4900 60  0000 C CNN
 F 2 "paddle:SMD_SC70-6" H 6050 3400 60  0001 C CNN
@@
 $EndComp
 $Comp
-L +3.3V #PWR702
+L +3.3V #PWR302
 U 1 1 59CECF46
 P 5450 4050
-F 0 "#PWR702" H 5450 3900 50  0001 C CNN
+F 0 "#PWR302" H 5450 3900 50  0001 C CNN
 F 1 "+3.3V" H 5450 4190 50  0000 C CNN
 F 2 "" H 5450 4050 50  0001 C CNN
@@
 $EndComp
 $Comp
-L GND #PWR703
+L GND #PWR303
 U 1 1 59CECF4C
 P 5450 4600
-F 0 "#PWR703" H 5450 4350 50  0001 C CNN
+F 0 "#PWR303" H 5450 4350 50  0001 C CNN
 F 1 "GND" H 5450 4450 50  0000 C CNN
 F 2 "" H 5450 4600 50  0001 C CNN
@@
 $EndComp
 $Comp
-L R_US R801
+L R_US R301
 U 1 1 59CF0D9D
 P 6050 2850
-F 0 "R801" H 6100 3250 60  0000 C CNN
+F 0 "R301" H 6100 3250 60  0000 C CNN
 F 1 "10k 0.1%" H 6500 3250 60  0000 C CNN
 F 2 "paddle:R_0805" H 6050 2500 60  0001 C CNN
@@
 $EndComp
 $Comp
-L R_US R802
+L R_US R302
 U 1 1 59CF0E0C
 P 6050 2950
-F 0 "R802" H 6100 3350 60  0000 C CNN
+F 0 "R302" H 6100 3350 60  0000 C CNN
 F 1 "10k 0.1%" H 6500 3350 60  0000 C CNN
 F 2 "paddle:R_0805" H 6050 2600 60  0001 C CNN
@@
 $EndComp
 $Comp
-L R_US R803
+L R_US R303
 U 1 1 59CF0E2B
 P 6050 3050
-F 0 "R803" H 6100 3450 60  0000 C CNN
+F 0 "R303" H 6100 3450 60  0000 C CNN
 F 1 "10k 0.1%" H 6500 3450 60  0000 C CNN
 F 2 "paddle:R_0805" H 6050 2700 60  0001 C CNN
@@
 $EndComp
 $Comp
-L R_US R804
+L R_US R304
 U 1 1 59CF0E51
 P 6050 3150
-F 0 "R804" H 6100 3550 60  0000 C CNN
+F 0 "R304" H 6100 3550 60  0000 C CNN
 F 1 "10k 0.1%" H 6500 3550 60  0000 C CNN
 F 2 "paddle:R_0805" H 6050 2800 60  0001 C CNN

Commit message: Update analog board to kicad v4
Parts:
- J301: symbol CONN_02X05 -> analog-rescue:CONN_02X05-RESCUE-analog
- R301, R302, R303, R304: symbol R_US -> paddle:R_US
- U301: symbol SP3003-04 -> paddle:SP3003-04
Changed lines of the file:
@@
-EESchema Schematic File Version 2
-LIBS:power
-LIBS:device
-LIBS:transistors
-LIBS:conn
-LIBS:linear
-LIBS:regul
-LIBS:paddle
+EESchema Schematic File Version 4
 LIBS:analog-cache
-EELAYER 25 0
+EELAYER 26 0
 EELAYER END
 $Descr A4 11693 8268
@@
 $EndDescr
 $Comp
-L CONN_02X05 J301
+L analog-rescue:CONN_02X05-RESCUE-analog J301
 U 1 1 59CECF11
 P 5300 3050
+AR Path="/59CECF11" Ref="J301"  Part="1"
+AR Path="/59CF67CB/59CECF11" Ref="J301"  Part="1"
 F 0 "J301" H 5300 3350 50  0000 C CNN
 F 1 "CONN_02X05" H 5300 2750 50  0000 C CNN
@@
 $EndComp
 $Comp
-L +3.3VA #PWR301
+L power:+3.3VA #PWR301
 U 1 1 59CECF30
 P 4900 2800
@@
 $EndComp
 $Comp
-L GND #PWR304
+L power:GND #PWR304
 U 1 1 59CECF36
 P 5700 3350
@@
 $EndComp
 $Comp
-L SP3003-04 U301
+L paddle:SP3003-04 U301
 U 1 1 59CECF3F
 P 6050 4350
@@
 $EndComp
 $Comp
-L +3.3V #PWR302
+L power:+3.3V #PWR302
 U 1 1 59CECF46
 P 5450 4050
@@
 $EndComp
 $Comp
-L GND #PWR303
+L power:GND #PWR303
 U 1 1 59CECF4C
 P 5450 4600
@@
 $EndComp
 $Comp
-L R_US R301
+L paddle:R_US R301
 U 1 1 59CF0D9D
 P 6050 2850
@@
 $EndComp
 $Comp
-L R_US R302
+L paddle:R_US R302
 U 1 1 59CF0E0C
 P 6050 2950
@@
 $EndComp
 $Comp
-L R_US R303
+L paddle:R_US R303
 U 1 1 59CF0E2B
 P 6050 3050
@@
 $EndComp
 $Comp
-L R_US R304
+L paddle:R_US R304
 U 1 1 59CF0E51
 P 6050 3150

Commit message: Add ADS1220 A/D
Connections:
- wire segments 23 -> 27
Changed lines of the file:
@@
 U 1 1 59CECF11
 P 5300 3050
-AR Path="/59CECF11" Ref="J301"  Part="1"
-AR Path="/59CF67CB/59CECF11" Ref="J301"  Part="1"
 F 0 "J301" H 5300 3350 50  0000 C CNN
 F 1 "CONN_02X05" H 5300 2750 50  0000 C CNN
@@
 $EndComp
 $Comp
-L power:+3.3VA #PWR301
+L power:+3.3VA #PWR0301
 U 1 1 59CECF30
 P 4900 2800
-F 0 "#PWR301" H 4900 2600 50  0001 C CNN
+F 0 "#PWR0301" H 4900 2600 50  0001 C CNN
 F 1 "+3.3VA" H 4900 3000 50  0000 C CNN
 F 2 "" H 4900 2800 50  0001 C CNN
@@
 $EndComp
 $Comp
-L power:GND #PWR304
+L power:GND #PWR0304
 U 1 1 59CECF36
 P 5700 3350
-F 0 "#PWR304" H 5700 3100 50  0001 C CNN
+F 0 "#PWR0304" H 5700 3100 50  0001 C CNN
 F 1 "GND" H 5700 3200 50  0000 C CNN
 F 2 "" H 5700 3350 50  0001 C CNN
@@
 $EndComp
 $Comp
-L power:+3.3V #PWR302
+L power:+3.3V #PWR0302
 U 1 1 59CECF46
 P 5450 4050
-F 0 "#PWR302" H 5450 3900 50  0001 C CNN
+F 0 "#PWR0302" H 5450 3900 50  0001 C CNN
 F 1 "+3.3V" H 5450 4190 50  0000 C CNN
 F 2 "" H 5450 4050 50  0001 C CNN
@@
 $EndComp
 $Comp
-L power:GND #PWR303
+L power:GND #PWR0303
 U 1 1 59CECF4C
 P 5450 4600
-F 0 "#PWR303" H 5450 4350 50  0001 C CNN
+F 0 "#PWR0303" H 5450 4350 50  0001 C CNN
 F 1 "GND" H 5450 4450 50  0000 C CNN
 F 2 "" H 5450 4600 50  0001 C CNN
@@
 	6550 4650 7350 4650
 Wire Wire Line
-	6250 2850 7800 2850
+	6250 2850 6900 2850
 Wire Wire Line
-	6250 2950 7800 2950
+	6250 2950 7050 2950
 Wire Wire Line
-	6250 3050 7800 3050
+	6250 3050 7200 3050
 Wire Wire Line
-	6250 3150 7800 3150
+	6250 3150 7350 3150
 Wire Wire Line
 	6900 4050 6900 2850
@@
 NoConn ~ 5050 3150
 NoConn ~ 5050 3250
+Wire Wire Line
+	6900 2850 7800 2850
+Wire Wire Line
+	7050 2950 7800 2950
+Wire Wire Line
+	7200 3050 7800 3050
+Wire Wire Line
+	7350 3150 7800 3150
 $EndSCHEMATC

Commit message: Switch analog to ADS1220 a/d converter
Parts:
- R301, R302, R303, R304: value 10k 0.1% -> 10.0k 0.1%
Changed lines of the file:
@@
 P 6050 2850
 F 0 "R301" H 6100 3250 60  0000 C CNN
-F 1 "10k 0.1%" H 6500 3250 60  0000 C CNN
+F 1 "10.0k 0.1%" H 6500 3250 60  0000 C CNN
 F 2 "paddle:R_0805" H 6050 2500 60  0001 C CNN
 F 3 "" H 6075 2950 60  0000 C CNN
@@
 P 6050 2950
 F 0 "R302" H 6100 3350 60  0000 C CNN
-F 1 "10k 0.1%" H 6500 3350 60  0000 C CNN
+F 1 "10.0k 0.1%" H 6500 3350 60  0000 C CNN
 F 2 "paddle:R_0805" H 6050 2600 60  0001 C CNN
 F 3 "" H 6075 3050 60  0000 C CNN
@@
 P 6050 3050
 F 0 "R303" H 6100 3450 60  0000 C CNN
-F 1 "10k 0.1%" H 6500 3450 60  0000 C CNN
+F 1 "10.0k 0.1%" H 6500 3450 60  0000 C CNN
 F 2 "paddle:R_0805" H 6050 2700 60  0001 C CNN
 F 3 "" H 6075 3150 60  0000 C CNN
@@
 P 6050 3150
 F 0 "R304" H 6100 3550 60  0000 C CNN
-F 1 "10k 0.1%" H 6500 3550 60  0000 C CNN
+F 1 "10.0k 0.1%" H 6500 3550 60  0000 C CNN
 F 2 "paddle:R_0805" H 6050 2800 60  0001 C CNN
 F 3 "" H 6075 3250 60  0000 C CNN

Commit message: Analog board outline, holes, most footprints, schematic complete
Connections:
- net labels removed: +3.3V
Changed lines of the file:
@@
 $EndComp
 $Comp
-L power:GND #PWR0304
+L power:GND #PWR0302
 U 1 1 59CECF36
 P 5700 3350
-F 0 "#PWR0304" H 5700 3100 50  0001 C CNN
+F 0 "#PWR0302" H 5700 3100 50  0001 C CNN
 F 1 "GND" H 5700 3200 50  0000 C CNN
 F 2 "" H 5700 3350 50  0001 C CNN
@@
 $EndComp
 $Comp
-L power:+3.3V #PWR0302
-U 1 1 59CECF46
-P 5450 4050
-F 0 "#PWR0302" H 5450 3900 50  0001 C CNN
-F 1 "+3.3V" H 5450 4190 50  0000 C CNN
-F 2 "" H 5450 4050 50  0001 C CNN
-F 3 "" H 5450 4050 50  0001 C CNN
-	1    5450 4050
-	1    0    0    -1
-$EndComp
-$Comp
-L power:GND #PWR0303
+L power:GND #PWR0304
 U 1 1 59CECF4C
 P 5450 4600
-F 0 "#PWR0303" H 5450 4350 50  0001 C CNN
+F 0 "#PWR0304" H 5450 4350 50  0001 C CNN
 F 1 "GND" H 5450 4450 50  0000 C CNN
 F 2 "" H 5450 4600 50  0001 C CNN
@@
 	5700 3250 5700 3350
 Wire Wire Line
-	5550 4150 5450 4150
-Wire Wire Line
-	5450 4150 5450 4050
-Wire Wire Line
 	5550 4600 5450 4600
 Wire Wire Line
@@
 Wire Wire Line
 	7350 3150 7800 3150
+Wire Wire Line
+	5400 4150 5550 4150
+$Comp
+L power:+3.3VA #PWR0160
+U 1 1 5AA899F3
+P 5400 4050
+F 0 "#PWR0160" H 5400 3850 50  0001 C CNN
+F 1 "+3.3VA" H 5400 4250 50  0000 C CNN
+F 2 "" H 5400 4050 50  0001 C CNN
+F 3 "" H 5400 4050 50  0001 C CNN
+	1    5400 4050
+	1    0    0    -1
+$EndComp
+Wire Wire Line
+	5400 4050 5400 4150
 $EndSCHEMATC

Commit message: analog routed DRC passes
Changed lines of the file:
@@
 Wire Wire Line
 	6550 4650 7350 4650
-Wire Wire Line
-	6250 2850 6900 2850
-Wire Wire Line
-	6250 2950 7050 2950
-Wire Wire Line
-	6250 3050 7200 3050
-Wire Wire Line
-	6250 3150 7350 3150
-Wire Wire Line
-	6900 4050 6900 2850
-Connection ~ 6900 2850
-Wire Wire Line
-	7050 4250 7050 2950
-Connection ~ 7050 2950
-Wire Wire Line
-	7200 4450 7200 3050
-Connection ~ 7200 3050
-Wire Wire Line
-	7350 4650 7350 3150
-Connection ~ 7350 3150
 NoConn ~ 5050 2950
 NoConn ~ 5050 3050
 NoConn ~ 5050 3150
 NoConn ~ 5050 3250
-Wire Wire Line
-	6900 2850 7800 2850
-Wire Wire Line
-	7050 2950 7800 2950
-Wire Wire Line
-	7200 3050 7800 3050
-Wire Wire Line
-	7350 3150 7800 3150
 Wire Wire Line
 	5400 4150 5550 4150
@@
 Wire Wire Line
 	5400 4050 5400 4150
+Wire Wire Line
+	6250 3150 7200 3150
+Wire Wire Line
+	6250 3050 7350 3050
+Wire Wire Line
+	6250 2950 6900 2950
+Wire Wire Line
+	6250 2850 7050 2850
+Wire Wire Line
+	7350 4650 7350 3050
+Connection ~ 7350 3050
+Wire Wire Line
+	7350 3050 7800 3050
+Wire Wire Line
+	7200 4450 7200 3150
+Connection ~ 7200 3150
+Wire Wire Line
+	7200 3150 7800 3150
+Wire Wire Line
+	6900 4050 6900 2950
+Connection ~ 6900 2950
+Wire Wire Line
+	6900 2950 7800 2950
+Wire Wire Line
+	7050 4250 7050 2850
+Connection ~ 7050 2850
+Wire Wire Line
+	7050 2850 7800 2850
 $EndSCHEMATC
