File: kicad/analog/reference.sch (KiCad schematic (older format))
At the start: 13 parts, among them U901 REF5030, U902 TS5A3160

Commit message: checkpoint
Parts:
- gave numbers to parts that had none: 4
- renumbered C901 to C401, C902 to C402, C903 to C403, C904 to C404, C905 to C406, R903 to R401, TP901 to TP401, U901 to U401, U902 to U402
Changed lines of the file:
@@
 LIBS:paddle
 LIBS:analog-cache
-LIBS:processor-cache
 EELAYER 25 0
 EELAYER END
@@
 $EndDescr
 $Comp
-L C_Small C905
+L C_Small C406
 U 1 1 59CEDE0B
 P 7750 2950
-F 0 "C905" H 7760 3020 50  0000 L CNN
+F 0 "C406" H 7760 3020 50  0000 L CNN
 F 1 "0.1uF" H 7760 2870 50  0000 L CNN
 F 2 "paddle:SMD_0805" H 7750 2950 50  0001 C CNN
@@
 $EndComp
 $Comp
-L GND #PWR814
+L GND #PWR413
 U 1 1 59CEDE12
 P 7750 3100
-F 0 "#PWR814" H 7750 2850 50  0001 C CNN
+F 0 "#PWR413" H 7750 2850 50  0001 C CNN
 F 1 "GND" H 7750 2950 50  0000 C CNN
 F 2 "" H 7750 3100 50  0001 C CNN
@@
 $EndComp
 $Comp
-L GND #PWR813
+L GND #PWR412
 U 1 1 59CEDE18
 P 7300 3950
-F 0 "#PWR813" H 7300 3700 50  0001 C CNN
+F 0 "#PWR412" H 7300 3700 50  0001 C CNN
 F 1 "GND" H 7300 3800 50  0000 C CNN
 F 2 "" H 7300 3950 50  0001 C CNN
@@
 $EndComp
 $Comp
-L TEST TP901
+L TEST TP401
 U 1 1 59CEDE1E
 P 8150 3500
-F 0 "TP901" H 8150 3800 50  0000 C BNN
+F 0 "TP401" H 8150 3800 50  0000 C BNN
 F 1 "VREF" H 8150 3750 50  0000 C CNN
 F 2 "paddle:tp_th_1mm" H 8150 3500 50  0001 C CNN
@@
 $EndComp
 $Comp
-L GND #PWR811
+L GND #PWR409
 U 1 1 59CEDE2C
 P 5950 4050
-F 0 "#PWR811" H 5950 3800 50  0001 C CNN
+F 0 "#PWR409" H 5950 3800 50  0001 C CNN
 F 1 "GND" H 5950 3900 50  0000 C CNN
 F 2 "" H 5950 4050 50  0001 C CNN
@@
 $EndComp
 $Comp
-L +3.3VA #PWR812
+L +3.3VA #PWR411
 U 1 1 59CEDE47
 P 7300 2600
-F 0 "#PWR812" H 7300 2400 50  0001 C CNN
+F 0 "#PWR411" H 7300 2400 50  0001 C CNN
 F 1 "+3.3VA" H 7300 2800 50  0000 C CNN
 F 2 "" H 7300 2600 50  0001 C CNN
@@
 $EndComp
 $Comp
-L +3.3VA #PWR801
+L +3.3VA #PWR401
 U 1 1 59CEDE4D
 P 1500 3250
-F 0 "#PWR801" H 1500 3050 50  0001 C CNN
+F 0 "#PWR401" H 1500 3050 50  0001 C CNN
 F 1 "+3.3VA" H 1500 3450 50  0000 C CNN
 F 2 "" H 1500 3250 50  0001 C CNN
@@
 VREF
 $Comp
-L REF5030 U901
+L REF5030 U401
 U 1 1 59DEFBF3
 P 2700 3500
-F 0 "U901" H 2550 2700 60  0000 C CNN
+F 0 "U401" H 2550 2700 60  0000 C CNN
 F 1 "REF5030" H 2550 2600 60  0000 C CNN
 F 2 "paddle:TSSOP-8_3x3mm_Pitch0.65mm" H 2650 2700 60  0001 C CNN
@@
 $EndComp
 $Comp
-L GND #PWR803
+L GND #PWR403
 U 1 1 59DEFD98
 P 2900 4250
-F 0 "#PWR803" H 2900 4000 50  0001 C CNN
+F 0 "#PWR403" H 2900 4000 50  0001 C CNN
 F 1 "GND" H 2900 4100 50  0000 C CNN
 F 2 "" H 2900 4250 50  0001 C CNN
@@
 $EndComp
 $Comp
-L TS5A3160 U902
+L TS5A3160 U402
 U 1 1 59DF0BBD
 P 5950 3500
-F 0 "U902" H 5700 4000 50  0000 R CNN
+F 0 "U402" H 5700 4000 50  0000 R CNN
 F 1 "TS5A3160" H 5700 3900 50  0000 R CNN
 F 2 "" H 6000 3250 50  0001 L CNN
@@
 $EndComp
 $Comp
-L +3.3VA #PWR810
+L +3.3VA #PWR408
 U 1 1 59DF0C9C
 P 5950 3000
-F 0 "#PWR810" H 5950 2800 50  0001 C CNN
+F 0 "#PWR408" H 5950 2800 50  0001 C CNN
 F 1 "+3.3VA" H 5950 3200 50  0000 C CNN
 F 2 "" H 5950 3000 50  0001 C CNN
@@
 	5350 3650 5350 3750
 $Comp
-L +3.3VA #PWR805
+L +3.3VA #PWR407
 U 1 1 59DF172E
 P 4750 3650
-F 0 "#PWR805" H 4750 3450 50  0001 C CNN
+F 0 "#PWR407" H 4750 3450 50  0001 C CNN
 F 1 "+3.3VA" H 4750 3850 50  0000 C CNN
 F 2 "" H 4750 3650 50  0001 C CNN
@@
 	5950 4000 5950 4050
 $Comp
-L C_Small C901
+L C_Small C401
 U 1 1 59DF1FFE
 P 1950 3550
-F 0 "C901" H 1960 3620 50  0000 L CNN
+F 0 "C401" H 1960 3620 50  0000 L CNN
 F 1 "10uF" H 1960 3470 50  0000 L CNN
 F 2 "paddle:SMD_1206" H 1950 3550 50  0001 C CNN
@@
 Connection ~ 1950 3350
 $Comp
-L GND #PWR802
+L GND #PWR402
 U 1 1 59DF20EE
 P 1950 3700
-F 0 "#PWR802" H 1950 3450 50  0001 C CNN
+F 0 "#PWR402" H 1950 3450 50  0001 C CNN
 F 1 "GND" H 1950 3550 50  0000 C CNN
 F 2 "" H 1950 3700 50  0001 C CNN
@@
 	1950 3650 1950 3700
 $Comp
-L C_Small C903
+L C_Small C403
 U 1 1 59DF26BA
 P 3500 4000
-F 0 "C903" H 3510 4070 50  0000 L CNN
+F 0 "C403" H 3510 4070 50  0000 L CNN
 F 1 "10uF" H 3510 3920 50  0000 L CNN
 F 2 "paddle:SMD_1206" H 3500 4000 50  0001 C CNN
@@
 $EndComp
 $Comp
-L GND #PWR807
+L GND #PWR405
 U 1 1 59DF271A
 P 3500 4200
-F 0 "#PWR807" H 3500 3950 50  0001 C CNN
+F 0 "#PWR405" H 3500 3950 50  0001 C CNN
 F 1 "GND" H 3500 4050 50  0000 C CNN
 F 2 "" H 3500 4200 50  0001 C CNN
@@
 $EndComp
 $Comp
-L R_US R903
+L R_US R401
 U 1 1 59DF27CE
 P 3500 3650
-F 0 "R903" H 3525 3750 60  0000 C CNN
+F 0 "R401" H 3525 3750 60  0000 C CNN
 F 1 "1R0" H 3450 3550 60  0000 C CNN
 F 2 "paddle:SMD_0805" H 3500 3300 60  0001 C CNN
@@
 Connection ~ 3500 3350
 $Comp
-L C_Small C902
+L C_Small C402
 U 1 1 59DF29C2
 P 3200 3950
-F 0 "C902" H 3210 4020 50  0000 L CNN
+F 0 "C402" H 3210 4020 50  0000 L CNN
 F 1 "1uF" H 3210 3870 50  0000 L CNN
 F 2 "paddle:SMD_0805" H 3200 3950 50  0001 C CNN
@@
 	3200 3750 3200 3850
 $Comp
-L GND #PWR804
+L GND #PWR404
 U 1 1 59DF29C9
 P 3200 4100
-F 0 "#PWR804" H 3200 3850 50  0001 C CNN
+F 0 "#PWR404" H 3200 3850 50  0001 C CNN
 F 1 "GND" H 3200 3950 50  0000 C CNN
 F 2 "" H 3200 4100 50  0001 C CNN
@@
 	3200 4050 3200 4100
 $Comp
-L C_Small C904
+L C_Small C404
 U 1 1 59DF2AEE
 P 3850 3550
-F 0 "C904" H 3860 3620 50  0000 L CNN
+F 0 "C404" H 3860 3620 50  0000 L CNN
 F 1 "1uF" H 3860 3470 50  0000 L CNN
 F 2 "paddle:SMD_0805" H 3850 3550 50  0001 C CNN
@@
 $EndComp
 $Comp
-L GND #PWR808
+L GND #PWR406
 U 1 1 59DF2AF4
 P 3850 3700
-F 0 "#PWR808" H 3850 3450 50  0001 C CNN
+F 0 "#PWR406" H 3850 3450 50  0001 C CNN
 F 1 "GND" H 3850 3550 50  0000 C CNN
 F 2 "" H 3850 3700 50  0001 C CNN
@@
 	6400 3250 6600 3250
 $Comp
-L GND #PWR?
+L GND #PWR410
 U 1 1 59F5E52A
 P 6750 3900
-F 0 "#PWR?" H 6750 3650 50  0001 C CNN
+F 0 "#PWR410" H 6750 3650 50  0001 C CNN
 F 1 "GND" H 6750 3750 50  0000 C CNN
 F 2 "" H 6750 3900 50  0001 C CNN
@@
 $EndComp
 $Comp
-L C_Small C?
+L C_Small C405
 U 1 1 59F5E530
 P 6750 3750
-F 0 "C?" H 6760 3820 50  0000 L CNN
+F 0 "C405" H 6760 3820 50  0000 L CNN
 F 1 "0.001uF" H 6760 3670 50  0000 L CNN
 F 2 "paddle:SMD_0805" H 6750 3750 50  0001 C CNN
@@
 $EndComp
 $Comp
-L LTC2052 U?
-U 1 1 59F5E559
+L LTC2052 U201
+U 2 1 59F5E559
 P 7300 3600
-F 0 "U?" H 7300 3800 50  0000 L CNN
+F 0 "U201" H 7300 3800 50  0000 L CNN
 F 1 "LTC2052" H 7300 3400 50  0000 L CNN
 F 2 "" H 7300 3600 50  0001 C CNN
 F 3 "" H 7300 3600 50  0001 C CNN
-	1    7300 3600
+	2    7300 3600
 	1    0    0    -1
 $EndComp
@@
 	6750 3850 6750 3900
 $Comp
-L R_US R?
+L R_US R402
 U 1 1 59F5E53D
 P 4400 3350
-F 0 "R?" H 4425 3450 60  0000 C CNN
+F 0 "R402" H 4425 3450 60  0000 C CNN
 F 1 "20k" H 4350 3250 60  0000 C CNN
 F 2 "paddle:SMD_0805" H 4400 3000 60  0001 C CNN
@@
 	4750 3750 4750 3650
 $Comp
-L R_US R?
+L R_US R403
 U 1 1 59F968E9
 P 5050 3750
-F 0 "R?" H 5075 3850 60  0000 C CNN
+F 0 "R403" H 5075 3850 60  0000 C CNN
 F 1 "20k" H 5000 3650 60  0000 C CNN
 F 2 "paddle:SMD_0805" H 5050 3400 60  0001 C CNN

Commit message: Update analog board to kicad v4
Parts:
- C401, C402, C403, C404, C405, C406: symbol C_Small -> device:C_Small
- R401, R402, R403: symbol R_US -> paddle:R_US
- TP401: symbol TEST -> analog-rescue:TEST-RESCUE-analog
- U201: symbol LTC2052 -> paddle:LTC2052
- U401: symbol REF5030 -> paddle:REF5030
- U402: symbol TS5A3160 -> paddle:TS5A3160
Changed lines of the file:
@@
-EESchema Schematic File Version 2
-LIBS:power
-LIBS:device
-LIBS:transistors
-LIBS:conn
-LIBS:linear
-LIBS:regul
-LIBS:paddle
+EESchema Schematic File Version 4
 LIBS:analog-cache
-EELAYER 25 0
+EELAYER 26 0
 EELAYER END
 $Descr A4 11693 8268
@@
 $EndDescr
 $Comp
-L C_Small C406
+L device:C_Small C406
 U 1 1 59CEDE0B
 P 7750 2950
@@
 $EndComp
 $Comp
-L GND #PWR413
+L power:GND #PWR413
 U 1 1 59CEDE12
 P 7750 3100
@@
 $EndComp
 $Comp
-L GND #PWR412
+L power:GND #PWR412
 U 1 1 59CEDE18
 P 7300 3950
@@
 $EndComp
 $Comp
-L TEST TP401
+L analog-rescue:TEST-RESCUE-analog TP401
 U 1 1 59CEDE1E
 P 8150 3500
@@
 $EndComp
 $Comp
-L GND #PWR409
+L power:GND #PWR409
 U 1 1 59CEDE2C
 P 5950 4050
@@
 $EndComp
 $Comp
-L +3.3VA #PWR411
+L power:+3.3VA #PWR411
 U 1 1 59CEDE47
 P 7300 2600
@@
 $EndComp
 $Comp
-L +3.3VA #PWR401
+L power:+3.3VA #PWR401
 U 1 1 59CEDE4D
 P 1500 3250
@@
 VREF
 $Comp
-L REF5030 U401
+L paddle:REF5030 U401
 U 1 1 59DEFBF3
 P 2700 3500
@@
 $EndComp
 $Comp
-L GND #PWR403
+L power:GND #PWR403
 U 1 1 59DEFD98
 P 2900 4250
@@
 $EndComp
 $Comp
-L TS5A3160 U402
+L paddle:TS5A3160 U402
 U 1 1 59DF0BBD
 P 5950 3500
@@
 $EndComp
 $Comp
-L +3.3VA #PWR408
+L power:+3.3VA #PWR408
 U 1 1 59DF0C9C
 P 5950 3000
@@
 	5350 3650 5350 3750
 $Comp
-L +3.3VA #PWR407
+L power:+3.3VA #PWR407
 U 1 1 59DF172E
 P 4750 3650
@@
 	5950 4000 5950 4050
 $Comp
-L C_Small C401
+L device:C_Small C401
 U 1 1 59DF1FFE
 P 1950 3550
@@
 Connection ~ 1950 3350
 $Comp
-L GND #PWR402
+L power:GND #PWR402
 U 1 1 59DF20EE
 P 1950 3700
@@
 	1950 3650 1950 3700
 $Comp
-L C_Small C403
+L device:C_Small C403
 U 1 1 59DF26BA
 P 3500 4000
@@
 $EndComp
 $Comp
-L GND #PWR405
+L power:GND #PWR405
 U 1 1 59DF271A
 P 3500 4200
@@
 $EndComp
 $Comp
-L R_US R401
+L paddle:R_US R401
 U 1 1 59DF27CE
 P 3500 3650
@@
 Connection ~ 3500 3350
 $Comp
-L C_Small C402
+L device:C_Small C402
 U 1 1 59DF29C2
 P 3200 3950
@@
 	3200 3750 3200 3850
 $Comp
-L GND #PWR404
+L power:GND #PWR404
 U 1 1 59DF29C9
 P 3200 4100
@@
 	3200 4050 3200 4100
 $Comp
-L C_Small C404
+L device:C_Small C404
 U 1 1 59DF2AEE
 P 3850 3550
@@
 $EndComp
 $Comp
-L GND #PWR406
+L power:GND #PWR406
 U 1 1 59DF2AF4
 P 3850 3700
@@
 	6400 3250 6600 3250
 $Comp
-L GND #PWR410
+L power:GND #PWR410
 U 1 1 59F5E52A
 P 6750 3900
@@
 $EndComp
 $Comp
-L C_Small C405
+L device:C_Small C405
 U 1 1 59F5E530
 P 6750 3750
@@
 $EndComp
 $Comp
-L LTC2052 U201
+L paddle:LTC2052 U201
 U 2 1 59F5E559
 P 7300 3600
@@
 	6750 3850 6750 3900
 $Comp
-L R_US R402
+L paddle:R_US R402
 U 1 1 59F5E53D
 P 4400 3350
@@
 	4750 3750 4750 3650
 $Comp
-L R_US R403
+L paddle:R_US R403
 U 1 1 59F968E9
 P 5050 3750

Commit message: Simplify reference, fix connector pinout
Parts:
- removed C405: 0.001uF, paddle:SMD_0805, symbol device:C_Small
- removed C406: 0.1uF, paddle:SMD_0805, symbol device:C_Small
- removed R402, R403: 20k, paddle:SMD_0805, symbol paddle:R_US
- removed U201: LTC2052, symbol paddle:LTC2052
- removed U402: TS5A3160, symbol paddle:TS5A3160
Connections:
- net labels removed: AN_REFSEL
- wire segments 33 -> 18

Commit message: Add ADS1220 A/D
Parts:
- added J401: Conn_01x03_Male, Pin_Headers:Pin_Header_Straight_1x03_Pitch1.27mm, symbol paddle:Conn_01x03_Male
Connections:
- wire segments 18 -> 21
Changed lines of the file:
@@
 L analog-rescue:TEST-RESCUE-analog TP401
 U 1 1 59CEDE1E
-P 6300 3250
-F 0 "TP401" H 6300 3550 50  0000 C BNN
-F 1 "VREF" H 6300 3500 50  0000 C CNN
-F 2 "paddle:tp_th_1mm" H 6300 3250 50  0001 C CNN
-F 3 "" H 6300 3250 50  0001 C CNN
-	1    6300 3250
-	1    0    0    -1
-$EndComp
-$Comp
-L power:+3.3VA #PWR401
+P 7100 3950
+F 0 "TP401" H 7100 4250 50  0000 C BNN
+F 1 "VREF" H 7100 4200 50  0000 C CNN
+F 2 "paddle:tp_th_1mm" H 7100 3950 50  0001 C CNN
+F 3 "" H 7100 3950 50  0001 C CNN
+	1    7100 3950
+	1    0    0    -1
+$EndComp
+$Comp
+L power:+3.3VA #PWR0401
 U 1 1 59CEDE4D
 P 3150 3150
-F 0 "#PWR401" H 3150 2950 50  0001 C CNN
+F 0 "#PWR0401" H 3150 2950 50  0001 C CNN
 F 1 "+3.3VA" H 3150 3350 50  0000 C CNN
 F 2 "" H 3150 3150 50  0001 C CNN
@@
 Wire Wire Line
 	3150 3250 3150 3150
-Wire Wire Line
-	6050 3250 6300 3250
-Wire Wire Line
-	6300 3250 6450 3250
-Connection ~ 6300 3250
-Text HLabel 6450 3250 2    60   Output ~ 0
+Text HLabel 7200 4000 2    60   Output ~ 0
 VREF
 $Comp
@@
 $EndComp
 $Comp
-L power:GND #PWR403
+L power:GND #PWR0403
 U 1 1 59DEFD98
 P 4550 4150
-F 0 "#PWR403" H 4550 3900 50  0001 C CNN
+F 0 "#PWR0403" H 4550 3900 50  0001 C CNN
 F 1 "GND" H 4550 4000 50  0000 C CNN
 F 2 "" H 4550 4150 50  0001 C CNN
@@
 Connection ~ 3600 3250
 $Comp
-L power:GND #PWR402
+L power:GND #PWR0402
 U 1 1 59DF20EE
 P 3600 3600
-F 0 "#PWR402" H 3600 3350 50  0001 C CNN
+F 0 "#PWR0402" H 3600 3350 50  0001 C CNN
 F 1 "GND" H 3600 3450 50  0000 C CNN
 F 2 "" H 3600 3600 50  0001 C CNN
@@
 $EndComp
 $Comp
-L power:GND #PWR405
+L power:GND #PWR0405
 U 1 1 59DF271A
 P 5150 4100
-F 0 "#PWR405" H 5150 3850 50  0001 C CNN
+F 0 "#PWR0405" H 5150 3850 50  0001 C CNN
 F 1 "GND" H 5150 3950 50  0000 C CNN
 F 2 "" H 5150 4100 50  0001 C CNN
@@
 	4850 3650 4850 3750
 $Comp
-L power:GND #PWR404
+L power:GND #PWR0404
 U 1 1 59DF29C9
 P 4850 4000
-F 0 "#PWR404" H 4850 3750 50  0001 C CNN
+F 0 "#PWR0404" H 4850 3750 50  0001 C CNN
 F 1 "GND" H 4850 3850 50  0000 C CNN
 F 2 "" H 4850 4000 50  0001 C CNN
@@
 $EndComp
 $Comp
-L power:GND #PWR406
+L power:GND #PWR0406
 U 1 1 59DF2AF4
 P 5500 3600
-F 0 "#PWR406" H 5500 3350 50  0001 C CNN
+F 0 "#PWR0406" H 5500 3350 50  0001 C CNN
 F 1 "GND" H 5500 3450 50  0000 C CNN
 F 2 "" H 5500 3600 50  0001 C CNN
@@
 Wire Wire Line
 	5150 3250 5500 3250
-Wire Wire Line
-	5500 3250 6050 3250
-Wire Wire Line
-	6050 3250 6050 3250
+$Comp
+L paddle:Conn_01x03_Male J401
+U 1 1 5A9DDC91
+P 6850 3050
+F 0 "J401" V 6910 3190 50  0000 L CNN
+F 1 "Conn_01x03_Male" V 7001 3190 50  0000 L CNN
+F 2 "Pin_Headers:Pin_Header_Straight_1x03_Pitch1.27mm" H 6850 3050 50  0001 C CNN
+F 3 "~" H 6850 3050 50  0001 C CNN
+	1    6850 3050
+	0    1    1    0
+$EndComp
+Wire Wire Line
+	5500 3250 6750 3250
+Wire Wire Line
+	6950 3250 6950 3450
+Wire Wire Line
+	6950 3450 7050 3450
+$Comp
+L power:+3.3VA #PWR0407
+U 1 1 5A9DE065
+P 7050 3450
+F 0 "#PWR0407" H 7050 3250 50  0001 C CNN
+F 1 "+3.3VA" H 7050 3650 50  0000 C CNN
+F 2 "" H 7050 3450 50  0001 C CNN
+F 3 "" H 7050 3450 50  0001 C CNN
+	1    7050 3450
+	0    1    1    0
+$EndComp
+Wire Wire Line
+	6850 3250 6850 4000
+Wire Wire Line
+	6850 4000 7100 4000
+Wire Wire Line
+	7100 4000 7100 3950
+Wire Wire Line
+	7100 4000 7200 4000
+Connection ~ 7100 4000
 $EndSCHEMATC

Commit message: Switch analog to ADS1220 a/d converter
Parts:
- removed J401: Conn_01x03_Male, Pin_Headers:Pin_Header_Straight_1x03_Pitch1.27mm, symbol paddle:Conn_01x03_Male
- added C402: 100pF, paddle:SMD_0805, symbol device:C_Small
- added C403: 0.1uF, paddle:SMD_0805, symbol device:C_Small
- added R401: 20k 0.1%, paddle:SMD_0805, symbol paddle:R_US
- added R402: 20.0k 0.1%, paddle:SMD_0805, symbol paddle:R_US
- added R403: DNP, paddle:SMD_0805, symbol paddle:R_US
- added U401: LTC2052, symbol paddle:LTC2052
- renumbered C402 to C404, C403 to C405, C404 to C406, R401 to R404, U401 to U402
Connections:
- net labels added: BRIDGE_COMP
- wire segments 21 -> 42

Commit message: Analog board outline, holes, most footprints, schematic complete
Parts:
- U402: renamed from U401; footprint (none) -> paddle:SO-8_5.3x6.2mm_Pitch1.27mm
- renumbered C406 to C402, C404 to C403, C405 to C404, C403 to C405, C402 to C406, R404 to R401, R401 to R402, R402 to R403, R403 to R404, U402 to U401
Connections:
- no-connect marks 0 -> 1
Changed lines of the file:
@@
 $EndComp
 $Comp
-L power:+3.3VA #PWR0403
+L power:+3.3VA #PWR0401
 U 1 1 59CEDE4D
 P 3350 1900
-F 0 "#PWR0403" H 3350 1700 50  0001 C CNN
+F 0 "#PWR0401" H 3350 1700 50  0001 C CNN
 F 1 "+3.3VA" H 3350 2100 50  0000 C CNN
 F 2 "" H 3350 1900 50  0001 C CNN
@@
 VREF
 $Comp
-L paddle:REF5030 U402
+L paddle:REF5030 U401
 U 1 1 59DEFBF3
 P 4550 2150
-F 0 "U402" H 4400 1350 60  0000 C CNN
+F 0 "U401" H 4400 1350 60  0000 C CNN
 F 1 "REF5030" H 4400 1250 60  0000 C CNN
 F 2 "paddle:TSSOP-8_3x3mm_Pitch0.65mm" H 4500 1350 60  0001 C CNN
@@
 $EndComp
 $Comp
-L power:GND #PWR0409
+L power:GND #PWR0406
 U 1 1 59DEFD98
 P 4750 2900
-F 0 "#PWR0409" H 4750 2650 50  0001 C CNN
+F 0 "#PWR0406" H 4750 2650 50  0001 C CNN
 F 1 "GND" H 4750 2750 50  0000 C CNN
 F 2 "" H 4750 2900 50  0001 C CNN
@@
 Connection ~ 3800 2000
 $Comp
-L power:GND #PWR0404
+L power:GND #PWR0402
 U 1 1 59DF20EE
 P 3800 2350
-F 0 "#PWR0404" H 3800 2100 50  0001 C CNN
+F 0 "#PWR0402" H 3800 2100 50  0001 C CNN
 F 1 "GND" H 3800 2200 50  0000 C CNN
 F 2 "" H 3800 2350 50  0001 C CNN
@@
 	3800 2300 3800 2350
 $Comp
-L device:C_Small C405
+L device:C_Small C404
 U 1 1 59DF26BA
 P 5350 2650
-F 0 "C405" H 5360 2720 50  0000 L CNN
+F 0 "C404" H 5360 2720 50  0000 L CNN
 F 1 "10uF" H 5360 2570 50  0000 L CNN
 F 2 "paddle:SMD_1206" H 5350 2650 50  0001 C CNN
@@
 $EndComp
 $Comp
-L power:GND #PWR0411
+L power:GND #PWR0405
 U 1 1 59DF271A
 P 5350 2850
-F 0 "#PWR0411" H 5350 2600 50  0001 C CNN
+F 0 "#PWR0405" H 5350 2600 50  0001 C CNN
 F 1 "GND" H 5350 2700 50  0000 C CNN
 F 2 "" H 5350 2850 50  0001 C CNN
@@
 $EndComp
 $Comp
-L paddle:R_US R404
+L paddle:R_US R401
 U 1 1 59DF27CE
 P 5350 2300
-F 0 "R404" H 5375 2400 60  0000 C CNN
+F 0 "R401" H 5375 2400 60  0000 C CNN
 F 1 "1R0" H 5300 2200 60  0000 C CNN
 F 2 "paddle:SMD_0805" H 5350 1950 60  0001 C CNN
@@
 Connection ~ 5350 2000
 $Comp
-L device:C_Small C404
+L device:C_Small C403
 U 1 1 59DF29C2
 P 5050 2600
-F 0 "C404" H 5060 2670 50  0000 L CNN
+F 0 "C403" H 5060 2670 50  0000 L CNN
 F 1 "1uF" H 5060 2520 50  0000 L CNN
 F 2 "paddle:SMD_0805" H 5050 2600 50  0001 C CNN
@@
 	5050 2400 5050 2500
 $Comp
-L power:GND #PWR0410
+L power:GND #PWR0404
 U 1 1 59DF29C9
 P 5050 2750
-F 0 "#PWR0410" H 5050 2500 50  0001 C CNN
+F 0 "#PWR0404" H 5050 2500 50  0001 C CNN
 F 1 "GND" H 5050 2600 50  0000 C CNN
 F 2 "" H 5050 2750 50  0001 C CNN
@@
 	5050 2700 5050 2750
 $Comp
-L device:C_Small C406
+L device:C_Small C402
 U 1 1 59DF2AEE
 P 5700 2200
-F 0 "C406" H 5710 2270 50  0000 L CNN
+F 0 "C402" H 5710 2270 50  0000 L CNN
 F 1 "1uF" H 5710 2120 50  0000 L CNN
 F 2 "paddle:SMD_0805" H 5700 2200 50  0001 C CNN
@@
 $EndComp
 $Comp
-L power:GND #PWR0412
+L power:GND #PWR0403
 U 1 1 59DF2AF4
 P 5700 2350
-F 0 "#PWR0412" H 5700 2100 50  0001 C CNN
+F 0 "#PWR0403" H 5700 2100 50  0001 C CNN
 F 1 "GND" H 5700 2200 50  0000 C CNN
 F 2 "" H 5700 2350 50  0001 C CNN
@@
 BRIDGE_COMP
 $Comp
-L power:GND #PWR0405
+L power:GND #PWR0410
 U 1 1 5AA286B9
 P 3950 5200
-F 0 "#PWR0405" H 3950 4950 50  0001 C CNN
+F 0 "#PWR0410" H 3950 4950 50  0001 C CNN
 F 1 "GND" H 3950 5050 50  0000 C CNN
 F 2 "" H 3950 5200 50  0001 C CNN
@@
 $EndComp
 $Comp
-L device:C_Small C402
+L device:C_Small C406
 U 1 1 5AA286BF
 P 3950 5050
-F 0 "C402" H 3960 5120 50  0000 L CNN
+F 0 "C406" H 3960 5120 50  0000 L CNN
 F 1 "100pF" H 3960 4970 50  0000 L CNN
 F 2 "paddle:SMD_0805" H 3950 5050 50  0001 C CNN
@@
 $EndComp
 $Comp
-L power:GND #PWR0408
+L power:GND #PWR0411
 U 1 1 5AA286C6
 P 4700 5200
-F 0 "#PWR0408" H 4700 4950 50  0001 C CNN
+F 0 "#PWR0411" H 4700 4950 50  0001 C CNN
 F 1 "GND" H 4700 5050 50  0000 C CNN
 F 2 "" H 4700 5200 50  0001 C CNN
@@
 $EndComp
 $Comp
-L device:C_Small C403
+L device:C_Small C405
 U 1 1 5AA286D9
 P 4500 4350
-F 0 "C403" H 4510 4420 50  0000 L CNN
+F 0 "C405" H 4510 4420 50  0000 L CNN
 F 1 "0.1uF" H 4510 4270 50  0000 L CNN
 F 2 "paddle:SMD_0805" H 4500 4350 50  0001 C CNN
@@
 $EndComp
 $Comp
-L power:GND #PWR0406
+L power:GND #PWR0409
 U 1 1 5AA286E0
 P 4500 4500
-F 0 "#PWR0406" H 4500 4250 50  0001 C CNN
+F 0 "#PWR0409" H 4500 4250 50  0001 C CNN
 F 1 "GND" H 4500 4350 50  0000 C CNN
 F 2 "" H 4500 4500 50  0001 C CNN
@@
 	4700 4200 4700 4700
 $Comp
-L paddle:R_US R403
+L paddle:R_US R404
 U 1 1 5AA286FA
 P 4500 5800
-F 0 "R403" H 4525 5900 60  0000 C CNN
+F 0 "R404" H 4525 5900 60  0000 C CNN
 F 1 "DNP" H 4450 5700 60  0000 C CNN
 F 2 "paddle:SMD_0805" H 4500 5450 60  0001 C CNN
@@
 Connection ~ 4150 4800
 $Comp
-L paddle:LTC2052 U401
+L paddle:LTC2052 U402
 U 1 1 5AA28708
 P 4700 4900
-F 0 "U401" H 4700 5100 50  0000 L CNN
+F 0 "U402" H 4700 5100 50  0000 L CNN
 F 1 "LTC2052" H 4700 4700 50  0000 L CNN
-F 2 "" H 4700 4900 50  0001 C CNN
+F 2 "paddle:SO-8_5.3x6.2mm_Pitch1.27mm" H 4700 4900 50  0001 C CNN
 F 3 "" H 4700 4900 50  0001 C CNN
 	1    4700 4900
@@
 	5200 4900 5550 4900
 $Comp
-L paddle:R_US R401
+L paddle:R_US R402
 U 1 1 5AA2B321
 P 3300 4450
-F 0 "R401" H 3325 4550 60  0000 C CNN
+F 0 "R402" H 3325 4550 60  0000 C CNN
 F 1 "20k 0.1%" H 3250 4350 60  0000 C CNN
 F 2 "paddle:SMD_0805" H 3300 4100 60  0001 C CNN
@@
 $EndComp
 $Comp
-L paddle:R_US R402
+L paddle:R_US R403
 U 1 1 5AA2B328
 P 3300 5100
-F 0 "R402" H 3325 5200 60  0000 C CNN
+F 0 "R403" H 3325 5200 60  0000 C CNN
 F 1 "20.0k 0.1%" H 3250 5000 60  0000 C CNN
 F 2 "paddle:SMD_0805" H 3300 4750 60  0001 C CNN
@@
 Connection ~ 3300 4800
 $Comp
-L power:GND #PWR0402
+L power:GND #PWR0412
 U 1 1 5AA2B333
 P 3300 5400
-F 0 "#PWR0402" H 3300 5150 50  0001 C CNN
+F 0 "#PWR0412" H 3300 5150 50  0001 C CNN
 F 1 "GND" H 3300 5250 50  0000 C CNN
 F 2 "" H 3300 5400 50  0001 C CNN
@@
 	1    0    0    -1
 $EndComp
-Wire Wire Line
-	3300 5300 3300 5400
-$Comp
-L power:+3.3VA #PWR0401
+$Comp
+L power:+3.3VA #PWR0408
 U 1 1 5AA2B33A
 P 3300 4250
-F 0 "#PWR0401" H 3300 4050 50  0001 C CNN
+F 0 "#PWR0408" H 3300 4050 50  0001 C CNN
 F 1 "+3.3VA" H 3300 4450 50  0000 C CNN
 F 2 "" H 3300 4250 50  0001 C CNN
@@
 Wire Wire Line
 	5700 2000 6450 2000
+Wire Wire Line
+	3300 5400 3300 5300
+NoConn ~ 4050 2300
 $EndSCHEMATC
