File: kicad/analog/reference.sch (KiCad schematic (older format))
At the start: 13 parts, among them U401 REF5030, U402 LTC2052

Commit message: separate opamps for - input
Parts:
- removed C405: 0.1uF, paddle:SMD_0805, symbol device:C_Small
- removed C406: 100pF, paddle:SMD_0805, symbol device:C_Small
- removed R404: DNP, paddle:SMD_0805, symbol paddle:R_US
- removed U402: LTC2052, paddle:SO-8_5.3x6.2mm_Pitch1.27mm, symbol paddle:LTC2052
- renumbered C403 to C404, C404 to C405, C402 to C406, R402 to R401, R403 to R402, R401 to R404
Connections:
- wire segments 42 -> 23
Changed lines of the file:
@@
 $EndComp
 $Comp
-L power:+3.3VA #PWR0401
+L power:+3.3VA #PWR0403
 U 1 1 59CEDE4D
 P 3350 1900
-F 0 "#PWR0401" H 3350 1700 50  0001 C CNN
+F 0 "#PWR0403" H 3350 1700 50  0001 C CNN
 F 1 "+3.3VA" H 3350 2100 50  0000 C CNN
 F 2 "" H 3350 1900 50  0001 C CNN
@@
 $EndComp
 $Comp
-L power:GND #PWR0406
+L power:GND #PWR0409
 U 1 1 59DEFD98
 P 4750 2900
-F 0 "#PWR0406" H 4750 2650 50  0001 C CNN
+F 0 "#PWR0409" H 4750 2650 50  0001 C CNN
 F 1 "GND" H 4750 2750 50  0000 C CNN
 F 2 "" H 4750 2900 50  0001 C CNN
@@
 Connection ~ 3800 2000
 $Comp
-L power:GND #PWR0402
+L power:GND #PWR0404
 U 1 1 59DF20EE
 P 3800 2350
-F 0 "#PWR0402" H 3800 2100 50  0001 C CNN
+F 0 "#PWR0404" H 3800 2100 50  0001 C CNN
 F 1 "GND" H 3800 2200 50  0000 C CNN
 F 2 "" H 3800 2350 50  0001 C CNN
@@
 	3800 2300 3800 2350
 $Comp
-L device:C_Small C404
+L device:C_Small C405
 U 1 1 59DF26BA
 P 5350 2650
-F 0 "C404" H 5360 2720 50  0000 L CNN
+F 0 "C405" H 5360 2720 50  0000 L CNN
 F 1 "10uF" H 5360 2570 50  0000 L CNN
 F 2 "paddle:SMD_1206" H 5350 2650 50  0001 C CNN
@@
 $EndComp
 $Comp
-L power:GND #PWR0405
+L power:GND #PWR0411
 U 1 1 59DF271A
 P 5350 2850
-F 0 "#PWR0405" H 5350 2600 50  0001 C CNN
+F 0 "#PWR0411" H 5350 2600 50  0001 C CNN
 F 1 "GND" H 5350 2700 50  0000 C CNN
 F 2 "" H 5350 2850 50  0001 C CNN
@@
 $EndComp
 $Comp
-L paddle:R_US R401
+L paddle:R_US R404
 U 1 1 59DF27CE
 P 5350 2300
-F 0 "R401" H 5375 2400 60  0000 C CNN
+F 0 "R404" H 5375 2400 60  0000 C CNN
 F 1 "1R0" H 5300 2200 60  0000 C CNN
 F 2 "paddle:SMD_0805" H 5350 1950 60  0001 C CNN
@@
 Connection ~ 5350 2000
 $Comp
-L device:C_Small C403
+L device:C_Small C404
 U 1 1 59DF29C2
 P 5050 2600
-F 0 "C403" H 5060 2670 50  0000 L CNN
+F 0 "C404" H 5060 2670 50  0000 L CNN
 F 1 "1uF" H 5060 2520 50  0000 L CNN
 F 2 "paddle:SMD_0805" H 5050 2600 50  0001 C CNN
@@
 	5050 2400 5050 2500
 $Comp
-L power:GND #PWR0404
+L power:GND #PWR0410
 U 1 1 59DF29C9
 P 5050 2750
-F 0 "#PWR0404" H 5050 2500 50  0001 C CNN
+F 0 "#PWR0410" H 5050 2500 50  0001 C CNN
 F 1 "GND" H 5050 2600 50  0000 C CNN
 F 2 "" H 5050 2750 50  0001 C CNN
@@
 	5050 2700 5050 2750
 $Comp
-L device:C_Small C402
+L device:C_Small C406
 U 1 1 59DF2AEE
 P 5700 2200
-F 0 "C402" H 5710 2270 50  0000 L CNN
+F 0 "C406" H 5710 2270 50  0000 L CNN
 F 1 "1uF" H 5710 2120 50  0000 L CNN
 F 2 "paddle:SMD_0805" H 5700 2200 50  0001 C CNN
@@
 $EndComp
 $Comp
-L power:GND #PWR0403
+L power:GND #PWR0412
 U 1 1 59DF2AF4
 P 5700 2350
-F 0 "#PWR0403" H 5700 2100 50  0001 C CNN
+F 0 "#PWR0412" H 5700 2100 50  0001 C CNN
 F 1 "GND" H 5700 2200 50  0000 C CNN
 F 2 "" H 5700 2350 50  0001 C CNN
@@
 BRIDGE_COMP
 $Comp
-L power:GND #PWR0410
-U 1 1 5AA286B9
-P 3950 5200
-F 0 "#PWR0410" H 3950 4950 50  0001 C CNN
-F 1 "GND" H 3950 5050 50  0000 C CNN
-F 2 "" H 3950 5200 50  0001 C CNN
-F 3 "" H 3950 5200 50  0001 C CNN
-	1    3950 5200
-	1    0    0    -1
-$EndComp
-$Comp
-L device:C_Small C406
-U 1 1 5AA286BF
-P 3950 5050
-F 0 "C406" H 3960 5120 50  0000 L CNN
-F 1 "100pF" H 3960 4970 50  0000 L CNN
-F 2 "paddle:SMD_0805" H 3950 5050 50  0001 C CNN
-F 3 "" H 3950 5050 50  0001 C CNN
-	1    3950 5050
-	-1   0    0    1
-$EndComp
-$Comp
-L power:GND #PWR0411
-U 1 1 5AA286C6
-P 4700 5200
-F 0 "#PWR0411" H 4700 4950 50  0001 C CNN
-F 1 "GND" H 4700 5050 50  0000 C CNN
-F 2 "" H 4700 5200 50  0001 C CNN
-F 3 "" H 4700 5200 50  0001 C CNN
-	1    4700 5200
-	1    0    0    -1
-$EndComp
-$Comp
-L power:+3.3VA #PWR0407
-U 1 1 5AA286D3
-P 4700 4100
-F 0 "#PWR0407" H 4700 3900 50  0001 C CNN
-F 1 "+3.3VA" H 4700 4300 50  0000 C CNN
-F 2 "" H 4700 4100 50  0001 C CNN
-F 3 "" H 4700 4100 50  0001 C CNN
-	1    4700 4100
-	1    0    0    -1
-$EndComp
-$Comp
-L device:C_Small C405
-U 1 1 5AA286D9
-P 4500 4350
-F 0 "C405" H 4510 4420 50  0000 L CNN
-F 1 "0.1uF" H 4510 4270 50  0000 L CNN
-F 2 "paddle:SMD_0805" H 4500 4350 50  0001 C CNN
-F 3 "" H 4500 4350 50  0001 C CNN
-	1    4500 4350
-	-1   0    0    1
-$EndComp
-$Comp
-L power:GND #PWR0409
-U 1 1 5AA286E0
-P 4500 4500
-F 0 "#PWR0409" H 4500 4250 50  0001 C CNN
-F 1 "GND" H 4500 4350 50  0000 C CNN
-F 2 "" H 4500 4500 50  0001 C CNN
-F 3 "" H 4500 4500 50  0001 C CNN
-	1    4500 4500
-	1    0    0    -1
-$EndComp
-Wire Wire Line
-	5000 4900 5100 4900
-Wire Wire Line
-	4250 5000 4250 5450
-Wire Wire Line
-	3950 4800 3950 4950
-Connection ~ 3950 4800
-Wire Wire Line
-	3950 5150 3950 5200
-Connection ~ 5100 4900
-Wire Wire Line
-	5100 4900 5100 5450
-Wire Wire Line
-	4500 4450 4500 4500
-Wire Wire Line
-	4700 4100 4700 4200
-Wire Wire Line
-	4500 4250 4500 4200
-Wire Wire Line
-	4500 4200 4700 4200
-Connection ~ 4700 4200
-Wire Wire Line
-	4400 5000 4250 5000
-Wire Wire Line
-	4700 5100 4700 5200
-Wire Wire Line
-	5100 5450 4250 5450
-Wire Wire Line
-	3950 4800 4150 4800
-Wire Wire Line
-	5100 4900 5200 4900
-Wire Wire Line
-	4700 4200 4700 4700
-$Comp
-L paddle:R_US R404
-U 1 1 5AA286FA
-P 4500 5800
-F 0 "R404" H 4525 5900 60  0000 C CNN
-F 1 "DNP" H 4450 5700 60  0000 C CNN
-F 2 "paddle:SMD_0805" H 4500 5450 60  0001 C CNN
-F 3 "" H 4525 5900 60  0000 C CNN
-	1    4500 5800
-	1    0    0    -1
-$EndComp
-Wire Wire Line
-	4700 5800 5200 5800
-Wire Wire Line
-	5200 5800 5200 4900
-Connection ~ 5200 4900
-Wire Wire Line
-	4300 5800 4150 5800
-Wire Wire Line
-	4150 5800 4150 4800
-Connection ~ 4150 4800
-$Comp
-L paddle:LTC2052 U402
-U 1 1 5AA28708
-P 4700 4900
-F 0 "U402" H 4700 5100 50  0000 L CNN
-F 1 "LTC2052" H 4700 4700 50  0000 L CNN
-F 2 "paddle:SO-8_5.3x6.2mm_Pitch1.27mm" H 4700 4900 50  0001 C CNN
-F 3 "" H 4700 4900 50  0001 C CNN
-	1    4700 4900
-	1    0    0    -1
-$EndComp
-Wire Wire Line
-	5200 4900 5550 4900
-$Comp
-L paddle:R_US R402
+L paddle:R_US R401
 U 1 1 5AA2B321
 P 3300 4450
-F 0 "R402" H 3325 4550 60  0000 C CNN
+F 0 "R401" H 3325 4550 60  0000 C CNN
 F 1 "20k 0.1%" H 3250 4350 60  0000 C CNN
 F 2 "paddle:SMD_0805" H 3300 4100 60  0001 C CNN
@@
 $EndComp
 $Comp
-L paddle:R_US R403
+L paddle:R_US R402
 U 1 1 5AA2B328
 P 3300 5100
-F 0 "R403" H 3325 5200 60  0000 C CNN
+F 0 "R402" H 3325 5200 60  0000 C CNN
 F 1 "20.0k 0.1%" H 3250 5000 60  0000 C CNN
 F 2 "paddle:SMD_0805" H 3300 4750 60  0001 C CNN
@@
 	0    -1   -1   0
 $EndComp
-Wire Wire Line
-	3300 4650 3300 4800
-Wire Wire Line
-	3300 4900 3300 4800
-Connection ~ 3300 4800
-$Comp
-L power:GND #PWR0412
+$Comp
+L power:GND #PWR0402
 U 1 1 5AA2B333
 P 3300 5400
-F 0 "#PWR0412" H 3300 5150 50  0001 C CNN
+F 0 "#PWR0402" H 3300 5150 50  0001 C CNN
 F 1 "GND" H 3300 5250 50  0000 C CNN
 F 2 "" H 3300 5400 50  0001 C CNN
@@
 $EndComp
 $Comp
-L power:+3.3VA #PWR0408
+L power:+3.3VA #PWR0401
 U 1 1 5AA2B33A
 P 3300 4250
-F 0 "#PWR0408" H 3300 4050 50  0001 C CNN
+F 0 "#PWR0401" H 3300 4050 50  0001 C CNN
 F 1 "+3.3VA" H 3300 4450 50  0000 C CNN
 F 2 "" H 3300 4250 50  0001 C CNN
@@
 $EndComp
 Wire Wire Line
-	3300 4800 3950 4800
-Wire Wire Line
-	4150 4800 4400 4800
-Wire Wire Line
 	5700 2000 6450 2000
 Wire Wire Line
 	3300 5400 3300 5300
 NoConn ~ 4050 2300
+Wire Wire Line
+	3300 4650 3300 4800
+Wire Wire Line
+	3300 4800 5100 4800
+Wire Wire Line
+	5100 4800 5100 4900
+Wire Wire Line
+	5100 4900 5550 4900
+Connection ~ 3300 4800
+Wire Wire Line
+	3300 4800 3300 4900
 $EndSCHEMATC

Commit message: analog routed DRC passes
Parts:
- removed TP401: VREF, paddle:tp_th_1mm, symbol analog-rescue:TEST-RESCUE-analog
Connections:
- wire segments 23 -> 21
Changed lines of the file:
@@
 $EndDescr
-$Comp
-L analog-rescue:TEST-RESCUE-analog TP401
-U 1 1 59CEDE1E
-P 6450 1950
-F 0 "TP401" H 6450 2250 50  0000 C BNN
-F 1 "VREF" H 6450 2200 50  0000 C CNN
-F 2 "paddle:tp_th_1mm" H 6450 1950 50  0001 C CNN
-F 3 "" H 6450 1950 50  0001 C CNN
-	1    6450 1950
-	1    0    0    -1
-$EndComp
 $Comp
 L power:+3.3VA #PWR0403
@@
 Wire Wire Line
 	5350 2000 5700 2000
-Wire Wire Line
-	6450 2000 6450 1950
-Wire Wire Line
-	6450 2000 6550 2000
-Connection ~ 6450 2000
 Text HLabel 5550 4900 2    50   Output ~ 0
 BRIDGE_COMP
@@
 $EndComp
 Wire Wire Line
-	5700 2000 6450 2000
-Wire Wire Line
 	3300 5400 3300 5300
 NoConn ~ 4050 2300
@@
 Wire Wire Line
 	3300 4800 3300 4900
+Wire Wire Line
+	5700 2000 6550 2000
 $EndSCHEMATC
