File: kicad/processor/USB.sch (KiCad schematic (older format))
At the start: 18 parts, among them Q501 MMBT4401, Q502 MMBT4401, SW501 SWITCH_PUSHBUTTON, SW502 SWITCH_PUSHBUTTON, U501 USB_B_Socket, U502 SP3003-04, U503 CP2102N

Commit message: Split analog SPI to be separate from SD pins, USB bus powered, added caps, updated todo, more
Parts:
- added C503: 4.7uF, paddle:SMD_0805, symbol device:C_Small
- added C504: 0.1uF, paddle:SMD_0805, symbol device:C_Small
- added R506: 1k, paddle:R_0603, symbol paddle:R_US
- C501: value 10uF -> 4.7uF
Connections:
- wire segments 62 -> 86
Changed lines of the file:
@@
 L device:C_Small C502
 U 1 1 59C7A8A4
-P 4400 2350
-F 0 "C502" H 4410 2420 50  0000 L CNN
-F 1 "0.1uF" H 4410 2270 50  0000 L CNN
-F 2 "paddle:SMD_0805" H 4400 2350 50  0001 C CNN
-F 3 "" H 4400 2350 50  0001 C CNN
-	1    4400 2350
+P 4050 2500
+F 0 "C502" H 4060 2570 50  0000 L CNN
+F 1 "0.1uF" H 4060 2420 50  0000 L CNN
+F 2 "paddle:SMD_0805" H 4050 2500 50  0001 C CNN
+F 3 "" H 4050 2500 50  0001 C CNN
+	1    4050 2500
 	1    0    0    -1
 $EndComp
@@
 L power:GND #PWR065
 U 1 1 59C7A8AB
-P 4400 2500
-F 0 "#PWR065" H 4400 2250 50  0001 C CNN
-F 1 "GND" H 4400 2350 50  0000 C CNN
-F 2 "" H 4400 2500 50  0001 C CNN
-F 3 "" H 4400 2500 50  0001 C CNN
-	1    4400 2500
+P 4050 2650
+F 0 "#PWR065" H 4050 2400 50  0001 C CNN
+F 1 "GND" H 4050 2500 50  0000 C CNN
+F 2 "" H 4050 2650 50  0001 C CNN
+F 3 "" H 4050 2650 50  0001 C CNN
+	1    4050 2650
 	1    0    0    -1
 $EndComp
@@
 L device:C_Small C501
 U 1 1 59C7A8B1
-P 4150 2350
-F 0 "C501" H 4160 2420 50  0000 L CNN
-F 1 "10uF" H 4160 2270 50  0000 L CNN
-F 2 "paddle:SMD_0805" H 4150 2350 50  0001 C CNN
-F 3 "" H 4150 2350 50  0001 C CNN
-	1    4150 2350
+P 3800 2500
+F 0 "C501" H 3810 2570 50  0000 L CNN
+F 1 "4.7uF" H 3810 2420 50  0000 L CNN
+F 2 "paddle:SMD_0805" H 3800 2500 50  0001 C CNN
+F 3 "" H 3800 2500 50  0001 C CNN
+	1    3800 2500
 	1    0    0    -1
 $EndComp
@@
 L power:GND #PWR066
 U 1 1 59C7A8B8
-P 4150 2500
-F 0 "#PWR066" H 4150 2250 50  0001 C CNN
-F 1 "GND" H 4150 2350 50  0000 C CNN
-F 2 "" H 4150 2500 50  0001 C CNN
-F 3 "" H 4150 2500 50  0001 C CNN
-	1    4150 2500
+P 3800 2650
+F 0 "#PWR066" H 3800 2400 50  0001 C CNN
+F 1 "GND" H 3800 2500 50  0000 C CNN
+F 2 "" H 3800 2650 50  0001 C CNN
+F 3 "" H 3800 2650 50  0001 C CNN
+	1    3800 2650
 	1    0    0    -1
 $EndComp
@@
 NoConn ~ 6150 2500
 NoConn ~ 6150 2350
-Text HLabel 9300 3900 2    60   Input ~ 0
+Text HLabel 9300 3900 2    60   Output ~ 0
 TXD
 Text HLabel 9000 4050 2    60   Input ~ 0
@@
 Text HLabel 8000 4700 2    60   Input ~ 0
 BOOTLOAD*
-Text HLabel 3950 3250 2    60   Input ~ 0
+Text HLabel 2950 3250 2    60   Input ~ 0
 +VBUS
 $Comp
@@
 F 3 "" V 7250 2950 60  0001 C CNN
 	1    7300 2950
-	-1   0    0    1
+	1    0    0    -1
 $EndComp
 $Comp
@@
 F 3 "" V 7250 2650 60  0001 C CNN
 	1    7300 2650
-	-1   0    0    1
+	1    0    0    -1
 $EndComp
 $Comp
@@
 $EndComp
 $Comp
-L power:GND #PWR067
-U 1 1 59C74BF4
-P 7650 2750
-F 0 "#PWR067" H 7650 2500 50  0001 C CNN
-F 1 "GND" H 7650 2600 50  0000 C CNN
-F 2 "" H 7650 2750 50  0001 C CNN
-F 3 "" H 7650 2750 50  0001 C CNN
-	1    7650 2750
-	1    0    0    -1
-$EndComp
-$Comp
-L power:GND #PWR068
-U 1 1 59C74C20
-P 7600 3050
-F 0 "#PWR068" H 7600 2800 50  0001 C CNN
-F 1 "GND" H 7600 2900 50  0000 C CNN
-F 2 "" H 7600 3050 50  0001 C CNN
-F 3 "" H 7600 3050 50  0001 C CNN
-	1    7600 3050
-	1    0    0    -1
-$EndComp
-$Comp
 L paddle:R_US R501
 U 1 1 59C74D40
@@
 F 3 "" H 6525 2300 60  0000 C CNN
 	1    6500 2200
-	1    0    0    -1
-$EndComp
-$Comp
-L power:+3.3V #PWR069
-U 1 1 59C74D81
-P 3900 2100
-F 0 "#PWR069" H 3900 1950 50  0001 C CNN
-F 1 "+3.3V" H 3900 2240 50  0000 C CNN
-F 2 "" H 3900 2100 50  0001 C CNN
-F 3 "" H 3900 2100 50  0001 C CNN
-	1    3900 2100
 	1    0    0    -1
 $EndComp
@@
 	4500 2800 4650 2800
 Wire Wire Line
-	4650 2200 4650 2500
-Wire Wire Line
-	4400 2450 4400 2500
-Wire Wire Line
-	4400 2200 4400 2250
-Wire Wire Line
-	4150 2450 4150 2500
-Wire Wire Line
-	3900 2200 4650 2200
-Connection ~ 4400 2200
-Connection ~ 4650 2350
-Connection ~ 4650 2200
+	4050 2600 4050 2650
+Wire Wire Line
+	4050 2350 4050 2400
+Wire Wire Line
+	3800 2600 3800 2650
 Connection ~ 6900 3600
 Wire Wire Line
-	8000 4700 8000 4950
+	8000 4700 8000 4900
 Wire Wire Line
 	8050 4200 8050 3800
 Wire Wire Line
-	6150 3600 7050 3600
+	6150 3600 6900 3600
 Wire Wire Line
 	6900 5500 8000 5500
@@
 	6900 3600 6900 5500
 Wire Wire Line
-	6150 4200 8050 4200
+	6150 4200 6350 4200
 Wire Wire Line
 	6350 4200 6350 5150
 Wire Wire Line
-	8050 3100 8050 3400
+	8050 3100 8050 3300
 Connection ~ 6350 4200
 Wire Wire Line
 	6350 5150 7100 5150
 Wire Wire Line
-	4150 2250 4150 2200
-Connection ~ 4150 2200
+	3800 2400 3800 2350
 Wire Wire Line
 	6150 2650 6600 2650
@@
 	7000 2950 7150 2950
 Wire Wire Line
-	7450 2650 7650 2650
-Wire Wire Line
-	7650 2650 7650 2750
-Wire Wire Line
-	7450 2950 7600 2950
-Wire Wire Line
-	7600 2950 7600 3050
-Wire Wire Line
-	3900 2100 3900 2200
-Wire Wire Line
 	6300 2200 6150 2200
 Wire Wire Line
@@
 	6900 2200 6700 2200
 Wire Wire Line
-	2150 4200 2500 4200
+	2150 4200 2250 4200
 Wire Wire Line
 	2500 4200 2500 4350
-Wire Wire Line
-	2150 3450 4650 3450
 Wire Wire Line
 	2150 4050 2250 4050
@@
 Connection ~ 2250 4200
 Wire Wire Line
-	3900 3450 3900 3250
-Wire Wire Line
-	3900 3250 3950 3250
-Connection ~ 3900 3450
+	2900 3450 2900 3250
+Wire Wire Line
+	2900 3250 2950 3250
 Wire Wire Line
 	3600 4350 3600 3750
@@
 	2750 3600 2750 3750
 Wire Wire Line
-	2750 3750 4650 3750
+	2750 3750 3600 3750
 Wire Wire Line
 	2150 3750 2650 3750
@@
 	2850 3700 2850 3600
 Wire Wire Line
-	2850 3600 4650 3600
+	2850 3600 3400 3600
 $Comp
 L paddle:SWITCH_PUSHBUTTON SW?
@@
 NoConn ~ 3200 4350
 NoConn ~ 3300 5350
+Wire Wire Line
+	6900 3600 7050 3600
+Wire Wire Line
+	6350 4200 8050 4200
+Wire Wire Line
+	3800 2350 4050 2350
+Wire Wire Line
+	2250 4200 2500 4200
+Wire Wire Line
+	3600 3750 4650 3750
+Wire Wire Line
+	8050 3300 8050 3400
+Wire Wire Line
+	8000 4900 8000 4950
+Wire Wire Line
+	3400 3600 4650 3600
+$Comp
+L paddle:R_US R506
+U 1 1 5AA540A2
+P 4500 1850
+F 0 "R506" H 4525 1950 60  0000 C CNN
+F 1 "1k" H 4525 1750 60  0000 C CNN
+F 2 "paddle:R_0603" H 4500 1500 60  0001 C CNN
+F 3 "" H 4525 1950 60  0000 C CNN
+	1    4500 1850
+	0    1    1    0
+$EndComp
+Wire Wire Line
+	4650 2200 4500 2200
+Wire Wire Line
+	4500 2200 4500 2050
+$Comp
+L power:+3.3V #PWR0501
+U 1 1 5AA559DF
+P 4500 1600
+F 0 "#PWR0501" H 4500 1450 50  0001 C CNN
+F 1 "+3.3V" H 4500 1740 50  0000 C CNN
+F 2 "" H 4500 1600 50  0001 C CNN
+F 3 "" H 4500 1600 50  0001 C CNN
+	1    4500 1600
+	1    0    0    -1
+$EndComp
+Wire Wire Line
+	4500 1600 4500 1650
+Connection ~ 4050 2350
+$Comp
+L device:C_Small C504
+U 1 1 5AA5F6E5
+P 4150 3000
+F 0 "C504" H 4160 3070 50  0000 L CNN
+F 1 "0.1uF" H 4160 2920 50  0000 L CNN
+F 2 "paddle:SMD_0805" H 4150 3000 50  0001 C CNN
+F 3 "" H 4150 3000 50  0001 C CNN
+	1    4150 3000
+	1    0    0    -1
+$EndComp
+$Comp
+L power:GND #PWR0503
+U 1 1 5AA5F6EC
+P 4150 3150
+F 0 "#PWR0503" H 4150 2900 50  0001 C CNN
+F 1 "GND" H 4150 3000 50  0000 C CNN
+F 2 "" H 4150 3150 50  0001 C CNN
+F 3 "" H 4150 3150 50  0001 C CNN
+	1    4150 3150
+	1    0    0    -1
+$EndComp
+$Comp
+L device:C_Small C503
+U 1 1 5AA5F6F2
+P 3900 3000
+F 0 "C503" H 3910 3070 50  0000 L CNN
+F 1 "4.7uF" H 3910 2920 50  0000 L CNN
+F 2 "paddle:SMD_0805" H 3900 3000 50  0001 C CNN
+F 3 "" H 3900 3000 50  0001 C CNN
+	1    3900 3000
+	1    0    0    -1
+$EndComp
+$Comp
+L power:GND #PWR0502
+U 1 1 5AA5F6F9
+P 3900 3150
+F 0 "#PWR0502" H 3900 2900 50  0001 C CNN
+F 1 "GND" H 3900 3000 50  0000 C CNN
+F 2 "" H 3900 3150 50  0001 C CNN
+F 3 "" H 3900 3150 50  0001 C CNN
+	1    3900 3150
+	1    0    0    -1
+$EndComp
+Wire Wire Line
+	4150 3100 4150 3150
+Wire Wire Line
+	4150 2850 4150 2900
+Wire Wire Line
+	3900 3100 3900 3150
+Wire Wire Line
+	3900 2900 3900 2850
+Wire Wire Line
+	3900 2850 4150 2850
+Connection ~ 4150 2850
+Wire Wire Line
+	4050 2350 4650 2350
+Wire Wire Line
+	4350 2850 4350 2500
+Wire Wire Line
+	4350 2500 4650 2500
+Wire Wire Line
+	4150 2850 4350 2850
+Wire Wire Line
+	3900 2850 3650 2850
+Wire Wire Line
+	3650 2850 3650 3450
+Connection ~ 3900 2850
+Connection ~ 3650 3450
+Wire Wire Line
+	3650 3450 3800 3450
+Wire Wire Line
+	3800 3450 4650 3450
+Connection ~ 2900 3450
+Wire Wire Line
+	2900 3450 3650 3450
+Wire Wire Line
+	2150 3450 2900 3450
+Wire Wire Line
+	7450 2650 7750 2650
+Wire Wire Line
+	7750 2650 7750 2950
+Wire Wire Line
+	7450 2950 7750 2950
+Connection ~ 7750 2650
+Wire Wire Line
+	7750 1250 4050 1250
+Wire Wire Line
+	4050 1250 4050 2350
+Wire Wire Line
+	7750 1250 7750 2650
 $EndSCHEMATC
