File: kicad/processor/gps.sch (KiCad schematic (older format))
At the start: 12 parts, among them Q301 DMG3415U, U301 FGPMMOPA6H

Commit message: Split analog SPI to be separate from SD pins, USB bus powered, added caps, updated todo, more
Connections:
- wire segments 34 -> 40
Changed lines of the file:
@@
 	4550 4150 4550 4800
 Wire Wire Line
-	3350 2800 3350 3150
+	3350 2800 3350 2850
 $Comp
 L device:Q_PMOS_GSD Q301
@@
 ENABLE*
 Wire Wire Line
-	2950 3350 3050 3350
+	2950 3350 3000 3350
 $Comp
 L paddle:R_US R301
@@
 	5050 5500 5050 5650
 Wire Wire Line
-	5050 4050 5050 5200
+	5050 4050 5050 4900
 $Comp
 L device:C_Small C303
@@
 	3550 3750 3350 3750
 Wire Wire Line
-	3750 3750 5300 3750
+	3750 3750 4000 3750
 $Comp
 L paddle:Battery_single-cell BT301
@@
 $EndComp
 Connection ~ 5050 4900
+Wire Wire Line
+	4250 3750 4700 3750
+Wire Wire Line
+	4000 3750 4250 3750
+Wire Wire Line
+	3000 3350 3050 3350
+Wire Wire Line
+	3350 2850 3350 3150
+Wire Wire Line
+	4700 3750 5300 3750
+Wire Wire Line
+	5050 4900 5050 5200
 $EndSCHEMATC
