File: kicad/processor/power.sch (KiCad schematic (older format))
At the start: 32 parts, among them J201 V_QI, J202 GND, J203 Battery, Q201 DMG3415U, Q202 DMG3415U, Q203 DMG3414U, Q204 DMG3415U, Q205 DMG3415U, SW201 SW, U201 MCP73832, U202 NCP694-3.3

Commit message: Split analog SPI to be separate from SD pins, USB bus powered, added caps, updated todo, more
Parts:
- removed C204, C205: 10uF, paddle:SMD_0805, symbol device:C_Small
- added C204, C205: 100uF/10V, Capacitors_THT:CP_Radial_D6.3mm_P2.50mm, symbol paddle:CP
- added R211: 1R0, paddle:R_0603, symbol paddle:R_US
- D201, D203, D204: value SS24FL -> Schottky
- R205: value 1Meg -> 100k
Connections:
- wire segments 73 -> 99
Changed lines of the file:
@@
 $EndDescr
-$Comp
-L device:C_Small C204
-U 1 1 59B553A2
-P 6700 5900
-F 0 "C204" H 6710 5970 50  0000 L CNN
-F 1 "10uF" H 6710 5820 50  0000 L CNN
-F 2 "paddle:SMD_0805" H 6700 5900 50  0001 C CNN
-F 3 "" H 6700 5900 50  0001 C CNN
-	1    6700 5900
-	1    0    0    -1
-$EndComp
 $Comp
 L power:GND #PWR029
 U 1 1 59B553A9
-P 6700 6050
-F 0 "#PWR029" H 6700 5800 50  0001 C CNN
-F 1 "GND" H 6700 5900 50  0000 C CNN
-F 2 "" H 6700 6050 50  0001 C CNN
-F 3 "" H 6700 6050 50  0001 C CNN
-	1    6700 6050
+P 6700 6100
+F 0 "#PWR029" H 6700 5850 50  0001 C CNN
+F 1 "GND" H 6700 5950 50  0000 C CNN
+F 2 "" H 6700 6100 50  0001 C CNN
+F 3 "" H 6700 6100 50  0001 C CNN
+	1    6700 6100
 	1    0    0    -1
 $EndComp
@@
 $EndComp
 $Comp
-L device:C_Small C205
-U 1 1 59B5F0CA
-P 8500 5950
-F 0 "C205" H 8510 6020 50  0000 L CNN
-F 1 "10uF" H 8510 5870 50  0000 L CNN
-F 2 "paddle:SMD_0805" H 8500 5950 50  0001 C CNN
-F 3 "" H 8500 5950 50  0001 C CNN
-	1    8500 5950
-	1    0    0    -1
-$EndComp
-$Comp
 L power:GND #PWR037
 U 1 1 59B5F0D0
-P 8500 6100
-F 0 "#PWR037" H 8500 5850 50  0001 C CNN
-F 1 "GND" H 8500 5950 50  0000 C CNN
-F 2 "" H 8500 6100 50  0001 C CNN
-F 3 "" H 8500 6100 50  0001 C CNN
-	1    8500 6100
+P 8500 6150
+F 0 "#PWR037" H 8500 5900 50  0001 C CNN
+F 1 "GND" H 8500 6000 50  0000 C CNN
+F 2 "" H 8500 6150 50  0001 C CNN
+F 3 "" H 8500 6150 50  0001 C CNN
+	1    8500 6150
 	1    0    0    -1
 $EndComp
@@
 	1    5250 4750
 	1    0    0    -1
-$EndComp
-$Comp
-L paddle:Schottky D204
-U 1 1 59D1851A
-P 7950 5500
-F 0 "D204" H 7950 5600 50  0000 C CNN
-F 1 "SS24FL" H 7950 5400 50  0000 C CNN
-F 2 "paddle:D_SOD-123" H 7950 5325 50  0001 C CNN
-F 3 "" H 7950 5500 50  0001 C CNN
-	1    7950 5500
-	-1   0    0    1
 $EndComp
 $Comp
@@
 $EndComp
 Wire Wire Line
-	6700 6000 6700 6050
-Wire Wire Line
-	6700 4300 6700 5800
+	6700 4300 6700 4650
 Wire Wire Line
 	9000 1950 8900 1950
@@
 	6150 4100 6400 4100
 Wire Wire Line
-	5250 5250 5850 5250
+	5250 5250 5450 5250
 Wire Wire Line
 	6150 5450 6150 5650
@@
 	7350 6000 7450 6000
 Wire Wire Line
-	7350 5500 7350 6000
-Wire Wire Line
-	6700 5750 7450 5750
+	7350 5500 7350 5750
+Wire Wire Line
+	6700 5750 7350 5750
 Wire Wire Line
 	7450 6250 7350 6250
@@
 	4000 1850 4000 1900
 Wire Wire Line
-	3650 1850 5300 1850
+	3650 1850 3800 1850
 Connection ~ 4000 1850
 Wire Wire Line
@@
 	5200 2100 5300 2100
 Wire Wire Line
-	8450 5750 9400 5750
-Wire Wire Line
-	8500 6050 8500 6100
-Wire Wire Line
-	8500 5500 8500 5850
+	8450 5750 8500 5750
+Wire Wire Line
+	8500 5500 8500 5750
 Connection ~ 8500 5750
 Wire Wire Line
@@
 	7650 1850 7650 2350
 Wire Wire Line
-	7050 1550 7050 2950
+	7050 1550 7050 2550
 Connection ~ 7050 2850
 Wire Wire Line
 	7050 3350 7050 3400
 Wire Wire Line
-	6200 1850 8100 1850
+	6200 1850 6400 1850
 Wire Wire Line
 	7050 2550 7350 2550
@@
 Connection ~ 3800 1850
 Wire Wire Line
-	2300 2950 2900 2950
+	2300 2950 2650 2950
 Wire Wire Line
 	3800 2950 3300 2950
@@
 	2650 3450 2650 3500
 Wire Wire Line
-	2550 1850 3250 1850
+	2550 1850 2800 1850
 Wire Wire Line
 	3450 2150 3450 2600
@@
 Connection ~ 6700 3650
 Wire Wire Line
-	7650 3650 7650 2750
+	7650 3650 7650 3450
 $Comp
 L paddle:SWITCH_PUSHBUTTON SW?
@@
 Connection ~ 5700 5250
 Wire Wire Line
-	5700 4150 5700 4300
+	5700 4150 5700 4200
 Wire Wire Line
 	5700 3750 5700 3650
@@
 P 5250 4450
 F 0 "R205" H 5275 4550 60  0000 C CNN
-F 1 "1Meg" H 5275 4350 60  0000 C CNN
+F 1 "100k" H 5275 4350 60  0000 C CNN
 F 2 "paddle:R_0603" H 5250 4100 60  0001 C CNN
 F 3 "" H 5275 4550 60  0000 C CNN
@@
 $EndComp
 Wire Wire Line
-	5150 4200 5700 4200
+	5150 4200 5250 4200
 Wire Wire Line
 	5250 4200 5250 4250
@@
 Connection ~ 5250 4200
 Wire Wire Line
-	5700 3650 7650 3650
+	5700 3650 6150 3650
 $Comp
 L paddle:R_US R204
@@
 	0    1    1    0
 $EndComp
-$Comp
-L paddle:Schottky D201
-U 1 1 5A10FFA6
-P 5100 5250
-F 0 "D201" H 5100 5350 50  0000 C CNN
-F 1 "SS24FL" H 5100 5150 50  0000 C CNN
-F 2 "paddle:D_SOD-123" H 5100 5075 50  0001 C CNN
-F 3 "" H 5100 5250 50  0001 C CNN
-	1    5100 5250
-	1    0    0    -1
-$EndComp
-$Comp
-L paddle:Schottky D203
-U 1 1 5A110B0E
-P 7350 2850
-F 0 "D203" H 7350 2950 50  0000 C CNN
-F 1 "SS24FL" H 7350 2750 50  0000 C CNN
-F 2 "paddle:D_SOD-123" H 7350 2675 50  0001 C CNN
-F 3 "" H 7350 2850 50  0001 C CNN
-	1    7350 2850
-	1    0    0    -1
-$EndComp
 Text Label 5450 1550 0    60   ~ 0
 V+EXT
@@
 Text Label 7250 1850 0    60   ~ 0
 V+BAT_FUSED
+Wire Wire Line
+	7350 5750 7350 6000
+Wire Wire Line
+	7350 5750 7450 5750
+Wire Wire Line
+	6700 5750 6700 5800
+Wire Wire Line
+	4000 1850 4300 1850
+Wire Wire Line
+	4300 1850 4450 1850
+Wire Wire Line
+	8500 5750 9400 5750
+Wire Wire Line
+	8500 5750 8500 5850
+Wire Wire Line
+	7050 2850 7050 2950
+Wire Wire Line
+	7650 1850 8100 1850
+Wire Wire Line
+	7650 2850 7650 2750
+Wire Wire Line
+	7050 2550 7050 2850
+Wire Wire Line
+	6400 1850 7650 1850
+Wire Wire Line
+	3800 1850 4000 1850
+Wire Wire Line
+	2650 2950 2800 2950
+Wire Wire Line
+	2800 1850 3100 1850
+Wire Wire Line
+	6700 5100 6700 5750
+Wire Wire Line
+	3100 1850 3250 1850
+Wire Wire Line
+	2800 2950 2900 2950
+Wire Wire Line
+	6700 3650 7650 3650
+Wire Wire Line
+	5150 1850 5300 1850
+Wire Wire Line
+	5450 5250 5700 5250
+Wire Wire Line
+	6700 4650 6700 5100
+Wire Wire Line
+	4450 1850 5150 1850
+Wire Wire Line
+	5700 5250 5850 5250
+Wire Wire Line
+	6150 3650 6700 3650
+Wire Wire Line
+	5700 4200 5700 4300
+Wire Wire Line
+	5250 4200 5700 4200
+$Comp
+L paddle:Schottky D201
+U 1 1 5AA9A7C0
+P 7350 2850
+F 0 "D201" H 7350 3066 50  0000 C CNN
+F 1 "Schottky" H 7350 2975 50  0000 C CNN
+F 2 "paddle:D_SOD-123" H 7350 2675 50  0001 C CNN
+F 3 "" H 7350 2850 50  0001 C CNN
+	1    7350 2850
+	1    0    0    -1
+$EndComp
+$Comp
+L paddle:Schottky D204
+U 1 1 5AA9A948
+P 7950 5500
+F 0 "D204" H 7950 5284 50  0000 C CNN
+F 1 "Schottky" H 7950 5375 50  0000 C CNN
+F 2 "paddle:D_SOD-123" H 7950 5325 50  0001 C CNN
+F 3 "" H 7950 5500 50  0001 C CNN
+	1    7950 5500
+	-1   0    0    1
+$EndComp
+$Comp
+L paddle:Schottky D203
+U 1 1 5AA9AB71
+P 5100 5250
+F 0 "D203" H 5100 5466 50  0000 C CNN
+F 1 "Schottky" H 5100 5375 50  0000 C CNN
+F 2 "paddle:D_SOD-123" H 5100 5075 50  0001 C CNN
+F 3 "" H 5100 5250 50  0001 C CNN
+	1    5100 5250
+	1    0    0    -1
+$EndComp
+$Comp
+L paddle:CP C204
+U 1 1 5AAA2EB8
+P 6700 5950
+F 0 "C204" H 6818 5996 50  0000 L CNN
+F 1 "100uF/10V" H 6818 5905 50  0000 L CNN
+F 2 "Capacitors_THT:CP_Radial_D6.3mm_P2.50mm" H 6738 5800 50  0001 C CNN
+F 3 "" H 6700 5950 50  0001 C CNN
+	1    6700 5950
+	1    0    0    -1
+$EndComp
+$Comp
+L paddle:CP C205
+U 1 1 5AAA30EA
+P 8500 6000
+F 0 "C205" H 8618 6046 50  0000 L CNN
+F 1 "100uF/10V" H 8618 5955 50  0000 L CNN
+F 2 "Capacitors_THT:CP_Radial_D6.3mm_P2.50mm" H 8538 5850 50  0001 C CNN
+F 3 "" H 8500 6000 50  0001 C CNN
+	1    8500 6000
+	1    0    0    -1
+$EndComp
+$Comp
+L paddle:R_US R211
+U 1 1 5AAA67E6
+P 7650 3250
+F 0 "R211" H 7675 3350 60  0000 C CNN
+F 1 "1R0" H 7600 3150 60  0000 C CNN
+F 2 "paddle:R_0603" H 7650 2900 60  0001 C CNN
+F 3 "" H 7675 3350 60  0000 C CNN
+	1    7650 3250
+	0    -1   -1   0
+$EndComp
+Wire Wire Line
+	7650 3050 7650 2850
 $EndSCHEMATC

Commit message: processor laid out, todo complete, connector for wireless charge
Parts:
- removed J201: V_QI, paddle:TH_1.0, symbol processor-rescue:CONN_01X01_FEMALE-RESCUE-processor
- removed J202: GND, paddle:TH_1.0, symbol processor-rescue:CONN_01X01_FEMALE-RESCUE-processor
- added J201: S2B-PH-K-S(LF)(SN), paddle:JST_battery_header_B2B-PH-K-S, symbol processor-rescue:CONN_01X02-RESCUE-processor
- D201, D203, D204: value Schottky -> SS24FL
- J203: value Battery -> S2B-PH-K-S(LF)(SN)
Changed lines of the file:
@@
 AR Path="/59FFABEE/59B553AF" Ref="J203"  Part="1"
 F 0 "J203" H 9200 2050 50  0000 C CNN
-F 1 "Battery" V 9300 1900 50  0000 C CNN
+F 1 "S2B-PH-K-S(LF)(SN)" H 9500 1700 50  0000 C CNN
 F 2 "paddle:JST_battery_header_B2B-PH-K-S" H 9200 1900 50  0001 C CNN
 F 3 "" H 9200 1900 50  0001 C CNN
@@
 $EndComp
 $Comp
-L processor-rescue:CONN_01X01_FEMALE-RESCUE-processor J201
-U 1 1 59E5FA35
-P 2200 2950
-AR Path="/59E5FA35" Ref="J201"  Part="1"
-AR Path="/59FFABEE/59E5FA35" Ref="J201"  Part="1"
-F 0 "J201" H 2200 3050 50  0000 C CNN
-F 1 "V_QI" H 2200 2850 50  0000 C CNN
-F 2 "paddle:TH_1.0" H 2200 2950 50  0001 C CNN
-F 3 "" H 2200 2950 50  0001 C CNN
-	1    2200 2950
-	-1   0    0    1
-$EndComp
-$Comp
-L processor-rescue:CONN_01X01_FEMALE-RESCUE-processor J202
-U 1 1 59E5FAA8
-P 2200 3250
-AR Path="/59E5FAA8" Ref="J202"  Part="1"
-AR Path="/59FFABEE/59E5FAA8" Ref="J202"  Part="1"
-F 0 "J202" H 2200 3350 50  0000 C CNN
-F 1 "GND" H 2200 3150 50  0000 C CNN
-F 2 "paddle:TH_1.0" H 2200 3250 50  0001 C CNN
-F 3 "" H 2200 3250 50  0001 C CNN
-	1    2200 3250
-	-1   0    0    1
-$EndComp
-$Comp
 L power:GND #PWR042
 U 1 1 59E5FBC5
-P 2400 3350
-F 0 "#PWR042" H 2400 3100 50  0001 C CNN
-F 1 "GND" H 2400 3200 50  0000 C CNN
-F 2 "" H 2400 3350 50  0001 C CNN
-F 3 "" H 2400 3350 50  0001 C CNN
-	1    2400 3350
+P 2400 3150
+F 0 "#PWR042" H 2400 2900 50  0001 C CNN
+F 1 "GND" H 2400 3000 50  0000 C CNN
+F 2 "" H 2400 3150 50  0001 C CNN
+F 3 "" H 2400 3150 50  0001 C CNN
+	1    2400 3150
 	1    0    0    -1
 $EndComp
@@
 Connection ~ 3100 1850
 Wire Wire Line
-	2400 3350 2400 3250
-Wire Wire Line
-	2400 3250 2300 3250
+	2400 3150 2400 3050
+Wire Wire Line
+	2400 3050 2300 3050
 Connection ~ 6150 4100
 Wire Wire Line
@@
 P 7350 2850
 F 0 "D201" H 7350 3066 50  0000 C CNN
-F 1 "Schottky" H 7350 2975 50  0000 C CNN
+F 1 "SS24FL" H 7350 2975 50  0000 C CNN
 F 2 "paddle:D_SOD-123" H 7350 2675 50  0001 C CNN
 F 3 "" H 7350 2850 50  0001 C CNN
@@
 P 7950 5500
 F 0 "D204" H 7950 5284 50  0000 C CNN
-F 1 "Schottky" H 7950 5375 50  0000 C CNN
+F 1 "SS24FL" H 7950 5375 50  0000 C CNN
 F 2 "paddle:D_SOD-123" H 7950 5325 50  0001 C CNN
 F 3 "" H 7950 5500 50  0001 C CNN
@@
 P 5100 5250
 F 0 "D203" H 5100 5466 50  0000 C CNN
-F 1 "Schottky" H 5100 5375 50  0000 C CNN
+F 1 "SS24FL" H 5100 5375 50  0000 C CNN
 F 2 "paddle:D_SOD-123" H 5100 5075 50  0001 C CNN
 F 3 "" H 5100 5250 50  0001 C CNN
@@
 Wire Wire Line
 	7650 3050 7650 2850
+$Comp
+L processor-rescue:CONN_01X02-RESCUE-processor J201
+U 1 1 5AA6A05F
+P 2100 3000
+F 0 "J201" H 2100 3150 50  0000 C CNN
+F 1 "S2B-PH-K-S(LF)(SN)" H 2400 2800 50  0000 C CNN
+F 2 "paddle:JST_battery_header_B2B-PH-K-S" H 2100 3000 50  0001 C CNN
+F 3 "" H 2100 3000 50  0001 C CNN
+	1    2100 3000
+	-1   0    0    -1
+$EndComp
 $EndSCHEMATC

Commit message: As built changes: vbat sense, R207 100k, remove diode keepalive
Parts:
- added R? (x2): 10k, paddle:R_0603, symbol paddle:R_US
- D203: value SS24FL -> DNP SS24FL
- R207: value 1Meg -> 100k
Connections:
- net labels added: VBAT_SENSE
- wire segments 99 -> 105
Changed lines of the file:
@@
 P 5850 5450
 F 0 "R207" H 5875 5550 60  0000 C CNN
-F 1 "1Meg" H 5800 5350 60  0000 C CNN
+F 1 "100k" H 5800 5350 60  0000 C CNN
 F 2 "paddle:R_0603" H 5850 5100 60  0001 C CNN
 F 3 "" H 5875 5550 60  0000 C CNN
@@
 	2800 1850 3100 1850
 Wire Wire Line
-	6700 5100 6700 5750
+	6700 5100 6700 5550
 Wire Wire Line
 	3100 1850 3250 1850
@@
 P 5100 5250
 F 0 "D203" H 5100 5466 50  0000 C CNN
-F 1 "SS24FL" H 5100 5375 50  0000 C CNN
+F 1 "DNP SS24FL" H 5100 5375 50  0000 C CNN
 F 2 "paddle:D_SOD-123" H 5100 5075 50  0001 C CNN
 F 3 "" H 5100 5250 50  0001 C CNN
@@
 	-1   0    0    -1
 $EndComp
+$Comp
+L paddle:R_US R?
+U 1 1 5B1A3A3F
+P 6400 5850
+F 0 "R?" H 6425 5950 60  0000 C CNN
+F 1 "10k" H 6350 5750 60  0000 C CNN
+F 2 "paddle:R_0603" H 6400 5500 60  0001 C CNN
+F 3 "" H 6425 5950 60  0000 C CNN
+	1    6400 5850
+	0    -1   -1   0
+$EndComp
+$Comp
+L paddle:R_US R?
+U 1 1 5B1A3AC9
+P 6400 6350
+F 0 "R?" H 6425 6450 60  0000 C CNN
+F 1 "10k" H 6350 6250 60  0000 C CNN
+F 2 "paddle:R_0603" H 6400 6000 60  0001 C CNN
+F 3 "" H 6425 6450 60  0000 C CNN
+	1    6400 6350
+	0    -1   -1   0
+$EndComp
+Wire Wire Line
+	6400 6050 6400 6100
+Wire Wire Line
+	6400 5650 6400 5550
+Wire Wire Line
+	6400 5550 6700 5550
+Connection ~ 6700 5550
+Wire Wire Line
+	6700 5550 6700 5750
+$Comp
+L power:GND #PWR?
+U 1 1 5B1A93F6
+P 6400 6550
+F 0 "#PWR?" H 6400 6300 50  0001 C CNN
+F 1 "GND" H 6400 6400 50  0000 C CNN
+F 2 "" H 6400 6550 50  0001 C CNN
+F 3 "" H 6400 6550 50  0001 C CNN
+	1    6400 6550
+	1    0    0    -1
+$EndComp
+Wire Wire Line
+	6400 6100 4650 6100
+Connection ~ 6400 6100
+Wire Wire Line
+	6400 6100 6400 6150
+Text HLabel 4650 6100 0    60   Input ~ 0
+VBAT_SENSE
 $EndSCHEMATC
